File: l1/motordriver.kicad_sch (KiCad schematic)
At the start: 53 parts, among them IC2 VNH5019ATR-E, IC3 VNH5019ATR-E, IC4 VNH5019ATR-E, IC5 VNH5019ATR-E, J5 Conn_01x02, J6 Conn_01x02, J7 Conn_01x02, J8 Conn_01x02, Q1 AON6354, Q2 AON6354, Q3 AON6354, Q4 AON6354, SW2 SW_SPST

Commit message: rough ideation
Parts:
- renumbered C23 to C18, C24 to C19, C25 to C20, C26 to C21, C27 to C22, C28 to C23, C29 to C24, C30 to C25
