File: l1/l1.kicad_pcb (KiCad board)
At the start: 2 copper layers, 174 x 167.4 mm, 27 parts, among them SW1 SW_Push, U3 STM32G031K8Tx, U4 CD74HC4067SM, Y1 32KHz768

Commit message: rough ideation
Parts:
- removed C18, C19: 15p, Library:cap0603
- removed C20: 0u1, Library:cap0603
- removed H10, H11, H12, H13, H14, H15, H16, H17, H18, H19, H20, H5, H6, H7, H8, H9: MountingHole, MountingHole:MountingHole_3.2mm_M3_Pad
- removed SW1: SW_Push, Jumper:SolderJumper-2_P1.3mm_Open_TrianglePad1.0x1.5mm
- removed U3: STM32G031K8Tx, Package_QFP:LQFP-32_7x7mm_P0.8mm
- removed U4: CD74HC4067SM, Package_SO:SSOP-24_5.3x8.2mm_P0.65mm
- removed Y1: 32KHz768, Crystal:Crystal_SMD_3215-2Pin_3.2x1.5mm
- added C201: 10u, Library:cap0603, F.Cu at (1.90, 115.6)
- added C202: 0u1, Library:cap0603, F.Cu at (1.90, 118.7)
- added C203: 15p, Library:cap0603, F.Cu at (1.90, 121.8)
- added C204: 15p, Library:cap0603, F.Cu at (1.90, 124.9)
- added C205: 0u1, Library:cap0603, F.Cu at (1.90, 128.0)
- added C206: 0u1, Library:cap0603, F.Cu at (42.2, 120.1)
- added C207: 0u1, Library:cap0603, F.Cu at (42.2, 123.2)
- added D201: LED, Library:led2835, F.Cu at (2.33, 69.5)
- added D202: LED, Library:led2835, F.Cu at (2.33, 73.9)
- added D203: LED, Library:led2835, F.Cu at (2.33, 78.2)
- added D204: LED, Library:led2835, F.Cu at (2.33, 82.6)
- added D205: LED, Library:led2835, F.Cu at (2.33, 86.9)
- added D206: LED, Library:led2835, F.Cu at (2.33, 91.3)
- added D207: LED, Library:led2835, F.Cu at (7.88, 69.5)
- added D208: LED, Library:led2835, F.Cu at (7.88, 73.9)
- added D209: LED, Library:led2835, F.Cu at (7.88, 78.2)
- added D210: LED, Library:led2835, F.Cu at (7.88, 82.6)
- added D211: LED, Library:led2835, F.Cu at (7.88, 86.9)
- added D212: LED, Library:led2835, F.Cu at (7.88, 91.3)
- added D213: LED, Library:led2835, F.Cu at (13.4, 69.5)
- added D214: LED, Library:led2835, F.Cu at (13.4, 73.9)
- added D215: LED, Library:led2835, F.Cu at (13.4, 78.2)
- added D216: LED, Library:led2835, F.Cu at (13.4, 82.6)
- added D217: LED, Library:led2835, F.Cu at (13.4, 86.9)
- added D218: LED, Library:led2835, F.Cu at (13.4, 91.3)
- added D219: LED, Library:led2835, F.Cu at (19.0, 69.5)
- added D220: LED, Library:led2835, F.Cu at (19.0, 73.9)
- added D221: LED, Library:led2835, F.Cu at (19.0, 78.2)
- added D222: LED, Library:led2835, F.Cu at (19.0, 82.6)
- added D223: LED, Library:led2835, F.Cu at (19.0, 86.9)
- added D224: LED, Library:led2835, F.Cu at (19.0, 91.3)
- added D225: LED, Library:led2835, F.Cu at (24.5, 69.5)
- added D226: LED, Library:led2835, F.Cu at (24.5, 73.9)
- added D227: LED, Library:led2835, F.Cu at (24.5, 78.2)
- added D228: LED, Library:led2835, F.Cu at (24.5, 82.6)
- added D229: LED, Library:led2835, F.Cu at (24.5, 86.9)
- added D230: LED, Library:led2835, F.Cu at (24.5, 91.3)
- added J1: Conn_01x04, Connector_JST:JST_XH_S4B-XH-A_1x04_P2.50mm_Horizontal, F.Cu at (58.3, 104.5)
- added J201: Conn_01x04, Connector_JST:JST_XH_S4B-XH-A_1x04_P2.50mm_Horizontal, F.Cu at (7.72, 117.4)
- added R201: R_Photo, Library:als-pt19, F.Cu at (31.6, 102.6)
- added R202: R_Photo, Library:als-pt19, F.Cu at (31.6, 105.5)
- added R203: R_Photo, Library:als-pt19, F.Cu at (31.6, 108.4)
- added R204: R_Photo, Library:als-pt19, F.Cu at (31.6, 111.3)
- added R205: R_Photo, Library:als-pt19, F.Cu at (31.6, 114.2)
- added R206: R_Photo, Library:als-pt19, F.Cu at (31.6, 117.1)
- added R207: R_Photo, Library:als-pt19, F.Cu at (36.4, 102.6)
- added R208: R_Photo, Library:als-pt19, F.Cu at (36.4, 105.5)
- added R209: R_Photo, Library:als-pt19, F.Cu at (36.4, 108.4)
- added R210: R_Photo, Library:als-pt19, F.Cu at (36.4, 111.3)
- added R211: R_Photo, Library:als-pt19, F.Cu at (36.4, 114.2)
- added R212: R_Photo, Library:als-pt19, F.Cu at (36.4, 117.1)
- added R213: R_Photo, Library:als-pt19, F.Cu at (41.0, 102.6)
- added R214: R_Photo, Library:als-pt19, F.Cu at (41.0, 105.5)
- added R215: R_Photo, Library:als-pt19, F.Cu at (41.0, 108.4)
- added R216: R_Photo, Library:als-pt19, F.Cu at (41.0, 111.3)
- added R217: R_Photo, Library:als-pt19, F.Cu at (41.0, 114.2)
- added R218: R_Photo, Library:als-pt19, F.Cu at (41.0, 117.1)
- added R219: R_Photo, Library:als-pt19, F.Cu at (45.8, 102.6)
- added R220: R_Photo, Library:als-pt19, F.Cu at (45.8, 105.5)
- added R221: R_Photo, Library:als-pt19, F.Cu at (45.8, 108.4)
- added R222: R_Photo, Library:als-pt19, F.Cu at (45.8, 111.3)
- added R223: R_Photo, Library:als-pt19, F.Cu at (45.8, 114.2)
- added R224: R_Photo, Library:als-pt19, F.Cu at (45.8, 117.1)
- added R225: R_Photo, Library:als-pt19, F.Cu at (50.5, 102.6)
- added R226: R_Photo, Library:als-pt19, F.Cu at (50.5, 105.5)
- added R227: R_Photo, Library:als-pt19, F.Cu at (50.5, 108.4)
- added R228: R_Photo, Library:als-pt19, F.Cu at (50.5, 111.3)
- added R229: R_Photo, Library:als-pt19, F.Cu at (50.5, 114.2)
- added R230: R_Photo, Library:als-pt19, F.Cu at (50.5, 117.1)
- added R231: 3K24, Library:res0603, F.Cu at (42.2, 126.3)
- added R232: 10K, Library:res0603, F.Cu at (42.2, 129.4)
- added R233: 3K24, Library:res0603, F.Cu at (42.2, 132.5)
- added R234: 10K, Library:res0603, F.Cu at (42.2, 135.6)
- added R235: R, Library:res0603, F.Cu at (1.90, 95.0)
- added R236: R, Library:res0603, F.Cu at (1.90, 98.1)
- added R237: R, Library:res0603, F.Cu at (1.90, 101.2)
- added R238: R, Library:res0603, F.Cu at (1.90, 104.3)
- added R239: R, Library:res0603, F.Cu at (1.90, 107.4)
- added R240: R, Library:res0603, F.Cu at (1.90, 110.5)
- added R241: R, Library:res0603, F.Cu at (6.60, 95.0)
- added R242: R, Library:res0603, F.Cu at (6.60, 98.1)
- added R243: R, Library:res0603, F.Cu at (6.60, 101.2)
- added R244: R, Library:res0603, F.Cu at (6.60, 104.3)
- added R245: R, Library:res0603, F.Cu at (6.60, 107.4)
- added R246: R, Library:res0603, F.Cu at (6.60, 110.5)
- added R247: R, Library:res0603, F.Cu at (11.3, 95.0)
- added R248: R, Library:res0603, F.Cu at (11.3, 98.1)
- added R249: R, Library:res0603, F.Cu at (11.3, 101.2)
- added R250: R, Library:res0603, F.Cu at (11.3, 104.3)
- added R251: R, Library:res0603, F.Cu at (11.3, 107.4)
- added R252: R, Library:res0603, F.Cu at (11.3, 110.5)
- added R253: R, Library:res0603, F.Cu at (16.0, 95.0)
- added R254: R, Library:res0603, F.Cu at (16.0, 98.1)
- added R255: R, Library:res0603, F.Cu at (16.0, 101.2)
- added R256: R, Library:res0603, F.Cu at (16.0, 104.3)
- added R257: R, Library:res0603, F.Cu at (16.0, 107.4)
- added R258: R, Library:res0603, F.Cu at (16.0, 110.5)
- added R259: R, Library:res0603, F.Cu at (20.7, 95.0)
- added R260: R, Library:res0603, F.Cu at (20.7, 98.1)
- added R261: R, Library:res0603, F.Cu at (20.7, 101.2)
- added R262: R, Library:res0603, F.Cu at (20.7, 104.3)
- added R263: R, Library:res0603, F.Cu at (20.7, 107.4)
- added R264: R, Library:res0603, F.Cu at (20.7, 110.5)
- added SW201: SW_Push, Jumper:SolderJumper-2_P1.3mm_Open_TrianglePad1.0x1.5mm, F.Cu at (1.73, 131.3)
- added U201: STM32G071GBUx, Package_DFN_QFN:QFN-28_4x4mm_P0.5mm, F.Cu at (7.41, 130.8)
- added U202: CD74HC4067SM, Package_SO:SSOP-24_5.3x8.2mm_P0.65mm, F.Cu at (34.6, 123.6)
- added U203: CD74HC4067SM, Package_SO:SSOP-24_5.3x8.2mm_P0.65mm, F.Cu at (34.6, 133.6)
- added Y201: 32KHz768, Crystal:Crystal_SMD_3215-2Pin_3.2x1.5mm, F.Cu at (13.1, 129.3)
- H1, H2, H3, H4: footprint MountingHole:MountingHole_3.2mm_M3_Pad -> MountingHole:MountingHole_2.2mm_M2_ISO14580_Pad
- moved H2 181.5 mm to (33.3, 79.3)
- moved H4 155.8 mm to (33.3, 95.2)
- moved H1 148.5 mm to (33.3, 71.3)
- moved H3 132.7 mm to (33.3, 87.2)
Routing:
- net /Light Ring/STM32/RCC_OSC32_OUT: track 8.45 -> 0.00 mm
- net /Light Ring/STM32/NRST: track 5.36 -> 0.00 mm
- net /Light Ring/STM32/RCC_OSC32_IN: track 5.33 -> 0.00 mm
- removed copper zone on B.Cu, net GND
- removed copper zone on F.Cu, net GND
Other:
- board size 174 x 167.4 mm -> 113 x 113 mm
- rule pad_to_mask_clearance: 0.2 -> 0
- board text removed: "@sentinelsrobotics"
- board text removed: "github.com/senrobo"

Commit message: モーターエンコーダー
Parts:
- removed C201: 10u, Library:cap0603
- removed C202, C205, C206, C207: 0u1, Library:cap0603
- removed C203, C204: 15p, Library:cap0603
- removed H1, H2, H3, H4: MountingHole, MountingHole:MountingHole_2.2mm_M2_ISO14580_Pad
- removed J1, J201: Conn_01x04, Connector_JST:JST_XH_S4B-XH-A_1x04_P2.50mm_Horizontal
- removed R201, R202, R203, R204, R205, R206, R207, R208, R209, R210, R211, R212, R213, R214, R215, R216, R217, R218, R219, R220, R221, R222, R223, R224, R225, R226, R227, R228, R229, R230: R_Photo, Library:als-pt19
- removed R231, R233: 3K24, Library:res0603
- removed R232, R234: 10K, Library:res0603
- removed SW201: SW_Push, Jumper:SolderJumper-2_P1.3mm_Open_TrianglePad1.0x1.5mm
- removed U201: STM32G071GBUx, Package_DFN_QFN:QFN-28_4x4mm_P0.5mm
- removed U202, U203: CD74HC4067SM, Package_SO:SSOP-24_5.3x8.2mm_P0.65mm
- removed Y201: 32KHz768, Crystal:Crystal_SMD_3215-2Pin_3.2x1.5mm
- D201, D202, D203, D204, D205, D206, D207, D208, D209, D210, D211, D212, D213, D214, D215, D216, D217, D218, D219, D220, D221, D222, D223, D224, D225, D226, D227, D228, D229, D230, R235, R236, R237, R238, R239, R240, R241, R242, R243, R244, R245, R246, R247, R248, R249, R250, R251, R252, R253, R254, R255, R256, R257, R258, R259, R260, R261, R262, R263, R264: moved to B.Cu
- moved R242 200.6 mm to (206.4, 115.4), turned to 174 degrees
- moved R241 200.0 mm to (204.2, 125.9), turned to 162 degrees
- moved R243 199.8 mm to (206.4, 104.6), turned to -174 degrees
- moved R240 199.5 mm to (199.8, 135.8), turned to 150 degrees
- moved R244 197.8 mm to (204.2, 94.1), turned to -162 degrees
- moved D214 197.3 mm to (202.2, 130.9), turned to -24 degrees
- moved D215 196.8 mm to (205.6, 120.7), turned to -12 degrees
- moved D213 196.6 mm to (196.9, 140.3), turned to -36 degrees
- moved D216 195.2 mm to (206.7, 110.0)
- moved R239 195.1 mm to (193.5, 144.5), turned to 138 degrees
- moved R245 194.6 mm to (199.8, 84.2), turned to -150 degrees
- moved D217 192.5 mm to (205.6, 99.3), turned to 12 degrees
- moved D212 190.5 mm to (189.7, 148.3), turned to -48 degrees
- moved R246 190.1 mm to (193.5, 75.5), turned to -138 degrees
- moved R238 189.6 mm to (185.5, 151.7), turned to 126 degrees
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Connections:
- D202 pad 1: Net-(D202-K) -> Net-(D201-K)
- D203 pad 1: Net-(D203-K) -> Net-(D201-K)
- D204 pad 1: Net-(D204-K) -> Net-(D201-K)
- D205 pad 1: Net-(D205-K) -> Net-(D201-K)
- D206 pad 1: Net-(D206-K) -> Net-(D201-K)
- D207 pad 1: Net-(D207-K) -> Net-(D201-K)
- D208 pad 1: Net-(D208-K) -> Net-(D201-K)
- D209 pad 1: Net-(D209-K) -> Net-(D201-K)
- D210 pad 1: Net-(D210-K) -> Net-(D201-K)
- D211 pad 1: Net-(D211-K) -> Net-(D201-K)
- D212 pad 1: Net-(D212-K) -> Net-(D201-K)
- D213 pad 1: Net-(D213-K) -> Net-(D201-K)
- D214 pad 1: Net-(D214-K) -> Net-(D201-K)
- D215 pad 1: Net-(D215-K) -> Net-(D201-K)
- D216 pad 1: Net-(D216-K) -> Net-(D201-K)
- D217 pad 1: Net-(D217-K) -> Net-(D201-K)
- D218 pad 1: Net-(D218-K) -> Net-(D201-K)
- D219 pad 1: Net-(D219-K) -> Net-(D201-K)
- D220 pad 1: Net-(D220-K) -> Net-(D201-K)
- D221 pad 1: Net-(D221-K) -> Net-(D201-K)
- D222 pad 1: Net-(D222-K) -> Net-(D201-K)
- D223 pad 1: Net-(D223-K) -> Net-(D201-K)
- D224 pad 1: Net-(D224-K) -> Net-(D201-K)
- D225 pad 1: Net-(D225-K) -> Net-(D201-K)
- D226 pad 1: Net-(D226-K) -> Net-(D201-K)
- D227 pad 1: Net-(D227-K) -> Net-(D201-K)
- D228 pad 1: Net-(D228-K) -> Net-(D201-K)
- D229 pad 1: Net-(D229-K) -> Net-(D201-K)
- D230 pad 1: Net-(D230-K) -> Net-(D201-K)
- R236 pad 1: Net-(D202-K) -> Net-(D201-K)
- R237 pad 1: Net-(D203-K) -> Net-(D201-K)
- R238 pad 1: Net-(D204-K) -> Net-(D201-K)
- R239 pad 1: Net-(D205-K) -> Net-(D201-K)
- R240 pad 1: Net-(D206-K) -> Net-(D201-K)
- R241 pad 1: Net-(D207-K) -> Net-(D201-K)
- R242 pad 1: Net-(D208-K) -> Net-(D201-K)
- R243 pad 1: Net-(D209-K) -> Net-(D201-K)
- R244 pad 1: Net-(D210-K) -> Net-(D201-K)
- R245 pad 1: Net-(D211-K) -> Net-(D201-K)
- R246 pad 1: Net-(D212-K) -> Net-(D201-K)
- R247 pad 1: Net-(D213-K) -> Net-(D201-K)
- R248 pad 1: Net-(D214-K) -> Net-(D201-K)
- R249 pad 1: Net-(D215-K) -> Net-(D201-K)
- R250 pad 1: Net-(D216-K) -> Net-(D201-K)
- R251 pad 1: Net-(D217-K) -> Net-(D201-K)
- R252 pad 1: Net-(D218-K) -> Net-(D201-K)
- R253 pad 1: Net-(D219-K) -> Net-(D201-K)
- R254 pad 1: Net-(D220-K) -> Net-(D201-K)
- R255 pad 1: Net-(D221-K) -> Net-(D201-K)
- R256 pad 1: Net-(D222-K) -> Net-(D201-K)
- R257 pad 1: Net-(D223-K) -> Net-(D201-K)
- R258 pad 1: Net-(D224-K) -> Net-(D201-K)
- R259 pad 1: Net-(D225-K) -> Net-(D201-K)
- R260 pad 1: Net-(D226-K) -> Net-(D201-K)
- R261 pad 1: Net-(D227-K) -> Net-(D201-K)
- R262 pad 1: Net-(D228-K) -> Net-(D201-K)
- R263 pad 1: Net-(D229-K) -> Net-(D201-K)
- R264 pad 1: Net-(D230-K) -> Net-(D201-K)
Other:
- board size 113 x 113 mm -> 122 x 122 mm

Commit message: 死
Parts:
- removed R252, R253, R254, R255, R256, R257, R258, R259, R260, R261, R262, R263, R264: R, Library:res0603
- added C201: 2u2, Library:cap0603, F.Cu at (105.3, 111.2)
- added C202: 2u2, Library:cap0603, F.Cu at (105.3, 114.3)
- added C203: 2u2, Library:cap0603, F.Cu at (135.8, 95.8)
- added C204: 0u1, Library:cap0603, F.Cu at (135.8, 98.9)
- added C205: 0u1, Library:cap0603, F.Cu at (135.8, 102.0)
- added C206: 0u1, Library:cap0603, F.Cu at (135.8, 105.1)
- added C207: 0u1, Library:cap0603, F.Cu at (135.8, 108.2)
- added C208: 0u1, Library:cap0603, F.Cu at (135.8, 111.3)
- added C209: 0u1, Library:cap0603, F.Cu at (146.4, 73.7)
- added C210: 0u1, Library:cap0603, F.Cu at (146.4, 76.8)
- added C211: 0u1, Library:cap0603, F.Cu at (105.3, 82.4)
- added C212: 10n, Library:cap0603, F.Cu at (105.3, 85.5)
- added C213: 10u, Library:cap0603, F.Cu at (105.3, 88.6)
- added C214: 22u, Library:cap0603, F.Cu at (105.3, 91.7)
- added C215: 0u1, Library:cap0603, F.Cu at (105.3, 94.8)
- added C216: 22u, Library:cap0603, F.Cu at (105.3, 97.9)
- added C217: 1u, Library:cap0603, F.Cu at (110.0, 82.4)
- added C218: 0u1, Library:cap0603, F.Cu at (110.0, 85.5)
- added D231: LED, Library:led2835, F.Cu at (127.9, 78.7)
- added FB201: 100R, Library:fb0603, F.Cu at (105.3, 117.4)
- added H201: MountingHole, MountingHole:MountingHole_2.2mm_M2_ISO14580_Pad, F.Cu at (154.2, 97.0)
- added H202: MountingHole, MountingHole:MountingHole_2.2mm_M2_ISO14580_Pad, F.Cu at (154.2, 102.3)
- added H203: MountingHole, MountingHole:MountingHole_2.2mm_M2_ISO14580_Pad, F.Cu at (154.2, 107.7)
- added H204: MountingHole, MountingHole:MountingHole_2.2mm_M2_ISO14580_Pad, F.Cu at (154.2, 113.0)
- added J201: Conn_01x10, Library:526101071, F.Cu at (113.1, 105.6)
- added R201: R, Library:res0603, F.Cu at (135.8, 117.5)
- added R202: 1K, Library:res0603, F.Cu at (135.8, 120.6)
- added R203: R_Photo, Library:als-pt19, F.Cu at (135.8, 56.2)
- added R204: R_Photo, Library:als-pt19, F.Cu at (135.8, 59.1)
- added R205: R_Photo, Library:als-pt19, F.Cu at (135.8, 62.0)
- added R206: R_Photo, Library:als-pt19, F.Cu at (135.8, 64.9)
- added R207: R_Photo, Library:als-pt19, F.Cu at (135.8, 67.8)
- added R208: R_Photo, Library:als-pt19, F.Cu at (135.8, 70.7)
- added R209: R_Photo, Library:als-pt19, F.Cu at (140.5, 56.2)
- added R210: R_Photo, Library:als-pt19, F.Cu at (140.5, 59.1)
- added R211: R_Photo, Library:als-pt19, F.Cu at (140.5, 62.0)
- added R212: R_Photo, Library:als-pt19, F.Cu at (140.5, 64.9)
- added R213: R_Photo, Library:als-pt19, F.Cu at (140.5, 67.8)
- added R214: R_Photo, Library:als-pt19, F.Cu at (140.5, 70.7)
- added R215: R_Photo, Library:als-pt19, F.Cu at (145.2, 56.2)
- added R216: R_Photo, Library:als-pt19, F.Cu at (145.2, 59.1)
- added R217: R_Photo, Library:als-pt19, F.Cu at (145.2, 62.0)
- added R218: R_Photo, Library:als-pt19, F.Cu at (145.2, 64.9)
- added R219: R_Photo, Library:als-pt19, F.Cu at (145.2, 67.8)
- added R220: R_Photo, Library:als-pt19, F.Cu at (145.2, 70.7)
- added R221: R_Photo, Library:als-pt19, F.Cu at (149.9, 56.2)
- added R222: R_Photo, Library:als-pt19, F.Cu at (149.9, 59.1)
- added R223: R_Photo, Library:als-pt19, F.Cu at (149.9, 62.0)
- added R224: R_Photo, Library:als-pt19, F.Cu at (149.9, 64.9)
- added R225: R_Photo, Library:als-pt19, F.Cu at (149.9, 67.8)
- added R226: R_Photo, Library:als-pt19, F.Cu at (149.9, 70.7)
- added R227: R_Photo, Library:als-pt19, F.Cu at (154.6, 56.2)
- added R228: R_Photo, Library:als-pt19, F.Cu at (154.6, 59.1)
- added R229: R_Photo, Library:als-pt19, F.Cu at (154.6, 62.0)
- added R230: R_Photo, Library:als-pt19, F.Cu at (154.6, 64.9)
- added R231: R_Photo, Library:als-pt19, F.Cu at (154.6, 67.8)
- added R232: R_Photo, Library:als-pt19, F.Cu at (154.6, 70.7)
- added R233: 3K24, Library:res0603, F.Cu at (146.4, 79.9)
- added R234: 10K, Library:res0603, F.Cu at (146.4, 83.0)
- added SW201: SW_SPDT, Library:SS12D00G3, F.Cu at (126.6, 83.2)
- added U201: STM32F103CBTX, Package_QFP:LQFP-48_7x7mm_P0.5mm, F.Cu at (143.8, 100.0)
- added U202: CD74HC4067SM, Package_SO:SSOP-24_5.3x8.2mm_P0.65mm, F.Cu at (138.8, 77.2)
- added U203: CD74HC4067SM, Package_SO:SSOP-24_5.3x8.2mm_P0.65mm, F.Cu at (138.8, 87.2)
- added U204: TPS22917x, Library:SOT-23-6, F.Cu at (124.5, 94.4)
- added U205: ILD8150, Package_SO:Infineon_PG-DSO-8-27_3.9x4.9mm_EP2.65x3mm_ThermalVias, F.Cu at (126.0, 88.9)
- added Y201: 8Mhz, Crystal:Resonator_SMD_Murata_CSTxExxV-3Pin_3.0x1.1mm, F.Cu at (140.7, 107.4)
- D201: value LED -> RED; footprint Library:led2835 -> Library:led0603; moved to F.Cu
- D202, D203, D204, D205, D206, D207, D208, D209, D210, D211, D212, D213, D214, D215, D216, D217, D218, D219, D220, D221, D222, D223, D224, D225, D226, D227, D228, D229, D230, R250: moved to F.Cu
- R235: value R -> 3K24; moved to F.Cu
- R236, R249: value R -> 10K; moved to F.Cu
- R237, R238, R239, R240, R241, R242, R243, R244, R245, R246: value R -> 150; moved to F.Cu
- R247: value R -> 100K; moved to F.Cu
- R248: value R -> 1; moved to F.Cu
- R251: value R -> 0.3; moved to F.Cu
- moved D214 113.0 mm to (116.8, 57.0), turned to 0 degrees
- moved D209 111.4 mm to (111.3, 61.3), turned to 0 degrees
- moved D208 111.2 mm to (111.3, 57.0), turned to 0 degrees
- moved D210 110.9 mm to (111.3, 65.7), turned to 0 degrees
- moved D211 109.6 mm to (111.3, 70.0), turned to 0 degrees
- moved D212 107.7 mm to (111.3, 74.3), turned to 0 degrees
- moved D215 106.8 mm to (116.8, 61.3), turned to 0 degrees
- moved D213 105.4 mm to (111.3, 78.7), turned to 0 degrees
- moved D216 100.2 mm to (116.8, 65.7)
- moved R241 99.5 mm to (114.7, 82.4), turned to 0 degrees
- moved R240 97.4 mm to (110.0, 97.9), turned to 0 degrees
- moved R239 97.1 mm to (110.0, 94.8), turned to 0 degrees
- moved R242 96.5 mm to (114.7, 85.5), turned to 0 degrees
- moved R238 96.4 mm to (110.0, 91.7), turned to 0 degrees
- moved R237 95.2 mm to (110.0, 88.6), turned to 0 degrees
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Connections:
- D201 pad 2: +3V3 -> /Light Ring/STM32/MCU1 LED
- D202 pad 1: Net-(D201-K) -> Net-(D202-K)
- D202 pad 2: +3V3 -> /Light Ring/LED/LED VIN
- D203 pad 1: Net-(D201-K) -> Net-(D203-K)
- D203 pad 2: +3V3 -> /Light Ring/LED/LED VIN
- D204 pad 1: Net-(D201-K) -> Net-(D204-K)
- D204 pad 2: +3V3 -> /Light Ring/LED/LED VIN
- D205 pad 1: Net-(D201-K) -> Net-(D205-K)
- D205 pad 2: +3V3 -> /Light Ring/LED/LED VIN
- D206 pad 1: Net-(D201-K) -> Net-(D206-K)
- D206 pad 2: +3V3 -> /Light Ring/LED/LED VIN
- D207 pad 1: Net-(D201-K) -> Net-(D207-K)
- D207 pad 2: +3V3 -> /Light Ring/LED/LED VIN
- D208 pad 1: Net-(D201-K) -> Net-(D208-K)
- D208 pad 2: +3V3 -> /Light Ring/LED/LED VIN
- D209 pad 1: Net-(D201-K) -> Net-(D209-K)
- D209 pad 2: +3V3 -> /Light Ring/LED/LED VIN
- D210 pad 1: Net-(D201-K) -> Net-(D210-K)
- D210 pad 2: +3V3 -> /Light Ring/LED/LED VIN
- D211 pad 1: Net-(D201-K) -> Net-(D211-K)
- D211 pad 2: +3V3 -> /Light Ring/LED/LED VIN
- D212 pad 1: Net-(D201-K) -> Net-(D212-K)
- D212 pad 2: +3V3 -> Net-(D202-K)
- D213 pad 1: Net-(D201-K) -> Net-(D213-K)
- D213 pad 2: +3V3 -> Net-(D203-K)
- D214 pad 1: Net-(D201-K) -> Net-(D214-K)
- D214 pad 2: +3V3 -> Net-(D204-K)
- D215 pad 1: Net-(D201-K) -> Net-(D215-K)
- D215 pad 2: +3V3 -> Net-(D205-K)
- D216 pad 1: Net-(D201-K) -> Net-(D216-K)
- D216 pad 2: +3V3 -> Net-(D206-K)
- D217 pad 1: Net-(D201-K) -> Net-(D217-K)
- D217 pad 2: +3V3 -> Net-(D207-K)
- D218 pad 1: Net-(D201-K) -> Net-(D218-K)
- D218 pad 2: +3V3 -> Net-(D208-K)
- D219 pad 1: Net-(D201-K) -> Net-(D219-K)
- D219 pad 2: +3V3 -> Net-(D209-K)
- D220 pad 1: Net-(D201-K) -> Net-(D220-K)
- D220 pad 2: +3V3 -> Net-(D210-K)
- D221 pad 1: Net-(D201-K) -> Net-(D221-K)
- D221 pad 2: +3V3 -> Net-(D211-K)
- D222 pad 1: Net-(D201-K) -> Net-(D222-K)
- D222 pad 2: +3V3 -> Net-(D212-K)
- D223 pad 1: Net-(D201-K) -> Net-(D223-K)
- D223 pad 2: +3V3 -> Net-(D213-K)
- D224 pad 1: Net-(D201-K) -> Net-(D224-K)
- D224 pad 2: +3V3 -> Net-(D214-K)
- D225 pad 1: Net-(D201-K) -> Net-(D225-K)
- D225 pad 2: +3V3 -> Net-(D215-K)
- D226 pad 1: Net-(D201-K) -> Net-(D226-K)
- D226 pad 2: +3V3 -> Net-(D216-K)
- D227 pad 1: Net-(D201-K) -> Net-(D227-K)
- D227 pad 2: +3V3 -> Net-(D217-K)
- D228 pad 1: Net-(D201-K) -> Net-(D228-K)
- D228 pad 2: +3V3 -> Net-(D218-K)
- D229 pad 1: Net-(D201-K) -> Net-(D229-K)
- D229 pad 2: +3V3 -> Net-(D219-K)
- D230 pad 1: Net-(D201-K) -> Net-(D230-K)
- D230 pad 2: +3V3 -> Net-(D220-K)
- R235 pad 1: Net-(D201-K) -> GNDREF
- R235 pad 2: GNDREF -> /Light Ring/MUX/M2
- R236 pad 1: Net-(D201-K) -> GNDREF
- R236 pad 2: GNDREF -> Net-(U203-~{E})
- R237 pad 1: Net-(D201-K) -> Net-(D222-K)
- R237 pad 2: GNDREF -> /Light Ring/LED/LED VOUT
- R238 pad 1: Net-(D201-K) -> Net-(D223-K)
- R238 pad 2: GNDREF -> /Light Ring/LED/LED VOUT
- R239 pad 1: Net-(D201-K) -> Net-(D224-K)
- R239 pad 2: GNDREF -> /Light Ring/LED/LED VOUT
- R240 pad 1: Net-(D201-K) -> Net-(D225-K)
- R240 pad 2: GNDREF -> /Light Ring/LED/LED VOUT
- R241 pad 1: Net-(D201-K) -> Net-(D226-K)
- R241 pad 2: GNDREF -> /Light Ring/LED/LED VOUT
- R242 pad 1: Net-(D201-K) -> Net-(D227-K)
- R242 pad 2: GNDREF -> /Light Ring/LED/LED VOUT
- R243 pad 1: Net-(D201-K) -> Net-(D228-K)
- R243 pad 2: GNDREF -> /Light Ring/LED/LED VOUT
- R244 pad 1: Net-(D201-K) -> Net-(D229-K)
- R244 pad 2: GNDREF -> /Light Ring/LED/LED VOUT
- R245 pad 1: Net-(D201-K) -> Net-(D230-K)
- R245 pad 2: GNDREF -> /Light Ring/LED/LED VOUT
- R246 pad 1: Net-(D201-K) -> Net-(D231-K)
- R246 pad 2: GNDREF -> /Light Ring/LED/LED VOUT
- R247 pad 1: Net-(D201-K) -> Net-(U204-VOUT)
- R247 pad 2: GNDREF -> Net-(U204-QOD)
- R248 pad 1: Net-(D201-K) -> /Light Ring/LED/LED VOUT
- R248 pad 2: GNDREF -> Net-(R248-Pad2)
- R249 pad 1: Net-(D201-K) -> +3V3 FLIT
- R249 pad 2: GNDREF -> Net-(SW201-B)
- R250 pad 1: Net-(D201-K) -> Net-(SW201-B)
- R250 pad 2: GNDREF -> /Light Ring/LED/LED PWR
- R251 pad 1: Net-(D201-K) -> Net-(R248-Pad2)
Other:
- board outline removed
- rule pad_to_mask_clearance: 0 -> 0.15
