File: l1/l1.kicad_pcb (KiCad board)
At the start: 2 copper layers, 126.4 x 126.4 mm, 117 parts, among them J201 Conn_01x10, U201 STM32F103Cx, U202 CD74HC4067SM, U203 CD74HC4067SM, Y201 8Mhz

Commit message: MUX
Parts:
- added J202: Conn_01x04, Connector_PinHeader_2.54mm:PinHeader_1x04_P2.54mm_Horizontal, F.Cu at (40.4, 88.4)
- C201, C202, FB201: moved to B.Cu
- moved FB201 98.2 mm to (160.0, 91.8), turned to -90 degrees
- moved C201 98.0 mm to (160.8, 88.7)
- moved C202 97.1 mm to (160.8, 95.0)
- moved J201 10.00 mm to (155.5, 83.9), turned to 180 degrees
Connections:
- C209 pad 2: +3V3 -> +3V3 FILT
- C210 pad 2: +3V3 -> +3V3 FILT
- D202 pad 2: +3V3 -> +3V3 FILT
- D203 pad 2: +3V3 -> +3V3 FILT
- D204 pad 2: +3V3 -> +3V3 FILT
- D205 pad 2: +3V3 -> +3V3 FILT
- D206 pad 2: +3V3 -> +3V3 FILT
- D207 pad 2: +3V3 -> +3V3 FILT
- D208 pad 2: +3V3 -> +3V3 FILT
- D209 pad 2: +3V3 -> +3V3 FILT
- D210 pad 2: +3V3 -> +3V3 FILT
- D211 pad 2: +3V3 -> +3V3 FILT
- D212 pad 2: +3V3 -> +3V3 FILT
- D213 pad 2: +3V3 -> +3V3 FILT
- D214 pad 2: +3V3 -> +3V3 FILT
- D215 pad 2: +3V3 -> +3V3 FILT
- D216 pad 2: +3V3 -> +3V3 FILT
- D217 pad 2: +3V3 -> +3V3 FILT
- D218 pad 2: +3V3 -> +3V3 FILT
- D219 pad 2: +3V3 -> +3V3 FILT
- D220 pad 2: +3V3 -> +3V3 FILT
- D221 pad 2: +3V3 -> +3V3 FILT
- D222 pad 2: +3V3 -> +3V3 FILT
- D223 pad 2: +3V3 -> +3V3 FILT
- D224 pad 2: +3V3 -> +3V3 FILT
- D225 pad 2: +3V3 -> +3V3 FILT
- D226 pad 2: +3V3 -> +3V3 FILT
- D227 pad 2: +3V3 -> +3V3 FILT
- D228 pad 2: +3V3 -> +3V3 FILT
- D229 pad 2: +3V3 -> +3V3 FILT
- D230 pad 2: +3V3 -> +3V3 FILT
- D231 pad 2: +3V3 -> +3V3 FILT
- R203 pad 1: +3V3 -> +3V3 FILT
- R204 pad 1: +3V3 -> +3V3 FILT
- R205 pad 1: +3V3 -> +3V3 FILT
- R206 pad 1: +3V3 -> +3V3 FILT
- R207 pad 1: +3V3 -> +3V3 FILT
- R208 pad 1: +3V3 -> +3V3 FILT
- R209 pad 1: +3V3 -> +3V3 FILT
- R210 pad 1: +3V3 -> +3V3 FILT
- R211 pad 1: +3V3 -> +3V3 FILT
- R212 pad 1: +3V3 -> +3V3 FILT
- R213 pad 1: +3V3 -> +3V3 FILT
- R214 pad 1: +3V3 -> +3V3 FILT
- R215 pad 1: +3V3 -> +3V3 FILT
- R216 pad 1: +3V3 -> +3V3 FILT
- R217 pad 1: +3V3 -> +3V3 FILT
- R218 pad 1: +3V3 -> +3V3 FILT
- R219 pad 1: +3V3 -> +3V3 FILT
- R220 pad 1: +3V3 -> +3V3 FILT
- R221 pad 1: +3V3 -> +3V3 FILT
- R222 pad 1: +3V3 -> +3V3 FILT
- R223 pad 1: +3V3 -> +3V3 FILT
- R224 pad 1: +3V3 -> +3V3 FILT
- R225 pad 1: +3V3 -> +3V3 FILT
- R226 pad 1: +3V3 -> +3V3 FILT
- R227 pad 1: +3V3 -> +3V3 FILT
- R228 pad 1: +3V3 -> +3V3 FILT
- R229 pad 1: +3V3 -> +3V3 FILT
- R230 pad 1: +3V3 -> +3V3 FILT
- R231 pad 1: +3V3 -> +3V3 FILT
- R232 pad 1: +3V3 -> +3V3 FILT
- U202 pad 24: +3V3 -> +3V3 FILT
- U203 pad 24: +3V3 -> +3V3 FILT
Routing:
- net Net-(U203-I0): track 0.00 -> 57.8 mm
- net Net-(U202-I0): track 0.00 -> 57.8 mm
- net Net-(U203-I14): track 0.00 -> 52.4 mm
- net Net-(U202-I14): track 0.00 -> 52.4 mm
- net Net-(U202-I1): track 0.00 -> 52.4 mm
- net Net-(U203-I1): track 0.00 -> 52.4 mm
- net Net-(U202-I13): track 0.00 -> 46.5 mm
- net Net-(U203-I13): track 0.00 -> 46.5 mm
- net Net-(U202-I2): track 0.00 -> 45.0 mm
- net Net-(U203-I2): track 0.00 -> 45.0 mm
- net Net-(U203-I3): track 0.00 -> 41.5 mm
- net Net-(U202-I12): track 0.00 -> 41.5 mm
- net Net-(U202-I3): track 0.00 -> 41.5 mm
- net Net-(U203-I12): track 0.00 -> 41.5 mm
- net Net-(U202-I11): track 0.00 -> 37.3 mm
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