File: l1/l1.kicad_pcb (KiCad board)
At the start: 2 copper layers, 126.4 x 126.4 mm, 118 parts, among them J201 Conn_01x10, J202 Conn_01x04, U201 STM32F103Cx, U202 CD74HC4067SM, U203 CD74HC4067SM, Y201 8Mhz

Commit message: L1 finished
Parts:
- moved J202 124.3 mm to (159.0, 125.6), turned to -90 degrees
- moved R202 20.9 mm to (156.4, 120.4), turned to -90 degrees
- moved Y201 20.8 mm to (155.2, 99.6), turned to 0 degrees
- moved C202 20.1 mm to (168.6, 76.4), turned to 180 degrees
- moved C203 16.4 mm to (161.7, 115.0), turned to 0 degrees
- moved FB201 15.4 mm to (169.3, 79.5), turned to 90 degrees
- moved C205 14.5 mm to (148.7, 106.3), turned to 180 degrees
- moved C207 14.1 mm to (161.7, 112.8), turned to 0 degrees
- moved C206 14.1 mm to (152.4, 116.5), turned to -90 degrees
- moved C204 14.1 mm to (152.4, 103.5), turned to 90 degrees
- moved R201 14.0 mm to (148.7, 108.5), turned to 0 degrees
- moved C208 13.2 mm to (156.4, 103.5), turned to 90 degrees
- moved D201 13.2 mm to (156.4, 116.5), turned to 90 degrees
- moved C201 9.78 mm to (168.6, 82.7), turned to 180 degrees
- moved J201 3.89 mm to (155.2, 80.0)
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Connections:
- U201 pad 16: /Light Ring/MUX/M1 -> /Light Ring/MUX/M2
- U201 pad 19: /Light Ring/MUX/M2 -> /Light Ring/MUX/M1
- U202 pad 12: GND -> GNDREF
- U203 pad 12: GND -> GNDREF
Routing:
- net +3V3 FILT: track 17.7 -> 156.6 mm, vias 0 -> 5
- net +3V3: track 0.00 -> 60.9 mm, vias 0 -> 5
- net /Light Ring/MUX/M2: track 2.12 -> 60.9 mm, vias 0 -> 2
- net MCU SWDIO: track 0.00 -> 55.8 mm, vias 0 -> 1
- net MCU SWCLK: track 0.00 -> 52.1 mm, vias 0 -> 1
- net LED RX: track 0.00 -> 30.7 mm, vias 0 -> 1
- net LED TX: track 0.00 -> 29.7 mm, vias 0 -> 1
- net MCU RST: track 0.00 -> 27.7 mm, vias 0 -> 1
- net /Light Ring/MUX/M1: track 2.12 -> 27.9 mm
- net /Light Ring/MUX/M2 S0: track 0.00 -> 21.0 mm
- net /Light Ring/MUX/M1 S2: track 0.00 -> 19.9 mm
- net /Light Ring/MUX/M2 S1: track 0.00 -> 19.8 mm
- net /Light Ring/MUX/M1 S0: track 0.00 -> 19.7 mm
- net /Light Ring/MUX/M2 S2: track 0.00 -> 19.5 mm
- net /Light Ring/MUX/M1 S1: track 0.00 -> 18.9 mm
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
Commit message: small l1 change
Parts:
- moved C208 1.00 mm to (157.4, 103.5)
Routing:
- net +3V3 FILT: track 156.6 -> 156.0 mm

Commit message: L1
Parts:
- J202: footprint Connector_PinHeader_2.54mm:PinHeader_1x04_P2.54mm_Horizontal -> Connector_PinHeader_2.54mm:PinHeader_1x04_P2.54mm_Vertical; moved to B.Cu
- moved J202 7.65 mm to (151.4, 125.6)
Routing:
- net MCU SWCLK: track 52.1 -> 61.0 mm
- net +3V3: track 60.9 -> 66.8 mm, vias 5 -> 4
- net MCU SWDIO: track 55.8 -> 55.2 mm

Commit message: Silkscreen
Parts:
- added kibuzzard-678DDF96: G***, kibuzzard-678DDF96, B.Cu at (153.9, 129.5)
- added kibuzzard-678DDFCF: G***, kibuzzard-678DDFCF, B.Cu at (156.4, 129.5)
- added kibuzzard-678DDFF1: G***, kibuzzard-678DDFF1, B.Cu at (159.0, 129.5)
- added kibuzzard-678DE023: G***, kibuzzard-678DE023, B.Cu at (151.4, 129.5)
Connections:
- J202 pad 1: +3V3 -> +3V3 FILT
Routing:
- net +3V3: track 66.8 -> 15.3 mm, vias 4 -> 1
- net +3V3 FILT: track 156.0 -> 166.0 mm

Commit message: minor
Parts:
- C201, C202, FB201: moved to F.Cu
- moved FB201 2.90 mm to (166.5, 79.9)
- moved C202 1.32 mm to (167.3, 76.8), turned to 0 degrees
- moved C201 1.32 mm to (167.3, 83.0), turned to 0 degrees
Routing:
- net +3V3: track 15.3 -> 0.00 mm, vias 1 -> 0
- net +3V3 FILT: track 166.0 -> 164.5 mm, vias 5 -> 6
- added copper zone on F.Cu, net +3V3
- added copper zone on F.Cu, net +3V3 FILT

Commit message: l1
Parts:
- FB201: footprint Library:fb0603 -> Library:fb0805
- moved C201 0.50 mm to (167.3, 83.5)
- moved FB201 0.25 mm to (166.5, 80.2)

Commit message: Camunit
Parts:
- added C211: C, Library:cap0603, B.Cu at (159.8, 99.8)
- added SW201: IMU RST, Library:fb0805, B.Cu at (159.6, 97.2)
- added kibuzzard-679075F6: G***, kibuzzard-679075F6, B.Cu at (159.8, 95.4)
Routing:
- net MCU RST: track 27.6 -> 32.3 mm
- net LED RX: track 30.7 -> 31.8 mm
- net LED TX: track 29.7 -> 30.7 mm
