File: l1/miscellaneous.kicad_sch (KiCad schematic)
At the start: 20 parts

Commit message: rough ideation
Parts:
- removed H10, H11, H12, H13, H14, H15, H16, H17, H18, H19, H20, H5, H6, H7, H8, H9: MountingHole, MountingHole:MountingHole_3.2mm_M3_Pad, symbol Mechanical:MountingHole
- H1, H2, H3, H4: footprint MountingHole:MountingHole_3.2mm_M3_Pad -> MountingHole:MountingHole_2.2mm_M2_ISO14580_Pad

Commit message: 死
Parts:
- renumbered H1 to H201, H2 to H202, H3 to H203, H4 to H204
Changed lines of the file:
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@@
 		(dnp no)
 		(fields_autoplaced yes)
-		(property "Reference" "H3"
+		(property "Reference" "H203"
 			(at 76.2 31.7499 0)
 			(effects
@@
 			(project "l1"
 				(path "/0e4ddce5-5c0a-41d1-ab67-e7bad6d98362/7eb94f30-d7c3-42f0-a677-4d3b7a4adfd0"
-					(reference "H3")
+					(reference "H203")
 					(unit 1)
 				)
@@
 		(dnp no)
 		(fields_autoplaced yes)
-		(property "Reference" "H1"
+		(property "Reference" "H201"
 			(at 35.56 31.7499 0)
 			(effects
@@
 			(project "l1"
 				(path "/0e4ddce5-5c0a-41d1-ab67-e7bad6d98362/7eb94f30-d7c3-42f0-a677-4d3b7a4adfd0"
-					(reference "H1")
+					(reference "H201")
 					(unit 1)
 				)
@@
 		(dnp no)
 		(fields_autoplaced yes)
-		(property "Reference" "H4"
+		(property "Reference" "H204"
 			(at 96.52 31.7499 0)
 			(effects
@@
 			(project "l1"
 				(path "/0e4ddce5-5c0a-41d1-ab67-e7bad6d98362/7eb94f30-d7c3-42f0-a677-4d3b7a4adfd0"
-					(reference "H4")
+					(reference "H204")
 					(unit 1)
 				)
@@
 		(dnp no)
 		(fields_autoplaced yes)
-		(property "Reference" "H2"
+		(property "Reference" "H202"
 			(at 55.88 31.7499 0)
 			(effects
@@
 			(project "l1"
 				(path "/0e4ddce5-5c0a-41d1-ab67-e7bad6d98362/7eb94f30-d7c3-42f0-a677-4d3b7a4adfd0"
-					(reference "H2")
-					(unit 1)
-				)
+					(reference "H202")
+					(unit 1)
+				)

Commit message: Going to move to VNH
Parts:
- H201, H202, H203, H204: footprint MountingHole:MountingHole_2.2mm_M2_ISO14580_Pad -> MountingHole:MountingHole_3.2mm_M3_Pad
Changed lines of the file:
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@@
 			)
 		)
-		(property "Footprint" "MountingHole:MountingHole_2.2mm_M2_ISO14580_Pad"
+		(property "Footprint" "MountingHole:MountingHole_3.2mm_M3_Pad"
 			(at 73.66 33.02 0)
 			(effects
@@
 			)
 		)
-		(property "Footprint" "MountingHole:MountingHole_2.2mm_M2_ISO14580_Pad"
+		(property "Footprint" "MountingHole:MountingHole_3.2mm_M3_Pad"
 			(at 33.02 33.02 0)
 			(effects
@@
 			)
 		)
-		(property "Footprint" "MountingHole:MountingHole_2.2mm_M2_ISO14580_Pad"
+		(property "Footprint" "MountingHole:MountingHole_3.2mm_M3_Pad"
 			(at 93.98 33.02 0)
 			(effects
@@
 			)
 		)
-		(property "Footprint" "MountingHole:MountingHole_2.2mm_M2_ISO14580_Pad"
+		(property "Footprint" "MountingHole:MountingHole_3.2mm_M3_Pad"
 			(at 53.34 33.02 0)
 			(effects
