File: l1/mux.kicad_sch (KiCad schematic)
At the start: 38 parts, among them U4 CD74HC4067SM, U5 CD74HC4067SM

Commit message: rough ideation
Parts:
- renumbered C21 to C206, C22 to C207, R8 to R201, R9 to R202, R10 to R203, R11 to R204, R12 to R205, R13 to R206, R14 to R207, R15 to R208, R16 to R209, R17 to R210, R18 to R211, R19 to R212, R20 to R213, R21 to R214, R22 to R215, R23 to R216, R24 to R217, R25 to R218, R26 to R219, R27 to R220, R28 to R221, R29 to R222, R30 to R223, R31 to R224, R32 to R225, R33 to R226, R34 to R227, R35 to R228, R36 to R229, R37 to R230, R38 to R231, R39 to R232, R40 to R233, R41 to R234, U4 to U202, U5 to U203

Commit message: 死
Parts:
- renumbered C206 to C209, C207 to C210, R201 to R203, R202 to R204, R203 to R205, R204 to R206, R205 to R207, R206 to R208, R207 to R209, R208 to R210, R209 to R211, R210 to R212, R211 to R213, R212 to R214, R213 to R215, R214 to R216, R215 to R217, R216 to R218, R217 to R219, R218 to R220, R219 to R221, R220 to R222, R221 to R223, R222 to R224, R223 to R225, R224 to R226, R225 to R227, R226 to R228, R227 to R229, R228 to R230, R229 to R231, R230 to R232, R231 to R233, R232 to R234, R233 to R235, R234 to R236
Connections:
- net GND: no longer C209.1, C210.1, R233.1, R234.1, R235.1, R236.1
- new net GNDREF: C209.1, C210.1, R233.1, R234.1, R235.1, R236.1

Commit message: MUX
Connections:
- net +3V3 renamed +3V3 FILT

Commit message: L1 finished
Connections:
- net GND is gone; now on net GNDREF: U202.12 (GND), U203.12 (GND)
