File: l1/connections.kicad_sch (KiCad schematic)
At the start: 3 parts, among them J1 Conn_01x06, J2 Conn_01x02, J3 Conn_01x02

Commit message: rough ideation
Parts:
- removed J1: Conn_01x06, Connector_JST:JST_XH_B6B-XH-A_1x06_P2.50mm_Vertical, symbol Connector_Generic:Conn_01x06
- removed J2: Conn_01x02, Library:xt60-f, symbol Connector_Generic:Conn_01x02
- removed J3: Conn_01x02, Library:xt30-f, symbol Connector_Generic:Conn_01x02
- added J1: Conn_01x04, Connector_JST:JST_XH_S4B-XH-A_1x04_P2.50mm_Horizontal, symbol Connector_Generic:Conn_01x04
Connections:
- net +3V3: now also J1.1 (Pin_1)
- net GND: now also J1.4 (Pin_4)
- net RX: now also J1.3 (Pin_3)
- net TX: now also J1.2 (Pin_2)

Commit message: 死
Parts:
- removed J1: Conn_01x04, Connector_JST:JST_XH_S4B-XH-A_1x04_P2.50mm_Horizontal, symbol Connector_Generic:Conn_01x04
- added C201, C202: 2u2, Library:cap0603, symbol Device:C
- added FB201: 100R, Library:fb0603, symbol Device:FerriteBead
- added J201: Conn_01x10, Library:526101071, symbol Connector_Generic:Conn_01x10
Connections:
- net +3V3: now also C201.1, FB201.1, J201.1 (Pin_1)
- new net +3V3 FILT: C202.1, FB201.2
- new net GNDREF: C201.2, C202.2, J201.10 (Pin_10)
- new net LED RX: J201.3 (Pin_3)
- new net LED TX: J201.4 (Pin_4)
- new net MCU RST: J201.5 (Pin_5)
- new net MCU SWCLK: J201.7 (Pin_7)
- new net MCU SWDIO: J201.6 (Pin_6)
- no-connect marks 0 -> 3

Commit message: MUX
Parts:
- added J202: Conn_01x04, Connector_PinHeader_2.54mm:PinHeader_1x04_P2.54mm_Horizontal, symbol Connector_Generic:Conn_01x04
Connections:
- net +3V3: now also J202.1 (Pin_1)
- net GNDREF: now also J202.4 (Pin_4)
- net MCU SWCLK: now also J202.3 (Pin_3)
- net MCU SWDIO: now also J202.2 (Pin_2)

Commit message: L1
Parts:
- J202: footprint Connector_PinHeader_2.54mm:PinHeader_1x04_P2.54mm_Horizontal -> Connector_PinHeader_2.54mm:PinHeader_1x04_P2.54mm_Vertical
Changed lines of the file:
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@@
 			)
 		)
-		(property "Footprint" "Connector_PinHeader_2.54mm:PinHeader_1x04_P2.54mm_Horizontal"
+		(property "Footprint" "Connector_PinHeader_2.54mm:PinHeader_1x04_P2.54mm_Vertical"
 			(at 76.2 100.33 0)
 			(effects

Commit message: Silkscreen
Connections:
- net +3V3: no longer J202.1 (Pin_1)
- net +3V3 FILT: now also J202.1 (Pin_1)
Changed lines of the file:
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@@
+	(symbol
+		(lib_id "power:+3V3")
+		(at 83.82 95.25 0)
+		(unit 1)
+		(exclude_from_sim no)
+		(in_bom yes)
+		(on_board yes)
+		(dnp no)
+		(fields_autoplaced yes)
+		(property "Reference" "#PWR0227"
+			(at 83.82 99.06 0)
+			(effects
+				(font
+					(size 1.27 1.27)
+				)
+				(hide yes)
+			)
+		)
+		(property "Value" "+3V3 FILT"
+			(at 83.82 90.17 0)
+			(effects
+				(font
+					(size 1.27 1.27)
+				)
+			)
+		)
+		(property "Footprint" ""
+			(at 83.82 95.25 0)
+			(effects
+				(font
+					(size 1.27 1.27)
+				)
+				(hide yes)
+			)
+		)
+		(property "Datasheet" ""
+			(at 83.82 95.25 0)
+			(effects
+				(font
+					(size 1.27 1.27)
+				)
+				(hide yes)
+			)
+		)
+		(property "Description" "Power symbol creates a global label with name \"+3V3\""
+			(at 83.82 95.25 0)
+			(effects
+				(font
+					(size 1.27 1.27)
+				)
+				(hide yes)
+			)
+		)
+		(pin "1"
+		)
+		(instances
+			(project "l1"
+				(path "/0e4ddce5-5c0a-41d1-ab67-e7bad6d98362/db28a344-f5d1-410a-891a-2aeea8fe8f70"
+					(reference "#PWR0227")
+					(unit 1)
+				)
+			)
+		)
+	)
 	(symbol
 		(lib_id "power:+3V3")
@@
 					(unit 1)
 				)
-			)
-		)
-	)
-	(symbol
-		(lib_id "power:+3V3")
-		(at 83.82 95.25 0)
-		(unit 1)
-		(exclude_from_sim no)
-		(in_bom yes)
-		(on_board yes)
-		(dnp no)
-		(fields_autoplaced yes)
-		(property "Reference" "#PWR0227"
-			(at 83.82 99.06 0)
-			(effects
-				(font
-					(size 1.27 1.27)
-				)
-				(hide yes)
-			)
-		)
-		(property "Value" "+3V3"
-			(at 83.82 90.17 0)
-			(effects
-				(font
-					(size 1.27 1.27)
-				)
-			)
-		)
-		(property "Footprint" ""
-			(at 83.82 95.25 0)
-			(effects
-				(font
-					(size 1.27 1.27)
-				)
-				(hide yes)
-			)
-		)
-		(property "Datasheet" ""
-			(at 83.82 95.25 0)
-			(effects
-				(font
-					(size 1.27 1.27)
-				)
-				(hide yes)
-			)
-		)
-		(property "Description" "Power symbol creates a global label with name \"+3V3\""
-			(at 83.82 95.25 0)
-			(effects
-				(font
-					(size 1.27 1.27)
-				)
-				(hide yes)
-			)
-		)
-		(pin "1"
-		)
-		(instances
-			(project "l1"
-				(path "/0e4ddce5-5c0a-41d1-ab67-e7bad6d98362/db28a344-f5d1-410a-891a-2aeea8fe8f70"
-					(reference "#PWR0227")
-					(unit 1)
-				)

Commit message: l1
Parts:
- FB201: footprint Library:fb0603 -> Library:fb0805
Changed lines of the file:
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@@
 			)
 		)
-		(property "Footprint" "Library:fb0603"
+		(property "Footprint" "Library:fb0805"
 			(at 151.13 99.568 90)
 			(effects
