File: mdriver/topInterface/topInterface.kicad_pcb (KiCad board)
At the start: 2 copper layers, 79.4 x 31 mm, 9 parts, among them J1 Power, J2 Signal, J3 Conn_01x02, J4 Conn_01x06, J5 Conn_01x06

Commit message: driver
Parts:
- removed the J3 at (137.2, 113.9)
- renumbered J4 to J3, J5 to J4
Other:
- outline, holes or cut-outs redrawn

Commit message: driver
Parts:
- added ?: , , F.Cu at (137.1, 95.5)
Connections:
- J1 pad 1: +12V -> /FL IN 1
- J1 pad 2: +12V -> /FL IN 2
- J1 pad 3: +12V -> /BL IN 1
- J1 pad 4: +12V -> /BL IN 2
- J1 pad 5: GNDREF -> +3V3
- J1 pad 6: GNDREF -> +3V3
- J2 pad 1: /FL IN 1 -> /FR IN 1
- J2 pad 2: /FL IN 2 -> /FR IN 2
- J2 pad 3: /BL IN 1 -> /BR IN 1
- J2 pad 4: /BL IN 2 -> /BR IN 2
- J2 pad 5: /BR IN 2 -> +3V3
- J2 pad 6: /BR IN 1 -> +3V3
- J2 pad 7: /FR IN 2 -> GNDREF
- J2 pad 8: /FR IN 1 -> GNDREF
- J3 pad 2: /FL IN 1 -> /FR IN 1
- J3 pad 3: /FL IN 2 -> /FR IN 2
- J3 pad 4: /BL IN 1 -> /BR IN 1
- J3 pad 5: /BL IN 2 -> /BR IN 2
- J4 pad 2: /FR IN 1 -> /BL IN 1
- J4 pad 3: /FR IN 2 -> /BL IN 2
- J4 pad 4: /BR IN 1 -> /FL IN 1
- J4 pad 5: /BR IN 2 -> /FL IN 2
Routing:
- net +3V3: track 0.00 -> 30.5 mm
- net /FL IN 2: track 0.00 -> 25.2 mm
- net /FR IN 1: track 0.00 -> 25.2 mm
- net /FL IN 1: track 0.00 -> 17.2 mm
- net /FR IN 2: track 0.00 -> 17.2 mm
- net /BL IN 2: track 0.00 -> 16.1 mm
- net /BR IN 1: track 0.00 -> 16.1 mm
- net /BL IN 1: track 0.00 -> 9.32 mm
- net /BR IN 2: track 0.00 -> 9.32 mm
- added copper zone on B.Cu, net GNDREF
- added copper zone on F.Cu, net GNDREF
Other:
- outline, holes or cut-outs redrawn
- board text removed: "SEN LOGO"
