File: mdriver/topInterface/topInterface.kicad_pcb (KiCad board)
At the start: 2 copper layers, 79.4 x 31 mm, 9 parts, among them J1 Power, J2 Signal, J3 Conn_01x06, J4 Conn_01x06

Commit message: top interface
Parts:
- moved J1 55.2 mm to (166.1, 107.7)
- moved J2 55.2 mm to (110.9, 107.7)
Connections:
- net +3V3 renamed +5V FILT
- J1 pad 1: /FL IN 1 -> /FR IN 1
- J1 pad 3: /BL IN 1 -> /FR IN 2
- J1 pad 4: /BL IN 2 -> /FL IN 1
- J2 pad 1: /FR IN 1 -> /BR IN 1
- J2 pad 2: /FR IN 2 -> /BL IN 2
- J2 pad 3: /BR IN 1 -> /BR IN 2
- J2 pad 4: /BR IN 2 -> /BL IN 1
- J3 pad 2: /FR IN 1 -> /FR IN 2
- J3 pad 3: /FR IN 2 -> /FR IN 1
- J3 pad 4: /BR IN 1 -> /FL IN 2
- J3 pad 5: /BR IN 2 -> /FL IN 1
- J4 pad 2: /BL IN 1 -> /BR IN 2
- J4 pad 3: /BL IN 2 -> /BR IN 1
- J4 pad 4: /FL IN 1 -> /BL IN 2
- J4 pad 5: /FL IN 2 -> /BL IN 1
Routing:
- net +5V FILT: track 30.5 -> 65.4 mm
- net /BL IN 1: track 9.32 -> 29.6 mm
- net /FL IN 2: track 25.2 -> 12.1 mm
- net /FR IN 2: track 17.2 -> 29.6 mm
- net /FL IN 1: track 17.2 -> 8.58 mm
- net /FR IN 1: track 25.2 -> 19.4 mm
- net /BR IN 1: track 16.1 -> 12.1 mm
- net /BL IN 2: track 16.1 -> 19.4 mm
- net /BR IN 2: track 9.32 -> 8.58 mm

Commit message: Headers
Parts:
- moved J1 1.00 mm to (166.1, 106.7)
- moved J2 1.00 mm to (110.9, 106.7)
Changed lines of the file:
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@@
 		(locked yes)
 		(layer "F.Cu")
-		(at 166.070978 107.683123)
+		(at 166.070978 106.683123)
 		(descr "Through hole straight socket strip, 2x04, 2.54mm pitch, double cols (from Kicad 4.0.7), script generated")
 		(tags "Through hole socket strip THT 2x04 2.54mm double row")
@@
 		(locked yes)
 		(layer "F.Cu")
-		(at 110.870978 107.683123)
+		(at 110.870978 106.683123)
 		(descr "Through hole straight socket strip, 2x04, 2.54mm pitch, double cols (from Kicad 4.0.7), script generated")
 		(tags "Through hole socket strip THT 2x04 2.54mm double row")
@@
 	)
 	(segment
-		(start 106.120978 106.593123)
-		(end 108.395978 104.318123)
+		(start 108.180978 103.658123)
+		(end 116.210978 103.658123)
 		(width 0.2)
 		(layer "F.Cu")
@@
 	)
 	(segment
-		(start 108.395978 104.318123)
-		(end 116.870978 104.318123)
+		(start 116.210978 103.658123)
+		(end 125.720978 113.168123)
 		(width 0.2)
 		(layer "F.Cu")
@@
 	)
 	(segment
-		(start 106.910978 110.208123)
-		(end 106.120978 109.418123)
+		(start 106.120978 105.718123)
+		(end 108.180978 103.658123)
 		(width 0.2)
 		(layer "F.Cu")
@@
 	)
 	(segment
-		(start 116.870978 104.318123)
-		(end 125.720978 113.168123)
+		(start 108.330978 109.223123)
+		(end 106.845978 109.223123)
 		(width 0.2)
 		(layer "F.Cu")
@@
 	)
 	(segment
-		(start 106.120978 109.418123)
-		(end 106.120978 106.593123)
+		(start 106.845978 109.223123)
+		(end 106.120978 108.498123)
 		(width 0.2)
 		(layer "F.Cu")
@@
 	)
 	(segment
-		(start 108.330978 110.208123)
-		(end 106.910978 110.208123)
+		(start 106.120978 108.498123)
+		(end 106.120978 105.718123)
 		(width 0.2)
 		(layer "F.Cu")
@@
 	)
 	(segment
-		(start 165.080978 105.708123)
-		(end 158.655978 105.708123)
+		(start 166.080978 105.258123)
+		(end 165.840978 105.018123)
 		(width 0.2)
 		(layer "F.Cu")
@@
 	)
 	(segment
-		(start 158.655978 105.708123)
-		(end 151.180978 113.183123)
+		(start 159.350978 105.018123)
+		(end 151.190978 113.178123)
 		(width 0.2)
 		(layer "F.Cu")
@@
 	)
 	(segment
-		(start 166.070978 106.698123)
-		(end 165.080978 105.708123)
+		(start 166.080978 105.868123)
+		(end 166.080978 105.258123)
 		(width 0.2)
 		(layer "F.Cu")
@@
 	)
 	(segment
-		(start 166.070978 107.683123)
-		(end 166.070978 106.698123)
+		(start 165.840978 105.018123)
+		(end 159.350978 105.018123)
 		(width 0.2)
 		(layer "F.Cu")
@@
 	)
 	(segment
-		(start 110.870978 110.208123)
-		(end 115.260978 110.208123)
+		(start 110.880978 109.233123)
+		(end 114.285978 109.233123)
 		(width 0.2)
 		(layer "F.Cu")
@@
 	)
 	(segment
-		(start 115.260978 110.208123)
+		(start 114.285978 109.233123)
 		(end 118.220978 113.168123)
 		(width 0.2)
@@
 	)
 	(segment
-		(start 163.530978 107.683123)
-		(end 159.180978 107.683123)
+		(start 110.870978 109.223123)
+		(end 110.880978 109.233123)
+		(width 0.2)
+		(layer "F.Cu")
+		(net 4)
+	)
+	(segment
+		(start 160.175978 106.693123)
+		(end 153.690978 113.178123)
 		(width 0.2)
 		(layer "F.Cu")
@@
 	)
 	(segment
-		(start 159.180978 107.683123)
-		(end 153.680978 113.183123)
+		(start 163.540978 106.693123)
+		(end 160.175978 106.693123)
 		(width 0.2)
 		(layer "F.Cu")
@@
 	)
 	(segment
-		(start 115.220978 107.668123)
+		(start 114.235978 106.683123)
 		(end 120.720978 113.168123)
 		(width 0.2)
@@
 	)
 	(segment
-		(start 110.870978 107.668123)
-		(end 115.220978 107.668123)
+		(start 110.870978 106.683123)
+		(end 114.235978 106.683123)
 		(width 0.2)
 		(layer "F.Cu")
@@
 	)
 	(segment
-		(start 159.140978 110.223123)
-		(end 156.180978 113.183123)
+		(start 163.530978 109.243123)
+		(end 160.125978 109.243123)
 		(width 0.2)
 		(layer "F.Cu")
@@
 	)
 	(segment
-		(start 163.530978 110.223123)
-		(end 159.140978 110.223123)
+		(start 160.125978 109.243123)
+		(end 156.190978 113.178123)
 		(width 0.2)
 		(layer "F.Cu")
@@
 	)
 	(segment
-		(start 108.330978 107.668123)
-		(end 108.330978 106.683123)
+		(start 108.655978 105.008123)
+		(end 115.060978 105.008123)
 		(width 0.2)
 		(layer "F.Cu")
@@
 	)
 	(segment
-		(start 115.745978 105.693123)
+		(start 115.060978 105.008123)
 		(end 123.220978 113.168123)
 		(width 0.2)
@@
 	)
 	(segment
-		(start 109.320978 105.693123)
-		(end 115.745978 105.693123)
+		(start 108.330978 105.333123)
+		(end 108.655978 105.008123)
 		(width 0.2)
 		(layer "F.Cu")
@@
 	(segment
 		(start 108.330978 106.683123)
-		(end 109.320978 105.693123)
+		(end 108.330978 105.333123)
 		(width 0.2)
 		(layer "F.Cu")
@@
 	)
 	(segment
-		(start 166.070978 110.223123)
-		(end 167.490978 110.223123)
+		(start 168.290978 108.508123)
+		(end 168.290978 105.728123)
 		(width 0.2)
 		(layer "F.Cu")
@@
 	)
 	(segment
-		(start 168.280978 106.608123)
-		(end 166.005978 104.333123)
+		(start 168.290978 105.728123)
+		(end 166.230978 103.668123)
 		(width 0.2)
 		(layer "F.Cu")
@@
 	)
 	(segment
-		(start 166.005978 104.333123)
-		(end 157.530978 104.333123)
+		(start 166.080978 109.233123)
+		(end 167.565978 109.233123)
 		(width 0.2)
 		(layer "F.Cu")
@@
 	)
 	(segment
-		(start 168.280978 109.433123)
-		(end 168.280978 106.608123)
+		(start 158.200978 103.668123)
+		(end 148.690978 113.178123)
 		(width 0.2)
 		(layer "F.Cu")
@@
 	)
 	(segment
-		(start 157.530978 104.333123)
-		(end 148.680978 113.183123)
+		(start 166.230978 103.668123)
+		(end 158.200978 103.668123)
 		(width 0.2)
 		(layer "F.Cu")
@@
 	)
 	(segment
-		(start 167.490978 110.223123)
-		(end 168.280978 109.433123)
-		(width 0.2)
-		(layer "F.Cu")
+		(start 167.565978 109.233123)
+		(end 168.290978 108.508123)
+		(width 0.2)
+		(layer "F.Cu")

Commit message: headers
Routing:
- net +5V FILT: track 65.4 -> 66.6 mm
- net /FR IN 1: track 19.0 -> 19.8 mm
Changed lines of the file:
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@@
 		(start 108.180978 103.658123)
 		(end 116.210978 103.658123)
-		(width 0.2)
+		(width 0.254)
 		(layer "F.Cu")
 		(net 2)
@@
 		(start 116.210978 103.658123)
 		(end 125.720978 113.168123)
-		(width 0.2)
+		(width 0.254)
 		(layer "F.Cu")
 		(net 2)
@@
 		(start 106.120978 105.718123)
 		(end 108.180978 103.658123)
-		(width 0.2)
+		(width 0.254)
 		(layer "F.Cu")
 		(net 2)
@@
 		(start 108.330978 109.223123)
 		(end 106.845978 109.223123)
-		(width 0.2)
+		(width 0.254)
 		(layer "F.Cu")
 		(net 2)
@@
 		(start 106.845978 109.223123)
 		(end 106.120978 108.498123)
-		(width 0.2)
+		(width 0.254)
 		(layer "F.Cu")
 		(net 2)
@@
 		(start 106.120978 108.498123)
 		(end 106.120978 105.718123)
-		(width 0.2)
-		(layer "F.Cu")
-		(net 2)
-	)
-	(segment
-		(start 166.080978 105.258123)
+		(width 0.254)
+		(layer "F.Cu")
+		(net 2)
+	)
+	(segment
+		(start 166.070978 105.248123)
 		(end 165.840978 105.018123)
-		(width 0.2)
+		(width 0.254)
+		(layer "F.Cu")
+		(net 3)
+	)
+	(segment
+		(start 165.840978 105.018123)
+		(end 159.350978 105.018123)
+		(width 0.254)
+		(layer "F.Cu")
+		(net 3)
+	)
+	(segment
+		(start 166.070978 106.683123)
+		(end 166.070978 105.248123)
+		(width 0.254)
 		(layer "F.Cu")
 		(net 3)
@@
 		(start 159.350978 105.018123)
 		(end 151.190978 113.178123)
-		(width 0.2)
-		(layer "F.Cu")
-		(net 3)
-	)
-	(segment
-		(start 166.080978 105.868123)
-		(end 166.080978 105.258123)
-		(width 0.2)
-		(layer "F.Cu")
-		(net 3)
-	)
-	(segment
-		(start 165.840978 105.018123)
-		(end 159.350978 105.018123)
-		(width 0.2)
+		(width 0.254)
 		(layer "F.Cu")
 		(net 3)
@@
 		(start 110.880978 109.233123)
 		(end 114.285978 109.233123)
-		(width 0.2)
+		(width 0.254)
 		(layer "F.Cu")
 		(net 4)
@@
 		(start 114.285978 109.233123)
 		(end 118.220978 113.168123)
-		(width 0.2)
+		(width 0.254)
 		(layer "F.Cu")
 		(net 4)
@@
 		(start 160.175978 106.693123)
 		(end 153.690978 113.178123)
-		(width 0.2)
+		(width 0.254)
 		(layer "F.Cu")
 		(net 5)
@@
 		(start 163.540978 106.693123)
 		(end 160.175978 106.693123)
-		(width 0.2)
+		(width 0.254)
 		(layer "F.Cu")
 		(net 5)
@@
 		(start 114.235978 106.683123)
 		(end 120.720978 113.168123)
-		(width 0.2)
+		(width 0.254)
 		(layer "F.Cu")
 		(net 6)
@@
 		(start 110.870978 106.683123)
 		(end 114.235978 106.683123)
-		(width 0.2)
+		(width 0.254)
 		(layer "F.Cu")
 		(net 6)
@@
 		(start 163.530978 109.243123)
 		(end 160.125978 109.243123)
-		(width 0.2)
+		(width 0.254)
 		(layer "F.Cu")
 		(net 7)
@@
 		(start 160.125978 109.243123)
 		(end 156.190978 113.178123)
-		(width 0.2)
+		(width 0.254)
 		(layer "F.Cu")
 		(net 7)
@@
 		(start 108.655978 105.008123)
 		(end 115.060978 105.008123)
-		(width 0.2)
+		(width 0.254)
 		(layer "F.Cu")
 		(net 8)
@@
 		(start 115.060978 105.008123)
 		(end 123.220978 113.168123)
-		(width 0.2)
+		(width 0.254)
 		(layer "F.Cu")
 		(net 8)
@@
 		(start 108.330978 105.333123)
 		(end 108.655978 105.008123)
-		(width 0.2)
+		(width 0.254)
 		(layer "F.Cu")
 		(net 8)
@@
 		(start 108.330978 106.683123)
 		(end 108.330978 105.333123)
-		(width 0.2)
+		(width 0.254)
 		(layer "F.Cu")
 		(net 8)
@@
 		(start 168.290978 108.508123)
 		(end 168.290978 105.728123)
-		(width 0.2)
+		(width 0.254)
 		(layer "F.Cu")
 		(net 9)
@@
 		(start 168.290978 105.728123)
 		(end 166.230978 103.668123)
-		(width 0.2)
+		(width 0.254)
 		(layer "F.Cu")
 		(net 9)
@@
 		(start 166.080978 109.233123)
 		(end 167.565978 109.233123)
-		(width 0.2)
+		(width 0.254)
 		(layer "F.Cu")
 		(net 9)
@@
 		(start 158.200978 103.668123)
 		(end 148.690978 113.178123)
-		(width 0.2)
+		(width 0.254)
 		(layer "F.Cu")
 		(net 9)
@@
 		(start 166.230978 103.668123)
 		(end 158.200978 103.668123)
-		(width 0.2)
+		(width 0.254)
 		(layer "F.Cu")
 		(net 9)
@@
 		(start 167.565978 109.233123)
 		(end 168.290978 108.508123)
-		(width 0.2)
-		(layer "F.Cu")
-		(net 9)
-	)
-	(segment
-		(start 160.885978 115.408123)
-		(end 146.605978 115.408123)
+		(width 0.254)
+		(layer "F.Cu")
+		(net 9)
+	)
+	(segment
+		(start 160.110978 115.183123)
+		(end 146.380978 115.183123)
+		(width 1)
+		(layer "B.Cu")
+		(net 10)
+	)
+	(segment
+		(start 146.380978 115.183123)
+		(end 146.180978 114.983123)
+		(width 1)
+		(layer "B.Cu")
+		(net 10)
+	)
+	(segment
+		(start 146.180978 114.983123)
+		(end 146.180978 113.183123)
+		(width 1)
+		(layer "B.Cu")
+		(net 10)
+	)
+	(segment
+		(start 142.505978 108.533123)
+		(end 146.180978 112.208123)
+		(width 1)
+		(layer "B.Cu")
+		(net 10)
+	)
+	(segment
+		(start 115.730978 113.183123)
+		(end 120.380978 108.533123)
+		(width 1)
+		(layer "B.Cu")
+		(net 10)
+	)
+	(segment
+		(start 110.870978 111.763123)
+		(end 108.330978 111.763123)
+		(width 1)
+		(layer "B.Cu")
+		(net 10)
+	)
+	(segment
+		(start 120.380978 108.533123)
+		(end 142.505978 108.533123)
+		(width 1)
+		(layer "B.Cu")
+		(net 10)
+	)
+	(segment
+		(start 112.510978 111.763123)
+		(end 110.870978 111.763123)
+		(width 1)
+		(layer "B.Cu")
+		(net 10)
+	)
+	(segment
+		(start 166.070978 111.763123)
+		(end 163.530978 111.763123)
+		(width 1)
+		(layer "B.Cu")
+		(net 10)
+	)
+	(segment
+		(start 115.310978 112.763123)
+		(end 115.730978 113.183123)
 		(width 1)
 		(layer "B.Cu")
@@
 	)
 	(segment
-		(start 120.380978 108.533123)
-		(end 142.505978 108.533123)
-		(width 1)
-		(layer "B.Cu")
-		(net 10)
-	)
-	(segment
-		(start 108.330978 112.763123)
-		(end 110.870978 112.763123)
-		(width 1)
-		(layer "B.Cu")
-		(net 10)
-	)
-	(segment
-		(start 166.070978 112.763123)
-		(end 163.530978 112.763123)
-		(width 1)
-		(layer "B.Cu")
-		(net 10)
-	)
-	(segment
-		(start 110.870978 112.763123)
-		(end 115.310978 112.763123)
+		(start 113.930978 113.183123)
+		(end 112.510978 111.763123)
 		(width 1)
 		(layer "B.Cu")
@@
 	(segment
 		(start 115.730978 113.183123)
-		(end 120.380978 108.533123)
-		(width 1)
-		(layer "B.Cu")
-		(net 10)
-	)
-	(segment
-		(start 163.530978 112.763123)
-		(end 160.885978 115.408123)
-		(width 1)
-		(layer "B.Cu")
-		(net 10)
-	)
-	(segment
-		(start 115.310978 112.763123)
-		(end 115.730978 113.183123)
-		(width 1)
-		(layer "B.Cu")
-		(net 10)
-	)
-	(segment
-		(start 146.605978 115.408123)
-		(end 146.180978 114.983123)
-		(width 1)
-		(layer "B.Cu")
-		(net 10)
-	)
-	(segment
-		(start 142.505978 108.533123)
-		(end 146.180978 112.208123)
-		(width 1)
-		(layer "B.Cu")
-		(net 10)
-	)
-	(segment
-		(start 146.180978 114.983123)
-		(end 146.180978 113.183123)
-		(width 1)
-		(layer "B.Cu")
+		(end 113.930978 113.183123)
+		(width 1)
+		(layer "B.Cu")
+		(net 10)
+	)
+	(segment
+		(start 163.530978 111.763123)
+		(end 160.110978 115.183123)
+		(width 1)
+		(layer "B.Cu")
