File: mdriver/topInterface/topInterface.kicad_sch (KiCad schematic)
At the start: 4 parts

Commit message: mdriver
Parts:
- removed J?: Conn_01x10, symbol Connector_Generic:Conn_01x10
- added H1, H2, H3, H4: MountingHole, MountingHole:MountingHole_3.2mm_M3_Pad, symbol Mechanical:MountingHole
- added J4, J5: Conn_01x06, Connector_JST:JST_XH_B6B-XH-A_1x06_P2.50mm_Vertical, symbol Connector_Generic:Conn_01x06
- J1, J2: renamed from J?; footprint (none) -> Connector_PinSocket_2.54mm:PinSocket_2x04_P2.54mm_Vertical
- J3: renamed from J?; footprint (none) -> Library:xt30-f
Connections:
- net +3V3: now also J4.1 (Pin_1), J5.1 (Pin_1)
- net BL IN 1: now also J4.4 (Pin_4)
- net BL IN 2: now also J4.5 (Pin_5)
- net BR IN 1: now also J5.4 (Pin_4)
- net BR IN 2: now also J5.5 (Pin_5)
- net FL IN 1: now also J4.2 (Pin_2)
- net FL IN 2: now also J4.3 (Pin_3)
- net FR IN 1: now also J5.2 (Pin_2)
- net FR IN 2: now also J5.3 (Pin_3)
- net GNDREF: now also J4.6 (Pin_6), J5.6 (Pin_6)

Commit message: driver
Parts:
- removed J3: Conn_01x02, Library:xt30-f, symbol Connector_Generic:Conn_01x02
- renumbered J4 to J3, J5 to J4
Changed lines of the file:
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@@
-	(wire
-		(pts
-			(xy 44.45 74.93) (xy 44.45 77.47)
-		)
-		(stroke
-			(width 0)
-			(type default)
-		)
-	)
-	(wire
-		(pts
-			(xy 41.91 77.47) (xy 44.45 77.47)
-		)
-		(stroke
-			(width 0)
-			(type default)
-		)
-	)
 	(wire
 		(pts
@@
 	(wire
 		(pts
-			(xy 44.45 80.01) (xy 44.45 82.55)
-		)
-		(stroke
-			(width 0)
-			(type default)
-		)
-	)
-	(wire
-		(pts
 			(xy 86.36 96.52) (xy 88.9 96.52)
 		)
@@
 		(pts
 			(xy 35.56 46.99) (xy 38.1 46.99)
-		)
-		(stroke
-			(width 0)
-			(type default)
-		)
-	)
-	(wire
-		(pts
-			(xy 41.91 80.01) (xy 44.45 80.01)
 		)
 		(stroke
@@
 		(dnp no)
 		(fields_autoplaced yes)
-		(property "Reference" "J5"
+		(property "Reference" "J4"
 			(at 81.28 90.17 0)
 			(effects
@@
 			(project ""
 				(path "/dccdf601-29e8-4aa2-b806-b24390443d4f"
-					(reference "J5")
-					(unit 1)
-				)
-			)
-		)
-	)
-	(symbol
-		(lib_id "power:+12V")
-		(at 44.45 74.93 0)
-		(unit 1)
-		(exclude_from_sim no)
-		(in_bom yes)
-		(on_board yes)
-		(dnp no)
-		(fields_autoplaced yes)
-		(property "Reference" "#PWR03"
-			(at 44.45 78.74 0)
-			(effects
-				(font
-					(size 1.27 1.27)
-				)
-				(hide yes)
-			)
-		)
-		(property "Value" "+12V"
-			(at 44.45 69.85 0)
-			(effects
-				(font
-					(size 1.27 1.27)
-				)
-			)
-		)
-		(property "Footprint" ""
-			(at 44.45 74.93 0)
-			(effects
-				(font
-					(size 1.27 1.27)
-				)
-				(hide yes)
-			)
-		)
-		(property "Datasheet" ""
-			(at 44.45 74.93 0)
-			(effects
-				(font
-					(size 1.27 1.27)
-				)
-				(hide yes)
-			)
-		)
-		(property "Description" "Power symbol creates a global label with name \"+12V\""
-			(at 44.45 74.93 0)
-			(effects
-				(font
-					(size 1.27 1.27)
-				)
-				(hide yes)
-			)
-		)
-		(pin "1"
-		)
-		(instances
-			(project ""
-				(path "/dccdf601-29e8-4aa2-b806-b24390443d4f"
-					(reference "#PWR03")
+					(reference "J4")
 					(unit 1)
 				)
@@
 		(dnp no)
 		(fields_autoplaced yes)
-		(property "Reference" "J4"
+		(property "Reference" "J3"
 			(at 110.49 78.74 0)
 			(effects
@@
 			(project ""
 				(path "/dccdf601-29e8-4aa2-b806-b24390443d4f"
-					(reference "J4")
+					(reference "J3")
 					(unit 1)
 				)
@@
 					(unit 1)
 				)
-			)
-		)
-	)
-	(symbol
-		(lib_id "Connector_Generic:Conn_01x02")
-		(at 36.83 77.47 0)
-		(mirror y)
-		(unit 1)
-		(exclude_from_sim no)
-		(in_bom yes)
-		(on_board yes)
-		(dnp no)
-		(fields_autoplaced yes)
-		(property "Reference" "J3"
-			(at 36.83 71.12 0)
-			(effects
-				(font
-					(size 1.27 1.27)
-				)
-			)
-		)
-		(property "Value" "Conn_01x02"
-			(at 36.83 73.66 0)
-			(effects
-				(font
-					(size 1.27 1.27)
-				)
-			)
-		)
-		(property "Footprint" "Library:xt30-f"
-			(at 36.83 77.47 0)
-			(effects
-				(font
-					(size 1.27 1.27)
-				)
-				(hide yes)
-			)
-		)
-		(property "Datasheet" "~"
-			(at 36.83 77.47 0)
-			(effects
-				(font
-					(size 1.27 1.27)
-				)
-				(hide yes)
-			)
-		)
-		(property "Description" "Generic connector, single row, 01x02, script generated (kicad-library-utils/schlib/autogen/connector/)"
-			(at 36.83 77.47 0)
-			(effects
-				(font
-					(size 1.27 1.27)
-				)
-				(hide yes)
-			)
-		)
-		(pin "1"
-		)
-		(pin "2"
-		)
-		(instances
-			(project ""
-				(path "/dccdf601-29e8-4aa2-b806-b24390443d4f"
-					(reference "J3")
-					(unit 1)
-				)
-			)
-		)
-	)
-	(symbol
-		(lib_id "power:GNDREF")
-		(at 44.45 82.55 0)
-		(unit 1)
-		(exclude_from_sim no)
-		(in_bom yes)
-		(on_board yes)
-		(dnp no)
-		(fields_autoplaced yes)
-		(property "Reference" "#PWR04"
-			(at 44.45 88.9 0)
-			(effects
-				(font
-					(size 1.27 1.27)
-				)
-				(hide yes)
-			)
-		)
-		(property "Value" "GNDREF"
-			(at 44.45 87.63 0)
-			(effects
-				(font
-					(size 1.27 1.27)
-				)
-				(hide yes)
-			)
-		)
-		(property "Footprint" ""
-			(at 44.45 82.55 0)
-			(effects
-				(font
-					(size 1.27 1.27)
-				)
-				(hide yes)
-			)
-		)
-		(property "Datasheet" ""
-			(at 44.45 82.55 0)
-			(effects
-				(font
-					(size 1.27 1.27)
-				)
-				(hide yes)
-			)
-		)
-		(property "Description" "Power symbol creates a global label with name \"GNDREF\" , reference supply ground"
-			(at 44.45 82.55 0)
-			(effects
-				(font
-					(size 1.27 1.27)
-				)
-				(hide yes)
-			)
-		)
-		(pin "1"
-		)
-		(instances
-			(project ""
-				(path "/dccdf601-29e8-4aa2-b806-b24390443d4f"
-					(reference "#PWR04")
-					(unit 1)
-				)

Commit message: driver
Connections:
- net +3V3: now also J1.5 (Pin_5), J1.6 (Pin_6), J2.5 (Pin_5), J2.6 (Pin_6)
- net BL IN 1: now also J1.3 (Pin_3), J4.2 (Pin_2); no longer J2.3 (Pin_3), J3.4 (Pin_4)
- net BL IN 2: now also J1.4 (Pin_4), J4.3 (Pin_3); no longer J2.4 (Pin_4), J3.5 (Pin_5)
- net BR IN 1: now also J2.3 (Pin_3), J3.4 (Pin_4); no longer J2.6 (Pin_6), J4.4 (Pin_4)
- net BR IN 2: now also J2.4 (Pin_4), J3.5 (Pin_5); no longer J2.5 (Pin_5), J4.5 (Pin_5)
- net FL IN 1: now also J1.1 (Pin_1), J4.4 (Pin_4); no longer J2.1 (Pin_1), J3.2 (Pin_2)
- net FL IN 2: now also J1.2 (Pin_2), J4.5 (Pin_5); no longer J2.2 (Pin_2), J3.3 (Pin_3)
- net FR IN 1: now also J2.1 (Pin_1), J3.2 (Pin_2); no longer J2.8 (Pin_8), J4.2 (Pin_2)
- net FR IN 2: now also J2.2 (Pin_2), J3.3 (Pin_3); no longer J2.7 (Pin_7), J4.3 (Pin_3)
- net GNDREF: now also J2.7 (Pin_7), J2.8 (Pin_8); no longer J1.5 (Pin_5), J1.6 (Pin_6)
- removed net +12V: J1.1 (Pin_1), J1.2 (Pin_2), J1.3 (Pin_3), J1.4 (Pin_4)
Other:
- moved on the sheet: J1, J2

Commit message: Motor Driver
Connections:
- net +3V3: no longer J1.5 (Pin_5), J1.6 (Pin_6), J2.5 (Pin_5), J2.6 (Pin_6)
- net BL IN 1: now also J2.4 (Pin_4); no longer J1.3 (Pin_3)
- net BL IN 2: now also J2.2 (Pin_2); no longer J1.4 (Pin_4)
- net BR IN 1: now also J2.1 (Pin_1); no longer J2.3 (Pin_3)
- net BR IN 2: now also J2.3 (Pin_3); no longer J2.4 (Pin_4)
- net FL IN 1: now also J1.4 (Pin_4); no longer J1.1 (Pin_1)
- net FR IN 1: now also J1.1 (Pin_1); no longer J2.1 (Pin_1)
- net FR IN 2: now also J1.3 (Pin_3); no longer J2.2 (Pin_2)
- new net +5V FILT: J1.5 (Pin_5), J1.6 (Pin_6), J2.5 (Pin_5), J2.6 (Pin_6)

Commit message: top interface
Connections:
- net +3V3 is gone; now on net +5V FILT: J3.1 (Pin_1), J4.1 (Pin_1)
- net BL IN 1: now also J4.5 (Pin_5); no longer J4.2 (Pin_2)
- net BL IN 2: now also J4.4 (Pin_4); no longer J4.3 (Pin_3)
- net BR IN 1: now also J4.3 (Pin_3); no longer J3.4 (Pin_4)
- net BR IN 2: now also J4.2 (Pin_2); no longer J3.5 (Pin_5)
- net FL IN 1: now also J3.5 (Pin_5); no longer J4.4 (Pin_4)
- net FL IN 2: now also J3.4 (Pin_4); no longer J4.5 (Pin_5)
- net FR IN 1: now also J3.3 (Pin_3); no longer J3.2 (Pin_2)
- net FR IN 2: now also J3.2 (Pin_2); no longer J3.3 (Pin_3)
