File: mdriver/motorDriver/motorDriver.kicad_pcb (KiCad board)
At the start: 2 copper layers, 79.4 x 31 mm, 22 parts, among them IC1 TB67H450FNG,EL, IC2 TB67H450FNG,EL, IC3 TB67H450FNG,EL, IC4 TB67H450FNG,EL, J1 Conn_02x04_Counter_Clockwise, J2 Conn_02x04_Counter_Clockwise, J3 FL, J4 FR, J5 BL, J6 BR

Commit message: driver
Parts:
- added J7: Conn_01x02, Library:xt30-f, F.Cu at (137.2, 113.9)
Connections:
- J1 pad 1: +12V -> unconnected-(J1-Pin_1-Pad1)
- J1 pad 2: +12V -> unconnected-(J1-Pin_2-Pad2)
- J1 pad 3: +12V -> unconnected-(J1-Pin_3-Pad3)
- J1 pad 4: +12V -> unconnected-(J1-Pin_4-Pad4)
Other:
- board text removed: "SEN LOGO"

Commit message: Motor Driver
Parts:
- J1: value Conn_02x04_Counter_Clockwise -> Power
- J2: value Conn_02x04_Counter_Clockwise -> Signal
- moved J1 55.2 mm to (166.1, 107.7)
- moved J2 55.2 mm to (110.9, 107.7)
- moved C3 3.80 mm to (147.0, 92.4)
- moved C7 3.80 mm to (115.0, 92.4)
- moved C8 3.80 mm to (123.5, 92.4)
- moved C4 3.80 mm to (155.6, 92.4)
Connections:
- J1 pad 1: unconnected-(J1-Pin_1-Pad1) -> FR IN 1
- J1 pad 2: unconnected-(J1-Pin_2-Pad2) -> FL IN 2
- J1 pad 3: unconnected-(J1-Pin_3-Pad3) -> FR IN 2
- J1 pad 4: unconnected-(J1-Pin_4-Pad4) -> FL IN 1
- J1 pad 5: GNDREF -> +5V FILT
- J1 pad 6: GNDREF -> +5V FILT
- J2 pad 1: FL IN 1 -> BR IN 1
- J2 pad 2: FL IN 2 -> BL IN 2
- J2 pad 3: BL IN 1 -> BR IN 2
- J2 pad 4: BL IN 2 -> BL IN 1
- J2 pad 5: BR IN 2 -> +5V FILT
- J2 pad 6: BR IN 1 -> +5V FILT
- J2 pad 7: FR IN 2 -> GNDREF
- J2 pad 8: FR IN 1 -> GNDREF
Routing:
- net +5V FILT: track 0.00 -> 78.0 mm, vias 0 -> 4
- net BR IN 2: track 1.76 -> 27.2 mm
- net FL IN 1: track 1.76 -> 26.6 mm
- net BR IN 1: track 1.76 -> 23.7 mm
- net BL IN 1: track 1.76 -> 23.4 mm
- net FR IN 2: track 1.76 -> 22.9 mm
- net FL IN 2: track 1.76 -> 22.5 mm
- net BL IN 2: track 1.76 -> 19.6 mm
- net FR IN 1: track 1.76 -> 18.5 mm
- net +12V: vias 0 -> 8
- added copper zone on B.Cu, net +12V
- added copper zone on F.Cu, net +12V
- added copper zone on B.Cu, net +5V FILT
- added copper zone on F.Cu, net /BL OUT 1
- added copper zone on F.Cu, net /BL OUT 2
- added copper zone on F.Cu, net /BR OUT 1
- added copper zone on F.Cu, net /BR OUT 2
- added copper zone on F.Cu, net /FL OUT 1
- added copper zone on F.Cu, net /FL OUT 2
- added copper zone on F.Cu, net /FR OUT 1
- added copper zone on F.Cu, net /FR OUT 2
- added copper zone on B.Cu, net GNDREF
- added copper zone on F.Cu, net GNDREF

Commit message: Minor Change to Mdriver
Routing:
- net +5V FILT: track 78.0 -> 112.2 mm, vias 4 -> 0
- net +12V: vias 8 -> 4
- removed copper zone on B.Cu, net +5V FILT

Commit message: buck
Changed lines of the file:
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@@
 			(at 0 -3.5 180)
 			(layer "F.SilkS")
+			(hide yes)
 			(effects
 				(font
@@
 		(fp_arc
 			(start 4 2.487868)
-			(mid 3.912132 2.699998)
+			(mid 3.912133 2.700001)
 			(end 3.7 2.787867)
 			(stroke
@@
 		(fp_arc
 			(start 4 2.487868)
-			(mid 3.912132 2.699998)
+			(mid 3.912133 2.700001)
 			(end 3.7 2.787867)
 			(stroke
@@
 		(fp_arc
 			(start 4 2.487868)
-			(mid 3.912133 2.700001)
+			(mid 3.912132 2.699998)
 			(end 3.7 2.787867)
 			(stroke
@@
 		(fp_arc
 			(start 4 2.487868)
-			(mid 3.912132 2.699998)
+			(mid 3.912133 2.700001)
 			(end 3.7 2.787867)
 			(stroke
