File: mdriver/motorDriver/motorDriver.kicad_pcb (KiCad board)
At the start: 2 copper layers, 79.4 x 31 mm, 23 parts, among them IC1 TB67H450FNG,EL, IC2 TB67H450FNG,EL, IC3 TB67H450FNG,EL, IC4 TB67H450FNG,EL, J1 Power, J2 Signal, J3 FL, J4 FR, J5 BL, J6 BR, J7 Conn_01x02

Commit message: Headers
Parts:
- moved J1 1.00 mm to (166.1, 106.7)
- moved J2 1.00 mm to (110.9, 106.7)
Routing:
- net FL IN 1: track 26.6 -> 23.3 mm
- net BL IN 1: track 23.4 -> 21.1 mm
- net BL IN 2: track 19.6 -> 17.5 mm
- net FL IN 2: track 22.5 -> 20.9 mm
- net BR IN 2: track 27.2 -> 25.9 mm
- net FR IN 2: track 22.9 -> 21.6 mm
- net FR IN 1: track 18.5 -> 17.6 mm
- net BR IN 1: track 23.7 -> 23.1 mm
