File: supplyUnit/buckUnit/buckUnit.kicad_pcb (KiCad board)
At the start: 2 copper layers, 79.4 x 31 mm, 2 parts, among them J1 Conn_02x03_Counter_Clockwise, J2 Conn_02x03_Counter_Clockwise

Commit message: Buck
Parts:
- removed J1: Conn_02x03_Counter_Clockwise, Connector_PinSocket_2.54mm:PinSocket_2x03_P2.54mm_Vertical
- added C1: 10n, Buck:cap0603, F.Cu at (155.5, 104.9)
- added C2: 220u, Buck:EIA-7343-D, F.Cu at (150.7, 111.7)
- added C3: 0u1, Buck:cap0603, F.Cu at (157.3, 110.9)
- added C4: 10u, Buck:cap0603, F.Cu at (159.7, 100.1)
- added C5: 10n, Buck:cap0603, F.Cu at (120.6, 104.9)
- added C6: 220u, Buck:EIA-7343-D, F.Cu at (115.8, 111.7)
- added C7: 0u1, Buck:cap0603, F.Cu at (122.4, 111.0)
- added C8: 10u, Buck:cap0603, F.Cu at (124.8, 100.1)
- added D1: SS54, Buck:SMA (DO-214AC), F.Cu at (149.3, 98.7)
- added D2: SS54, Buck:SMA (DO-214AC), F.Cu at (114.4, 98.7)
- added J3: Conn_02x03_Counter_Clockwise, Connector_PinSocket_2.54mm:PinSocket_2x03_P2.54mm_Vertical, F.Cu at (158.3, 94.4)
- added L1: 15uH, Buck:0630 One Piece Inductor, F.Cu at (150.1, 104.8)
- added L2: 15uH, Buck:0630 One Piece Inductor, F.Cu at (115.2, 104.9)
- added R1: 10K, Buck:res0603, F.Cu at (159.3, 110.9)
- added R2: 5K9, Buck:res0603, F.Cu at (161.4, 110.9)
- added R3: 10K, Buck:res0603, F.Cu at (124.4, 111.0)
- added R4: 3K24, Buck:res0603, F.Cu at (126.5, 111.0)
- added U1: TPS5430DDA, Buck:TI_SO-PowerPAD-8, F.Cu at (159.5, 105.0)
- added U2: TPS5430DDA, Buck:TI_SO-PowerPAD-8, F.Cu at (124.6, 105.0)
- moved J2 42.3 mm to (116.1, 91.8), turned to 90 degrees
Connections:
- J2 pad 1: /Sol -> +12V
- J2 pad 2: GND -> +12V
- J2 pad 3: GND -> +12V
- J2 pad 4: GND -> +12V
- J2 pad 5: GND -> +12V
- J2 pad 6: GND -> +12V
Routing:
- net Net-(U2-VSENSE): track 0.00 -> 4.48 mm
- net Net-(U1-VSENSE): track 0.00 -> 4.47 mm
- net Net-(U2-BOOT): track 0.00 -> 3.63 mm
- net Net-(U1-BOOT): track 0.00 -> 3.63 mm
- net +12V: vias 0 -> 2
- added copper zone on B.Cu, net +12V
- added copper zone on F.Cu, net +12V
- added copper zone on F.Cu, net +3V3
- added copper zone on F.Cu, net +5V
- added copper zone on B.Cu, net GND
- added copper zone on F.Cu, net GND
- added copper zone on F.Cu, net Net-(D1-K)
- added copper zone on F.Cu, net Net-(D2-K)

Commit message: buck
Parts:
- added H1: MountingHole, MountingHole:MountingHole_3.2mm_M3_Pad, F.Cu at (110.0, 94.6)
- added H2: MountingHole, MountingHole:MountingHole_3.2mm_M3_Pad, F.Cu at (164.3, 94.6)
- added H3: MountingHole, MountingHole:MountingHole_3.2mm_M3_Pad, F.Cu at (101.5, 112.9)
- added H4: MountingHole, MountingHole:MountingHole_3.2mm_M3_Pad, F.Cu at (172.9, 112.9)
- added J1: VBAT, Library:xt60-f, F.Cu at (137.2, 93.1)
- added J4: Conn_01x05, Connector_JST:JST_XH_B5B-XH-A_1x05_P2.50mm_Vertical, F.Cu at (132.2, 106.2)
- added J5: L1, Connector_JST:JST_XH_B2B-XH-A_1x02_P2.50mm_Vertical, F.Cu at (131.6, 113.1)
- added J6: Conn_02x03_Counter_Clockwise, Connector_PinSocket_2.54mm:PinSocket_2x03_P2.54mm_Vertical, F.Cu at (116.1, 91.8)
- added J7: Conn_02x03_Counter_Clockwise, Connector_PinSocket_2.54mm:PinSocket_2x03_P2.54mm_Vertical, F.Cu at (158.3, 94.4)
- C1, C3, C4, C5, C7, C8: footprint Buck:cap0603 -> Library:cap0603
- C2, C6: footprint Buck:EIA-7343-D -> Library:eia-7343-d
- D1, D2: footprint Buck:SMA (DO-214AC) -> Library:SMA (DO-214AC)
- J2: value Conn_02x03_Counter_Clockwise -> Motor; footprint Connector_PinSocket_2.54mm:PinSocket_2x03_P2.54mm_Vertical -> Library:xt30-f
- J3: value Conn_02x03_Counter_Clockwise -> Dribbler; footprint Connector_PinSocket_2.54mm:PinSocket_2x03_P2.54mm_Vertical -> Connector_JST:JST_XH_B2B-XH-A_1x02_P2.50mm_Vertical
- L1, L2: footprint Buck:0630 One Piece Inductor -> Library:0630 One Piece Inductor
- R1, R2, R3, R4: footprint Buck:res0603 -> Library:res0603
- U1, U2: footprint Buck:TI_SO-PowerPAD-8 -> Library:TI_SO-PowerPAD-8
- moved J3 26.0 mm to (140.2, 113.1), turned to 0 degrees
- moved J2 22.4 mm to (136.8, 100.4), turned to 0 degrees
- moved C3 2.23 mm to (158.4, 112.9)
- moved C4 2.23 mm to (160.8, 102.0)
- moved D1 2.23 mm to (150.5, 100.6)
- moved R1 2.23 mm to (160.5, 112.9)
- moved R2 2.23 mm to (162.5, 112.9)
- moved C1 2.23 mm to (156.6, 106.8)
- moved C2 2.23 mm to (151.8, 113.6)
- moved L1 2.23 mm to (151.2, 106.8)
- moved U1 2.23 mm to (160.6, 106.9)
- moved C5 2.16 mm to (119.6, 106.9)
- moved L2 2.16 mm to (114.2, 106.8)
- moved U2 2.16 mm to (123.6, 107.0)
- moved C6 2.16 mm to (114.8, 113.7)
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Connections:
- J2 pad 2: +12V -> GND
- J3 pad 1: /Sol -> +12V
Routing:
- net Net-(U2-VSENSE): track 4.48 -> 2.05 mm
- net Net-(U1-VSENSE): track 4.47 -> 2.05 mm
- net +12V: vias 2 -> 0
- added copper zone on F.Cu, net (none)
- added copper zone on B.Cu, net GNDREF
- added copper zone on F.Cu, net GNDREF
- removed copper zone on B.Cu, net +12V
- removed copper zone on F.Cu, net +12V
- removed copper zone on F.Cu, net +3V3
- removed copper zone on F.Cu, net +5V
- removed copper zone on B.Cu, net GND
- removed copper zone on F.Cu, net GND
- removed copper zone on F.Cu, net Net-(D1-K)
- removed copper zone on F.Cu, net Net-(D2-K)
Other:
- rule pad_to_mask_clearance: 0 -> 0.2

Commit message: okl
Parts:
- removed C1, C5: 10n, Library:cap0603
- removed C2, C6: 220u, Library:eia-7343-d
- removed C3, C7: 0u1, Library:cap0603
- removed C4, C8: 10u, Library:cap0603
- removed D1, D2: SS54, Library:SMA (DO-214AC)
- removed L1, L2: 15uH, Library:0630 One Piece Inductor
- removed R1, R3: 10K, Library:res0603
- removed R2: 5K9, Library:res0603
- removed R4: 3K24, Library:res0603
- U1, U2: value TPS5430DDA -> OKL-T6-W12-C; footprint Library:TI_SO-PowerPAD-8 -> Library:MURATA_OKL-T-6-W12
- moved U2 5.44 mm to (118.2, 107.4), turned to 0 degrees
- moved U1 4.45 mm to (156.2, 107.4), turned to 180 degrees
Connections:
- J4 pad 4: GNDREF -> GND
- J4 pad 5: GNDREF -> GND
- U1 pad 1: Net-(U1-BOOT) -> unconnected-(U1-ON/OFF-Pad1)
- U1 pad 2: unconnected-(U1-NC-Pad2) -> +12V
- U1 pad 3: unconnected-(U1-NC-Pad3) -> GND
- U1 pad 4: Net-(U1-VSENSE) -> +3V3
- U1 pad 5: unconnected-(U1-EN-Pad5) -> +3V3
- U1 pad 6: GND -> Net-(U1-TRIM)
- U1 pad 7: +12V -> GND
- U1 pad 8: Net-(D1-K) -> unconnected-(U1-Pad8)
- U1 pad 9: GND -> (no net)
- U2 pad 1: Net-(U2-BOOT) -> unconnected-(U2-ON/OFF-Pad1)
- U2 pad 2: unconnected-(U2-NC-Pad2) -> +12V
- U2 pad 3: unconnected-(U2-NC-Pad3) -> GND
- U2 pad 4: Net-(U2-VSENSE) -> +5V
- U2 pad 5: unconnected-(U2-EN-Pad5) -> +5V
- U2 pad 6: GND -> Net-(U2-TRIM)
- U2 pad 7: +12V -> GND
- U2 pad 8: Net-(D2-K) -> unconnected-(U2-Pad8)
- U2 pad 9: GND -> (no net)
Routing:
- net Net-(U2-BOOT): track 3.63 -> 0.00 mm
- net Net-(U1-BOOT): track 3.63 -> 0.00 mm
- net Net-(U1-VSENSE): track 2.05 -> 0.00 mm
- net Net-(U2-VSENSE): track 2.05 -> 0.00 mm
- added copper zone on B.Cu, net GND
- added copper zone on F.Cu, net GND
- removed copper zone on B.Cu, net GNDREF
- removed copper zone on F.Cu, net GNDREF

Commit message: okl
Parts:
- added C1: 10u, Library:cap0603, B.Cu at (113.7, 104.8)
- added C2: 10u, Library:cap0603, B.Cu at (157.7, 104.8)
- added R1: 1K, Library:res0603, B.Cu at (161.5, 110.7)
- added R2: 1K, Library:res0603, B.Cu at (117.5, 110.7)
- added R3: 1K, Library:res0603, B.Cu at (159.2, 110.7)
- added R4: 330, Library:res0603, B.Cu at (115.2, 110.7)
- added R5: 180, Library:res0603, B.Cu at (156.9, 110.7)
- added R6: 10, Library:res0603, B.Cu at (112.9, 110.7)
- moved J5 17.7 mm to (149.1, 110.1), turned to -90 degrees
- moved J3 14.2 mm to (126.3, 110.1), turned to -90 degrees
- moved J4 5.48 mm to (132.2, 111.7)
- moved U1 3.16 mm to (159.2, 108.4), turned to 0 degrees
- moved U2 3.16 mm to (115.2, 108.4)
Routing:
- net Net-(U2-TRIM): track 0.00 -> 4.43 mm
- net Net-(U1-TRIM): track 0.00 -> 4.43 mm
- net Net-(R3-Pad2): track 0.00 -> 2.29 mm
- net Net-(R2-Pad2): track 0.00 -> 2.29 mm
- net Net-(R4-Pad2): track 0.00 -> 2.29 mm
- net Net-(R1-Pad2): track 0.00 -> 2.29 mm
