File: motorDriver/motorDriver.kicad_pcb (KiCad board)
At the start: 2 copper layers, 72.7 x 33.9 mm, 23 parts, among them IC1 TB67H450FNG,EL, IC2 TB67H450FNG,EL, IC3 TB67H450FNG,EL, IC4 TB67H450FNG,EL, J1 Conn_01x12, J3 FL, J4 FR, J5 BL, J6 BR, J7 Conn_01x02

Commit message: 死
Parts:
- removed ?: , 
- J1: value Conn_01x12 -> Conn_01x10; footprint Library:526101271 -> Library:526101071
Connections:
- J1 pad 10: FR IN 1 -> GNDREF
- J1 pad 2: +5V FILT -> BL IN 2
- J1 pad 3: BL IN 2 -> BL IN 1
- J1 pad 4: BL IN 1 -> BR IN 1
- J1 pad 5: BR IN 1 -> BR IN 2
- J1 pad 6: BR IN 2 -> FL IN 1
- J1 pad 7: FL IN 1 -> FL IN 2
- J1 pad 8: FL IN 2 -> FR IN 2
- J1 pad 9: FR IN 2 -> FR IN 1
Routing:
- net GNDREF: vias 54 -> 4
Other:
- board text added: "温"
- board text added: "表"
- board text added: "雨子"
- board text added: "面"
- board text added: "高"
