File: motorDriver/motorDriver.kicad_pcb (KiCad board)
At the start: 2 copper layers, 72.7 x 33.9 mm, 22 parts, among them IC1 TB67H450FNG,EL, IC2 TB67H450FNG,EL, IC3 TB67H450FNG,EL, IC4 TB67H450FNG,EL, J1 Conn_01x10, J3 FL, J4 FR, J5 BL, J6 BR, J7 Conn_01x02

Commit message: mdriver
Parts:
- moved J3 1.00 mm to (149.9, 113.7)
- moved J4 1.00 mm to (158.4, 113.7)
- moved J5 1.00 mm to (113.4, 113.7)
- moved J6 1.00 mm to (122.0, 113.7)

Commit message: 死
Parts:
- moved J3 1.00 mm to (148.9, 113.7)
- moved J4 0.95 mm to (157.5, 113.7)
- moved J5 0.95 mm to (114.4, 113.7)
- moved J6 0.95 mm to (122.9, 113.7)
Other:
- board text added: "JLCJLCJLCJLC"
