File: encoder/encoder.kicad_pcb (KiCad board)
At the start: 2 copper layers, 21.6 x 21.6 mm, 6 parts, among them J1 Conn_01x04

Commit message: 死
Parts:
- removed REF** (x2): IGN22, Library:IGN22
- added C2: 0u1, Library:cap0603, F.Cu at (142.7, 94.8)
- added C3: 4U7, Library:cap0603, F.Cu at (142.7, 97.9)
- added R1: 4K7, Library:res0603, F.Cu at (142.7, 101.0)
- added R2: 4K7, Library:res0603, F.Cu at (142.7, 104.1)
- C1: value 0u1 -> 4U7
- moved U1 3.09 mm to (165.6, 96.6), turned to 90 degrees
Connections:
- C1 pad 1: +3V3 -> /OUTA
Routing:
- net /OUTA: track 23.8 -> 9.84 mm
- net +3V3: track 23.1 -> 12.8 mm
- net /OUTB: track 19.8 -> 9.52 mm
- net GNDREF: track 12.5 -> 8.93 mm
