File: encoder/encoder.kicad_sch (KiCad schematic)
At the start: 4 parts, among them J1 Conn_01x04

Commit message: 死
Parts:
- added C1, C3: 4U7, Library:cap0603, symbol Device:C
- added R1, R2: 4K7, Library:res0603, symbol Device:R
- renumbered C1 to C2
Connections:
- net GNDREF: now also C1.2, C3.2, R1.2, R2.2
- net OUTA: now also C1.1, R1.1
- net OUTB: now also C3.1, R2.1
Other:
- moved on the sheet: C2, J1, U2
