File: processingUnit/stm32f4.kicad_sch (KiCad schematic)
At the start: 23 parts, among them J309 Conn_01x04, SW303 SW_Push, U303 STM32F446RET, U304 16MHz, Y301 32.768 kHz

Commit message: yes
Parts:
- renumbered C334 to C301, C335 to C302, C336 to C303, C337 to C304, C338 to C305, C333 to C306, C326 to C307, C327 to C308, C328 to C309, C329 to C310, C330 to C311, C331 to C312, C332 to C313, D306 to D301, D304 to D302, D305 to D303, J309 to J301, R314 to R301, R313 to R302, SW303 to SW301, U303 to U301, U304 to U302
Changed lines of the file:
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@@
 		(dnp no)
 		(fields_autoplaced yes)
-		(property "Reference" "#PWR0352"
+		(property "Reference" "#PWR0307"
 			(at 21.59 182.88 0)
 			(effects
@@
 			(project "l3"
 				(path "/1b1408da-cc6a-469f-a506-e797247b3ac8/9673eddf-80ee-4908-b21e-80531a02ef2e"
-					(reference "#PWR0352")
+					(reference "#PWR0307")
 					(unit 1)
 				)
@@
 		(dnp no)
 		(fields_autoplaced yes)
-		(property "Reference" "U303"
+		(property "Reference" "U301"
 			(at 99.06 138.43 0)
 			(effects
@@
 			(project "l3"
 				(path "/1b1408da-cc6a-469f-a506-e797247b3ac8/9673eddf-80ee-4908-b21e-80531a02ef2e"
-					(reference "U303")
+					(reference "U301")
 					(unit 1)
 				)
@@
 		(dnp no)
 		(fields_autoplaced yes)
-		(property "Reference" "#PWR0353"
+		(property "Reference" "#PWR0305"
 			(at 119.38 172.72 0)
 			(effects
@@
 			(project "l3"
 				(path "/1b1408da-cc6a-469f-a506-e797247b3ac8/9673eddf-80ee-4908-b21e-80531a02ef2e"
-					(reference "#PWR0353")
+					(reference "#PWR0305")
 					(unit 1)
 				)
@@
 		(dnp no)
 		(fields_autoplaced yes)
-		(property "Reference" "C332"
+		(property "Reference" "C313"
 			(at 86.36 166.3699 0)
 			(effects
@@
 			(project "l3"
 				(path "/1b1408da-cc6a-469f-a506-e797247b3ac8/9673eddf-80ee-4908-b21e-80531a02ef2e"
-					(reference "C332")
+					(reference "C313")
 					(unit 1)
 				)
@@
 		(dnp no)
 		(fields_autoplaced yes)
-		(property "Reference" "C330"
+		(property "Reference" "C311"
 			(at 66.04 166.3699 0)
 			(effects
@@
 			(project "l3"
 				(path "/1b1408da-cc6a-469f-a506-e797247b3ac8/9673eddf-80ee-4908-b21e-80531a02ef2e"
-					(reference "C330")
+					(reference "C311")
 					(unit 1)
 				)
@@
 		(dnp no)
 		(fields_autoplaced yes)
-		(property "Reference" "J309"
+		(property "Reference" "J301"
 			(at 142.24 142.24 0)
 			(effects
@@
 			(project "l3"
 				(path "/1b1408da-cc6a-469f-a506-e797247b3ac8/9673eddf-80ee-4908-b21e-80531a02ef2e"
-					(reference "J309")
+					(reference "J301")
 					(unit 1)
 				)
@@
 		(dnp no)
 		(fields_autoplaced yes)
-		(property "Reference" "C338"
+		(property "Reference" "C305"
 			(at 289.56 110.4899 0)
 			(effects
@@
 			(project "l3"
 				(path "/1b1408da-cc6a-469f-a506-e797247b3ac8/9673eddf-80ee-4908-b21e-80531a02ef2e"
-					(reference "C338")
+					(reference "C305")
 					(unit 1)
 				)
@@
 		(on_board yes)
 		(dnp no)
-		(property "Reference" "C337"
+		(property "Reference" "C304"
 			(at 269.24 110.4899 0)
 			(effects
@@
 			(project "l3"
 				(path "/1b1408da-cc6a-469f-a506-e797247b3ac8/9673eddf-80ee-4908-b21e-80531a02ef2e"
-					(reference "C337")
+					(reference "C304")
 					(unit 1)
 				)
@@
 		(dnp no)
 		(fields_autoplaced yes)
-		(property "Reference" "#PWR0357"
+		(property "Reference" "#PWR0301"
 			(at 250.19 71.12 0)
 			(effects
@@
 			(project "l3"
 				(path "/1b1408da-cc6a-469f-a506-e797247b3ac8/9673eddf-80ee-4908-b21e-80531a02ef2e"
-					(reference "#PWR0357")
+					(reference "#PWR0301")
 					(unit 1)
 				)
@@
 		(on_board yes)
 		(dnp no)
-		(property "Reference" "R314"
+		(property "Reference" "R301"
 			(at 243.84 59.69 90)
 			(effects
@@
 			(project "l3"
 				(path "/1b1408da-cc6a-469f-a506-e797247b3ac8/9673eddf-80ee-4908-b21e-80531a02ef2e"
-					(reference "R314")
+					(reference "R301")
 					(unit 1)
 				)
@@
 		(on_board yes)
 		(dnp no)
-		(property "Reference" "C335"
+		(property "Reference" "C302"
 			(at 234.95 110.4899 0)
 			(effects
@@
 			(project "l3"
 				(path "/1b1408da-cc6a-469f-a506-e797247b3ac8/9673eddf-80ee-4908-b21e-80531a02ef2e"
-					(reference "C335")
+					(reference "C302")
 					(unit 1)
 				)
@@
 		(dnp no)
 		(fields_autoplaced yes)
-		(property "Reference" "C331"
+		(property "Reference" "C312"
 			(at 76.2 166.3699 0)
 			(effects
@@
 			(project "l3"
 				(path "/1b1408da-cc6a-469f-a506-e797247b3ac8/9673eddf-80ee-4908-b21e-80531a02ef2e"
-					(reference "C331")
+					(reference "C312")
 					(unit 1)
 				)
@@
 		(dnp no)
 		(fields_autoplaced yes)
-		(property "Reference" "C328"
+		(property "Reference" "C309"
 			(at 45.72 166.3699 0)
 			(effects
@@
 			(project "l3"
 				(path "/1b1408da-cc6a-469f-a506-e797247b3ac8/9673eddf-80ee-4908-b21e-80531a02ef2e"
-					(reference "C328")
+					(reference "C309")
 					(unit 1)
 				)
@@
 		(dnp no)
 		(fields_autoplaced yes)
-		(property "Reference" "C329"
+		(property "Reference" "C310"
 			(at 55.88 166.3699 0)
 			(effects
@@
 			(project "l3"
 				(path "/1b1408da-cc6a-469f-a506-e797247b3ac8/9673eddf-80ee-4908-b21e-80531a02ef2e"
-					(reference "C329")
+					(reference "C310")
 					(unit 1)
 				)
@@
 		(dnp no)
 		(fields_autoplaced yes)
-		(property "Reference" "R313"
+		(property "Reference" "R302"
 			(at 217.17 110.4899 0)
 			(effects
@@
 			(project "l3"
 				(path "/1b1408da-cc6a-469f-a506-e797247b3ac8/9673eddf-80ee-4908-b21e-80531a02ef2e"
-					(reference "R313")
+					(reference "R302")
 					(unit 1)
 				)
@@
 		(on_board yes)
 		(dnp no)
-		(property "Reference" "D306"
+		(property "Reference" "D301"
 			(at 233.68 54.61 0)
 			(effects
@@
 			(project "l3"
 				(path "/1b1408da-cc6a-469f-a506-e797247b3ac8/9673eddf-80ee-4908-b21e-80531a02ef2e"
-					(reference "D306")
+					(reference "D301")
 					(unit 1)
 				)
@@
 		(dnp no)
 		(fields_autoplaced yes)
-		(property "Reference" "SW303"
+		(property "Reference" "SW301"
 			(at 193.04 111.7599 90)
 			(effects
@@
 			(project "l3"
 				(path "/1b1408da-cc6a-469f-a506-e797247b3ac8/9673eddf-80ee-4908-b21e-80531a02ef2e"
-					(reference "SW303")
+					(reference "SW301")
 					(unit 1)
 				)
@@
 		(dnp no)
 		(fields_autoplaced yes)
-		(property "Reference" "#PWR0355"
+		(property "Reference" "#PWR0306"
 			(at 157.48 175.26 0)
 			(effects
@@
 			(project "l3"
 				(path "/1b1408da-cc6a-469f-a506-e797247b3ac8/9673eddf-80ee-4908-b21e-80531a02ef2e"
-					(reference "#PWR0355")
+					(reference "#PWR0306")
 					(unit 1)
 				)
@@
 		(dnp no)
 		(fields_autoplaced yes)
-		(property "Reference" "U303"
+		(property "Reference" "U301"
 			(at 161.29 21.59 0)
 			(effects
@@
 			(project "l3"
 				(path "/1b1408da-cc6a-469f-a506-e797247b3ac8/9673eddf-80ee-4908-b21e-80531a02ef2e"
-					(reference "U303")
+					(reference "U301")
 					(unit 2)
 				)
@@
 		(dnp no)
 		(fields_autoplaced yes)
-		(property "Reference" "C333"
+		(property "Reference" "C306"
 			(at 123.19 154.9399 0)
 			(effects
@@
 			(project "l3"
 				(path "/1b1408da-cc6a-469f-a506-e797247b3ac8/9673eddf-80ee-4908-b21e-80531a02ef2e"
-					(reference "C333")
+					(reference "C306")
 					(unit 1)
 				)
@@
 		(on_board yes)
 		(dnp no)
-		(property "Reference" "C326"
+		(property "Reference" "C307"
 			(at 25.4 166.3699 0)
 			(effects
@@
 			(project "l3"
 				(path "/1b1408da-cc6a-469f-a506-e797247b3ac8/9673eddf-80ee-4908-b21e-80531a02ef2e"
-					(reference "C326")
+					(reference "C307")
 					(unit 1)
 				)
@@
 		(dnp no)
 		(fields_autoplaced yes)
-		(property "Reference" "D304"
+		(property "Reference" "D302"
 			(at 160.02 160.0199 90)
 			(effects
@@
 			(project "l3"
 				(path "/1b1408da-cc6a-469f-a506-e797247b3ac8/9673eddf-80ee-4908-b21e-80531a02ef2e"
-					(reference "D304")
+					(reference "D302")
 					(unit 1)
 				)
@@
 		(dnp no)
 		(fields_autoplaced yes)
-		(property "Reference" "C334"
+		(property "Reference" "C301"
 			(at 205.74 110.4899 0)
 			(effects
@@
 			(project "l3"
 				(path "/1b1408da-cc6a-469f-a506-e797247b3ac8/9673eddf-80ee-4908-b21e-80531a02ef2e"
-					(reference "C334")
+					(reference "C301")
 					(unit 1)
 				)
@@
 		(dnp no)
 		(fields_autoplaced yes)
-		(property "Reference" "D305"
+		(property "Reference" "D303"
 			(at 168.91 160.0199 90)
 			(effects
@@
 			(project "l3"
 				(path "/1b1408da-cc6a-469f-a506-e797247b3ac8/9673eddf-80ee-4908-b21e-80531a02ef2e"
-					(reference "D305")
+					(reference "D303")
 					(unit 1)
 				)
@@
 		(dnp no)
 		(fields_autoplaced yes)
-		(property "Reference" "C327"
+		(property "Reference" "C308"
 			(at 35.56 166.3699 0)
 			(effects
@@
 			(project "l3"
 				(path "/1b1408da-cc6a-469f-a506-e797247b3ac8/9673eddf-80ee-4908-b21e-80531a02ef2e"
-					(reference "C327")
+					(reference "C308")
 					(unit 1)
 				)
@@
 		(dnp no)
 		(fields_autoplaced yes)
-		(property "Reference" "#PWR0351"
+		(property "Reference" "#PWR0304"
 			(at 21.59 162.56 0)
 			(effects
@@
 			(project "l3"
 				(path "/1b1408da-cc6a-469f-a506-e797247b3ac8/9673eddf-80ee-4908-b21e-80531a02ef2e"
-					(reference "#PWR0351")
+					(reference "#PWR0304")
 					(unit 1)
 				)
@@
 		(dnp no)
 		(fields_autoplaced yes)
-		(property "Reference" "U304"
+		(property "Reference" "U302"
 			(at 241.3 93.98 0)
 			(effects
@@
 			(project "l3"
 				(path "/1b1408da-cc6a-469f-a506-e797247b3ac8/9673eddf-80ee-4908-b21e-80531a02ef2e"
-					(reference "U304")
+					(reference "U302")
 					(unit 1)
 				)
@@
 		(dnp no)
 		(fields_autoplaced yes)
-		(property "Reference" "#PWR0354"
+		(property "Reference" "#PWR0303"
 			(at 149.86 149.86 0)
 			(effects
@@
 			(project "l3"
 				(path "/1b1408da-cc6a-469f-a506-e797247b3ac8/9673eddf-80ee-4908-b21e-80531a02ef2e"
-					(reference "#PWR0354")
+					(reference "#PWR0303")
 					(unit 1)
 				)
@@
 		(dnp no)
 		(fields_autoplaced yes)
-		(property "Reference" "#PWR0356"
+		(property "Reference" "#PWR0302"
 			(at 201.93 128.27 0)
 			(effects
@@
 			(project "l3"
 				(path "/1b1408da-cc6a-469f-a506-e797247b3ac8/9673eddf-80ee-4908-b21e-80531a02ef2e"
-					(reference "#PWR0356")
+					(reference "#PWR0302")
 					(unit 1)
 				)
@@
 		(dnp no)
 		(fields_autoplaced yes)
-		(property "Reference" "C336"
+		(property "Reference" "C303"
 			(at 255.27 110.4899 0)
 			(effects
@@
 			(project "l3"
 				(path "/1b1408da-cc6a-469f-a506-e797247b3ac8/9673eddf-80ee-4908-b21e-80531a02ef2e"
-					(reference "C336")
-					(unit 1)
-				)
+					(reference "C303")
+					(unit 1)
+				)

Commit message: 死
Parts:
- renumbered C301 to C401, C302 to C402, C303 to C403, C304 to C404, C305 to C405, C306 to C406, C307 to C407, C308 to C408, C309 to C409, C310 to C410, C311 to C411, C312 to C412, C313 to C413, D301 to D401, D302 to D402, D303 to D403, J301 to J401, R301 to R401, R302 to R402, SW301 to SW401, U301 to U401, U302 to U402, Y301 to Y401
