File: processingUnit/l3.kicad_pcb (KiCad board)
At the start: 2 copper layers, 43 parts, among them J101 Conn_01x05, J102 Conn_01x04, J103 Conn_01x07, SW201 ENC RST, SW301 IMU RST, SW302 IMU RST, U201 STM32F103Cx, U301 STM32F103Cx, U302 BNO085, Y201 8Mhz, Y301 8Mhz

Commit message: L3 Schematic
Parts:
- removed J103: Conn_01x07, Connector_JST:JST_XH_S7B-XH-A_1x07_P2.50mm_Horizontal
- C303: value 2u2 -> 0u1
- C307, C308: value 0u1 -> 2u2
- C309: value C -> 0u1
- R302: value R -> 10K
- R303: value 4K7 -> R
- R304: value 4K7 -> 10K
- R305: value 1K -> 10K
- SW302: value IMU RST -> SW_SPST; footprint Button_Switch_THT:SW_PUSH_6mm -> Connector_JST:JST_XH_B2B-XH-A_1x02_P2.50mm_Vertical
- U301: value STM32F103Cx -> STM32F401C_B-C_Ux; footprint Package_DFN_QFN:QFN-48-1EP_7x7mm_P0.5mm_EP5.6x5.6mm_ThermalVias -> Package_DFN_QFN:QFN-48-1EP_7x7mm_P0.5mm_EP5.6x5.6mm
Connections:
- C309 pad 1: /IMU/BNO RST -> +3V3 FILT
- R301 pad 2: /IMU/BNO RST -> Net-(U302-P0)
- R302 pad 1: GNDREF -> +3V3 FILT
- R302 pad 2: /IMU/IMU BOOT0 -> Net-(U302-P1)
- R303 pad 1: +3V3 FILT -> GNDREF
- R303 pad 2: /IMU/IMU SCL -> /IMU/IMU BOOT0
- R304 pad 2: /IMU/IMU SDA -> /IMU/IMU MOSI
- R305 pad 1: Net-(D301-K) -> +3V3 FILT
- R305 pad 2: GNDREF -> /IMU/IMU MISO
- SW301 pad 2: /IMU/BNO RST -> /IMU/IMU RST
- SW302 pad 1: GNDREF -> /driver/M SW
- SW302 pad 2: /IMU/IMU RST -> GND
- U301 pad 15: /IMU/TNSY SCK -> /ENC/TNSY SCK
- U301 pad 16: /IMU/TNSY MISO -> /ENC/TNSY MISO
- U301 pad 17: /IMU/TNSY MOSI -> /ENC/TNSY MOSI
- U301 pad 21: unconnected-(U301C-PB10-Pad21) -> /IMU/IMU INT
- U301 pad 22: unconnected-(U301C-PB11-Pad22) -> +3V3 FILT
- U301 pad 25: unconnected-(U301C-PB12-Pad25) -> /IMU/IMU NSS
- U301 pad 26: unconnected-(U301C-PB13-Pad26) -> /IMU/IMU SCK
- U301 pad 27: unconnected-(U301C-PB14-Pad27) -> /IMU/IMU MISO
- U301 pad 28: unconnected-(U301C-PB15-Pad28) -> /IMU/IMU MOSI
- U301 pad 42: /IMU/IMU SCL -> unconnected-(U301C-PB6-Pad42)
- U301 pad 43: /IMU/IMU SDA -> unconnected-(U301C-PB7-Pad43)
- U301 pad 46: unconnected-(U301C-PB9-Pad46) -> /IMU/IMU RST
- U302 pad JP1_4: /IMU/IMU SCL -> /IMU/IMU SCK
- U302 pad JP1_5: /IMU/IMU SDA -> /IMU/IMU MISO
- U302 pad JP1_6: unconnected-(U302-~{INT}-PadJP1_6) -> /IMU/IMU INT
- U302 pad JP2_2: unconnected-(U302-P0-PadJP2_2) -> Net-(U302-P0)
- U302 pad JP2_3: unconnected-(U302-P1-PadJP2_3) -> Net-(U302-P1)
- U302 pad JP2_4: /IMU/BNO RST -> /IMU/IMU RST
- U302 pad JP2_5: unconnected-(U302-MOSI-PadJP2_5) -> /IMU/IMU MOSI
- U302 pad JP2_6: unconnected-(U302-CS-PadJP2_6) -> /IMU/IMU NSS

Commit message: Schematic L3
Parts:
- added C311: 470u, 2024l2:CP_Radial_D8.0mm_P3.50mm, F.Cu at (-104.6, 131.3)
- added C312: 0u1, 2024l2:cap0603, F.Cu at (-97.5, 136.3)
- added C313: 470u, 2024l2:CP_Radial_D8.0mm_P3.50mm, F.Cu at (-104.6, 140.8)
- added C314: 0u1, 2024l2:cap0603, F.Cu at (-97.5, 139.2)
- added C315: 470u, 2024l2:CP_Radial_D8.0mm_P3.50mm, F.Cu at (-104.6, 150.4)
- added C316: 0u1, 2024l2:cap0603, F.Cu at (-97.5, 142.1)
- added C317: 470u, 2024l2:CP_Radial_D8.0mm_P3.50mm, F.Cu at (-104.6, 159.9)
- added C318: 0u1, 2024l2:cap0603, F.Cu at (-97.5, 145.0)
- added IC301: VNH5019ATR-E, 2024l2:VNH5019A-E, F.Cu at (-100.2, 116.2)
- added IC302: VNH5019ATR-E, 2024l2:VNH5019A-E, F.Cu at (-81.8, 116.2)
- added IC303: VNH5019ATR-E, 2024l2:VNH5019A-E, F.Cu at (-63.4, 116.2)
- added IC304: VNH5019ATR-E, 2024l2:VNH5019A-E, F.Cu at (-45.0, 116.2)
- added J302: M1, Connector_JST:JST_PH_B6B-PH-K_1x06_P2.00mm_Vertical, F.Cu at (-75.4, 169.4)
- added J306: M1, Connector_JST:JST_PH_B6B-PH-K_1x06_P2.00mm_Vertical, F.Cu at (-75.4, 176.0)
- added J307: M1, Connector_JST:JST_PH_B6B-PH-K_1x06_P2.00mm_Vertical, F.Cu at (-75.4, 182.5)
- added J308: M1, Connector_JST:JST_PH_B6B-PH-K_1x06_P2.00mm_Vertical, F.Cu at (-75.4, 189.1)
- added Q301: AON6354, 2024l2:8-DFN (5x6), F.Cu at (-96.4, 130.7)
- added Q302: AON6354, 2024l2:8-DFN (5x6), F.Cu at (-89.5, 130.7)
- added Q303: AON6354, 2024l2:8-DFN (5x6), F.Cu at (-82.6, 130.7)
- added Q304: AON6354, 2024l2:8-DFN (5x6), F.Cu at (-75.7, 130.7)
- added R311: 3K3, 2024l2:res0603, F.Cu at (-97.5, 147.9)
- added R312: 3K3, 2024l2:res0603, F.Cu at (-97.5, 150.8)
- added R313: 3K3, 2024l2:res0603, F.Cu at (-97.5, 153.7)
- added R314: 3K3, 2024l2:res0603, F.Cu at (-97.5, 156.6)
- added R315: 1K, 2024l2:res0603, F.Cu at (-97.5, 159.5)
- added R316: 1K, 2024l2:res0603, F.Cu at (-92.8, 136.3)
- added R317: 1K, 2024l2:res0603, F.Cu at (-92.8, 139.2)
- added R318: 1K, 2024l2:res0603, F.Cu at (-92.8, 142.1)
- added R319: 1K, 2024l2:res0603, F.Cu at (-92.8, 145.0)
- added R320: 1K, 2024l2:res0603, F.Cu at (-92.8, 147.9)
- added R321: 1K, 2024l2:res0603, F.Cu at (-92.8, 150.8)
- added R322: 1K, 2024l2:res0603, F.Cu at (-92.8, 153.7)
- added R323: 1K, 2024l2:res0603, F.Cu at (-92.8, 156.6)
- added R324: 1K, 2024l2:res0603, F.Cu at (-92.8, 159.5)
- added R325: 10K, 2024l2:res0603, F.Cu at (-88.1, 136.3)
- added R326: 10K, 2024l2:res0603, F.Cu at (-88.1, 139.2)
- added R327: 3K3, 2024l2:res0603, F.Cu at (-88.1, 142.1)
- added R328: 3K3, 2024l2:res0603, F.Cu at (-88.1, 145.0)
- added R329: 3K3, 2024l2:res0603, F.Cu at (-88.1, 147.9)
- added R330: 3K3, 2024l2:res0603, F.Cu at (-88.1, 150.8)
- added R331: 1K, 2024l2:res0603, F.Cu at (-88.1, 153.7)
- added R332: 1K, 2024l2:res0603, F.Cu at (-88.1, 156.6)
- added R333: 1K, 2024l2:res0603, F.Cu at (-88.1, 159.5)
- added R334: 1K, 2024l2:res0603, F.Cu at (-83.4, 136.3)
- added R335: 1K, 2024l2:res0603, F.Cu at (-83.4, 139.2)
- added R336: 1K, 2024l2:res0603, F.Cu at (-83.4, 142.1)
- added R337: 1K, 2024l2:res0603, F.Cu at (-83.4, 145.0)
- added R338: 1K, 2024l2:res0603, F.Cu at (-83.4, 147.9)
- added R339: 1K, 2024l2:res0603, F.Cu at (-83.4, 150.8)
- added R340: 1K, 2024l2:res0603, F.Cu at (-83.4, 153.7)
- added R341: 10K, 2024l2:res0603, F.Cu at (-83.4, 156.6)
- added R342: 10K, 2024l2:res0603, F.Cu at (-83.4, 159.5)
- added R343: 1k, 2024l2:res0603, F.Cu at (-60.0, 168.1)
- added R344: 1k, 2024l2:res0603, F.Cu at (-60.0, 171.0)
- added R345: 1k, 2024l2:res0603, F.Cu at (-60.0, 173.9)
- added R346: 1k, 2024l2:res0603, F.Cu at (-60.0, 176.8)
- added R347: 1k, 2024l2:res0603, F.Cu at (-60.0, 179.7)
- added R348: 1k, 2024l2:res0603, F.Cu at (-60.0, 182.6)
- added R349: 1k, 2024l2:res0603, F.Cu at (-60.0, 185.5)
- added R350: 1k, 2024l2:res0603, F.Cu at (-60.0, 188.4)
- added SW303: SW_SPDT, 2024l2:SS12D00G3, F.Cu at (-85.2, 169.0)
- added U305: Teensy 4.0, 2024l2:Teensy 4.0, F.Cu at (-99.7, 185.9)
- moved C101 128.7 mm to (-104.1, 53.2)
- moved C102 128.7 mm to (-104.1, 56.3)
- moved C103 128.7 mm to (-104.1, 59.4)
- moved C104 128.7 mm to (-104.1, 62.5)
- moved C201 128.7 mm to (-80.1, 71.1)
- moved C202 128.7 mm to (-80.1, 74.2)
- moved C203 128.7 mm to (-80.1, 77.3)
- moved C204 128.7 mm to (-80.1, 80.4)
- moved C205 128.7 mm to (-80.1, 83.5)
- moved C206 128.7 mm to (-75.4, 71.1)
- moved C207 128.7 mm to (-75.4, 74.2)
- moved C301 128.7 mm to (-80.1, 39.6)
- moved C302 128.7 mm to (-80.1, 42.7)
- moved C303 128.7 mm to (-80.1, 45.8)
- moved C304 128.7 mm to (-80.1, 48.9)
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Connections:
- U201 pad 10: /ENC/M1 ENC A -> /ENC/M1 PWM
- U201 pad 11: /ENC/M1 ENC B -> /ENC/M1 DIR
- U201 pad 12: /ENC/M1 IN A -> /ENC/M2 PWM
- U201 pad 13: /ENC/M1 IN B -> /ENC/M2 DIR
- U201 pad 18: unconnected-(U201C-PB0-Pad18) -> /ENC/M1 ENC A
- U201 pad 19: unconnected-(U201C-PB1-Pad19) -> /ENC/M1 ENC B
- U201 pad 21: /ENC/M2 IN B -> /ENC/M4 ENC A
- U201 pad 22: /ENC/M3 IN A -> /ENC/M4 ENC B
- U201 pad 26: /ENC/M3 IN B -> unconnected-(U201C-PB13-Pad26)
- U201 pad 27: /ENC/M4 IN A -> unconnected-(U201C-PB14-Pad27)
- U201 pad 31: /ENC/M2 IN A -> unconnected-(U201C-PA10-Pad31)
- U201 pad 40: /ENC/M4 ENC A -> /ENC/M3 PWM
- U201 pad 41: /ENC/M4 ENC B -> /ENC/M3 DIR
- U201 pad 42: /ENC/M2 ENC A -> /ENC/M4 PWM
- U201 pad 43: /ENC/M2 ENC B -> /ENC/M4 DIR
- U201 pad 45: unconnected-(U201C-PB8-Pad45) -> /ENC/M2 ENC A
- U201 pad 46: unconnected-(U201C-PB9-Pad46) -> /ENC/M2 ENC B

Commit message: footprint
Parts:
- added J104: Conn_01x10, Library:526101071, F.Cu at (-49.6, 69.6)
- added J301: Conn_01x10, Library:526101071, F.Cu at (-49.6, 77.7)
- added R306: 10K, Library:res0603, F.Cu at (-35.2, 67.0)
- added R307: 10K, Library:res0603, F.Cu at (-35.2, 70.1)
- added R308: 10K, Library:res0603, F.Cu at (-35.2, 73.2)
- added R309: 10K, Library:res0603, F.Cu at (-35.2, 76.3)
- added R310: 1K, Library:res0603, F.Cu at (-35.2, 79.4)
- added U303: SN74LVC2G04, Library:SOT-23-6, F.Cu at (-57.0, 86.0)
- added U304: SN74LVC2G04, Library:SOT-23-6, F.Cu at (-57.0, 90.5)
- IC301, IC302, IC303, IC304: footprint 2024l2:VNH5019A-E -> Library:ST_MultiPowerSO-30
- R311, R312, R313, R314, R315, R316, R317, R318, R319, R320, R321, R322, R323, R324, R325, R326, R327, R328, R329, R330, R331, R332, R333, R334, R335, R336, R337, R338, R339, R340, R341, R342, R343, R344, R345, R346, R347, R348, R349, R350: footprint 2024l2:res0603 -> Library:res0603
- U305: footprint 2024l2:Teensy 4.0 -> Library:Teensy 4.0
Connections:
- R311 pad 2: +3V3 FILT -> GNDREF
- R312 pad 2: +3V3 FILT -> GNDREF
- R313 pad 2: +3V3 FILT -> GNDREF
- R314 pad 2: +3V3 FILT -> GNDREF
- R327 pad 2: +3V3 FILT -> GNDREF
- R328 pad 2: +3V3 FILT -> GNDREF
- R329 pad 2: +3V3 FILT -> GNDREF
- R330 pad 2: +3V3 FILT -> GNDREF
- SW302 pad 2: GND -> +3V3 FILT
Other:
- board outline added: 120 x 120 mm

Commit message: L3 layout
Parts:
- removed J104: Conn_01x10, Library:526101071
- added J309: Conn_01x02, Library:xt30-f, B.Cu at (73.8, 102.0)
- IC301, IC302, IC303, IC304, J301, J302, J306, J307, J308, Q301, Q302, Q303, Q304, R319, R321, R323, U303, U304: moved to B.Cu
- Y301: value 8Mhz -> 16Mhz
- moved J101 294.3 mm to (191.8, 105.2), turned to 90 degrees
- moved C313 290.1 mm to (181.8, 95.5)
- moved C311 287.7 mm to (181.8, 104.5)
- moved J306 282.3 mm to (192.6, 87.0), turned to 90 degrees
- moved IC301 277.2 mm to (177.0, 118.0), turned to 90 degrees
- moved R346 275.7 mm to (196.9, 76.8), turned to 180 degrees
- moved R345 273.9 mm to (196.9, 79.1), turned to 180 degrees
- moved J302 271.9 mm to (192.6, 123.0), turned to 90 degrees
- moved Q301 270.5 mm to (172.8, 104.8), turned to 90 degrees
- moved Q302 264.7 mm to (172.8, 95.2), turned to 90 degrees
- moved R344 263.4 mm to (196.9, 112.8), turned to 180 degrees
- moved R343 262.3 mm to (196.9, 115.1), turned to 180 degrees
- moved IC302 261.1 mm to (177.0, 82.0), turned to 90 degrees
- moved R323 260.3 mm to (164.8, 119.4)
- moved R321 259.9 mm to (164.8, 116.4)
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Connections:
- J308 pad 1: /driver/M4 OUT B -> /driver/M4 OUT A
- J308 pad 2: /driver/M4 OUT A -> /driver/M4 OUT B
- Y301 pad 2: /IMU/IMU OSC OUT -> GNDREF
- Y301 pad 3: GNDREF -> /IMU/IMU OSC OUT
Routing:
- net +5V FILT: track 0.00 -> 102.0 mm
- net /M2 ENC A: track 0.00 -> 3.60 mm
- net /M1 ENC A: track 0.00 -> 3.60 mm
- net /M4 ENC A: track 0.00 -> 3.60 mm
- net /M4 ENC B: track 0.00 -> 3.57 mm
- net /M2 ENC B: track 0.00 -> 3.57 mm
- net /M1 ENC B: track 0.00 -> 3.57 mm
- added copper zone on B.Cu, net /driver/M1 OUT A
- added copper zone on F.Cu, net /driver/M1 OUT A
- added copper zone on B.Cu, net /driver/M1 OUT B
- added copper zone on B.Cu, net /driver/M2 OUT A
- added copper zone on F.Cu, net /driver/M2 OUT A
- added copper zone on B.Cu, net /driver/M2 OUT B
- added copper zone on B.Cu, net /driver/M3 OUT A
- added copper zone on F.Cu, net /driver/M3 OUT A
- added copper zone on B.Cu, net /driver/M3 OUT B
- added copper zone on B.Cu, net /driver/M4 OUT A
- added copper zone on F.Cu, net /driver/M4 OUT A
- added copper zone on B.Cu, net /driver/M4 OUT B
- added copper zone on B.Cu, net GNDREF
- added copper zone on F.Cu, net GNDREF
- added copper zone on B.Cu, net Net-(C311-Pad1)
- added copper zone on F.Cu, net Net-(C311-Pad1)
- added copper zone on B.Cu, net Net-(C313-Pad1)
- added copper zone on F.Cu, net Net-(C313-Pad1)
- added copper zone on B.Cu, net Net-(C315-Pad1)
- added copper zone on F.Cu, net Net-(C315-Pad1)
- added copper zone on B.Cu, net Net-(C317-Pad1)
- added copper zone on F.Cu, net Net-(C317-Pad1)
