File: processingUnit/l3.kicad_pcb (KiCad board)
At the start: 2 copper layers, 120 x 120 mm, 113 parts, among them IC301 VNH5019ATR-E, IC302 VNH5019ATR-E, IC303 VNH5019ATR-E, IC304 VNH5019ATR-E, J101 Conn_01x05, J102 Conn_01x04, J301 Conn_01x10, J302 M1, J306 M1, J307 M1, J308 M1, J309 Conn_01x02, Q301 AON6354, Q302 AON6354, Q303 AON6354, Q304 AON6354, SW201 ENC RST, SW301 IMU RST, SW302 SW_SPST, SW303 SW_SPDT, U201 STM32F103Cx, U301 STM32F401C_B-C_Ux, U302 BNO085, U303 SN74LVC2G04, U304 SN74LVC2G04, U305 Teensy 4.0, Y201 8Mhz, Y301 16Mhz

Commit message: L3
Parts:
- C101, C102, C103, C104, C308, C309, FB101, FB102, R301, R302, R304, R305, R306, R307, R308, R309, R315, R317, R322: moved to B.Cu
- C311, C313, C315, C317: footprint 2024l2:CP_Radial_D8.0mm_P3.50mm -> Library:CP_Radial_D8.0mm_P3.50mm
- C312, C314, C316, C318: footprint 2024l2:cap0603 -> Library:cap0603; moved to B.Cu
- Q301, Q302, Q303, Q304: footprint 2024l2:8-DFN (5x6) -> Library:8-DFN (5x6)
- SW303: footprint 2024l2:SS12D00G3 -> Library:SS12D00G3
- Y301: footprint Crystal:Resonator_SMD_Murata_CSTxExxV-3Pin_3.0x1.1mm -> Library:CX3225SB16000D0FPLCC
- moved C314 278.4 mm to (177.8, 98.0), turned to -90 degrees
- moved C312 277.4 mm to (177.8, 102.0), turned to 90 degrees
- moved R322 266.6 mm to (163.4, 80.0), turned to 180 degrees
- moved R315 261.2 mm to (160.8, 120.6)
- moved R317 254.5 mm to (160.8, 117.4)
- moved C302 238.0 mm to (156.2, 70.6)
- moved C308 237.7 mm to (155.8, 104.0), turned to 180 degrees
- moved C309 236.2 mm to (155.8, 106.4), turned to 180 degrees
- moved C304 234.7 mm to (153.8, 67.6), turned to 90 degrees
- moved C305 232.0 mm to (153.0, 80.2), turned to -90 degrees
- moved SW301 230.1 mm to (147.2, 58.0)
- moved C310 229.5 mm to (156.6, 61.8), turned to 90 degrees
- moved U301 227.8 mm to (150.0, 74.0), turned to -90 degrees
- moved C301 227.4 mm to (143.6, 80.2), turned to 180 degrees
- moved R305 226.8 mm to (155.8, 96.2)
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Routing:
- net +3V3 FILT: track 0.00 -> 85.3 mm, vias 0 -> 4
- net /IMU/IMU RST: track 0.00 -> 74.9 mm, vias 0 -> 1
- net /IMU/IMU INT: track 0.00 -> 33.7 mm, vias 0 -> 1
- net /IMU/IMU SCK: track 0.00 -> 28.2 mm, vias 0 -> 2
- net /IMU/IMU MISO: track 0.00 -> 25.5 mm, vias 0 -> 2
- net /IMU/IMU MOSI: track 0.00 -> 25.3 mm
- net /IMU/IMU NSS: track 0.00 -> 21.3 mm
- net +3V3: track 0.00 -> 10.9 mm
- net +5V: track 0.00 -> 7.63 mm
- net /IMU/IMU OSC IN: track 0.00 -> 5.70 mm
- net /IMU/IMU OSC OUT: track 0.00 -> 3.77 mm
- net Net-(U302-P0): track 0.00 -> 2.57 mm
- net Net-(U302-P1): track 0.00 -> 2.54 mm
- net Net-(IC301-INA): track 0.00 -> 2.42 mm
- net Net-(IC301-INB): track 0.00 -> 2.28 mm
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
Commit message: STM32
Parts:
- moved R310 230.2 mm to (160.0, 76.0)
- moved D301 225.7 mm to (156.2, 76.0), turned to 180 degrees
- moved U201 150.9 mm to (-52.0, 93.6)
- moved Y201 52.4 mm to (-61.6, 93.2), turned to -90 degrees
- moved C206 39.3 mm to (-48.6, 99.8), turned to -90 degrees
- moved C204 38.9 mm to (-46.4, 99.8), turned to -90 degrees
- moved C205 35.2 mm to (-45.6, 90.4)
- moved C201 32.7 mm to (-58.2, 95.4), turned to 180 degrees
- moved C202 28.2 mm to (-55.2, 87.4), turned to 90 degrees
- moved D201 27.5 mm to (-49.8, 87.4), turned to -90 degrees
- moved R202 25.7 mm to (-49.8, 83.6), turned to 90 degrees
- moved C203 25.6 mm to (-58.2, 90.6), turned to 180 degrees
- moved SW201 25.4 mm to (-69.5, 96.9), turned to 90 degrees
- moved R201 23.7 mm to (-52.8, 87.4), turned to -90 degrees
- moved C207 15.8 mm to (-67.2, 87.7), turned to 180 degrees
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Routing:
- net /ENC/ENC RST: track 0.00 -> 20.7 mm
- net +3V3 FILT: track 85.3 -> 99.7 mm
- net /ENC/ENC OSC IN: track 0.00 -> 6.59 mm
- net /ENC/ENC OSC OUT: track 0.00 -> 6.30 mm
- net Net-(D201-K): track 0.00 -> 2.20 mm
- net Net-(D301-K): track 0.00 -> 2.20 mm
- net /IMU/IMU LED: track 0.00 -> 2.07 mm
- net /ENC/ENC LED: track 0.00 -> 2.00 mm

Commit message: STM32
Parts:
- moved SW201 228.0 mm to (154.7, 138.7), turned to 180 degrees
- moved C207 218.1 mm to (145.4, 136.5), turned to -90 degrees
- moved Y201 216.0 mm to (151.0, 130.9), turned to 0 degrees
- moved C201 213.8 mm to (153.2, 127.5), turned to -90 degrees
- moved C203 209.8 mm to (148.4, 127.5), turned to -90 degrees
- moved C206 207.0 mm to (157.6, 117.9), turned to 0 degrees
- moved U201 205.2 mm to (151.4, 121.2), turned to 90 degrees
- moved C204 204.6 mm to (157.6, 115.7), turned to 0 degrees
- moved C202 203.8 mm to (145.2, 124.5), turned to 180 degrees
- moved R201 201.0 mm to (145.2, 122.1), turned to 0 degrees
- moved D201 197.5 mm to (145.2, 119.1), turned to 0 degrees
- moved C205 195.3 mm to (148.2, 114.9), turned to 90 degrees
- moved R202 194.4 mm to (141.4, 119.1), turned to 180 degrees

Commit message: L3 Routing
Parts:
- R311, R312, R313, R314, R327, R328, R329, R330: moved to B.Cu
- R315, R317, R319, R321, R322, R323, U303, U304: moved to F.Cu
- moved R324 267.8 mm to (163.6, 82.4)
- moved R314 266.9 mm to (158.2, 80.2), turned to 180 degrees
- moved R313 264.9 mm to (158.2, 84.6), turned to 180 degrees
- moved R318 263.8 mm to (163.6, 80.2)
- moved R320 263.6 mm to (163.6, 86.8)
- moved R316 261.6 mm to (163.6, 84.6)
- moved R311 257.5 mm to (158.0, 116.2), turned to 180 degrees
- moved R312 257.3 mm to (158.0, 120.6), turned to 180 degrees
- moved R326 254.3 mm to (159.8, 82.4), turned to 180 degrees
- moved R325 248.6 mm to (159.8, 118.4), turned to 180 degrees
- moved R327 238.1 mm to (141.6, 79.4)
- moved R328 237.7 mm to (141.6, 83.8)
- moved R333 237.0 mm to (136.4, 83.8), turned to 180 degrees
- moved R331 236.5 mm to (136.4, 79.4), turned to 180 degrees
- moved R341 235.9 mm to (140.2, 81.6)
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Connections:
- J302 pad 5: /M1 ENC B -> M1 ENC B
- J302 pad 6: /M1 ENC A -> M1 ENC A
- J306 pad 5: /M2 ENC B -> M2 ENC B
- J306 pad 6: /M2 ENC A -> M2 ENC A
- J307 pad 5: /M3 ENC B -> M3 ENC B
- J307 pad 6: /M3 ENC A -> M3 ENC A
- J308 pad 5: /M4 ENC B -> M4 ENC B
- J308 pad 6: /M4 ENC A -> M4 ENC A
- R343 pad 2: /M1 ENC B -> M1 ENC B
- R344 pad 2: /M1 ENC A -> M1 ENC A
- R345 pad 2: /M2 ENC B -> M2 ENC B
- R346 pad 2: /M2 ENC A -> M2 ENC A
- R347 pad 2: /M3 ENC B -> M3 ENC B
- R348 pad 2: /M3 ENC A -> M3 ENC A
- R349 pad 2: /M4 ENC B -> M4 ENC B
- R350 pad 2: /M4 ENC A -> M4 ENC A
- U201 pad 18: /ENC/M1 ENC A -> M1 ENC A
- U201 pad 19: /ENC/M1 ENC B -> M1 ENC B
- U201 pad 21: /ENC/M4 ENC A -> M4 ENC A
- U201 pad 22: /ENC/M4 ENC B -> M4 ENC B
- U201 pad 29: /ENC/M3 ENC A -> M3 ENC A
- U201 pad 30: /ENC/M3 ENC B -> M3 ENC B
- U201 pad 45: /ENC/M2 ENC A -> M2 ENC A
- U201 pad 46: /ENC/M2 ENC B -> M2 ENC B
Routing:
- net +5V FILT: track 104.2 -> 243.2 mm, vias 0 -> 1
- net /driver/M SW: track 0.00 -> 111.4 mm, vias 0 -> 8
- net +3V3: track 10.9 -> 97.5 mm
- net /IMU/IMU RST: track 74.9 -> 33.5 mm
- net /IMU/IMU INT: track 33.7 -> 4.37 mm
- net /IMU/IMU SCK: track 28.2 -> 2.32 mm, vias 2 -> 0
- net /IMU/IMU MISO: track 25.5 -> 2.29 mm, vias 2 -> 0
- net /IMU/IMU MOSI: track 25.3 -> 2.49 mm
- net /IMU/IMU NSS: track 21.3 -> 2.51 mm
- net /driver/CPM1: track 0.00 -> 18.4 mm, vias 0 -> 2
- net /driver/CPM3: track 0.00 -> 18.1 mm, vias 0 -> 2
- net /driver/CPM2: track 0.00 -> 17.3 mm, vias 0 -> 2
- net /driver/CPM4: track 0.00 -> 17.0 mm, vias 0 -> 2
- net /ENC/ENC RST: track 20.7 -> 3.86 mm
- net /tnsy/TEENSY PWR: track 0.00 -> 4.85 mm
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- added copper zone on B.Cu, net +12V

Commit message: L3
Parts:
- J101, R315, R316, R317, R318, R319, R320, R321, R322, R323, R324, R325, R326, R331, R332, R333, R334, R335, R336, R337, R338, R339, R340, R341, R342: moved to B.Cu
- moved U304 86.6 mm to (135.2, 100.0), turned to 180 degrees
- moved U303 65.7 mm to (164.8, 100.0), turned to 0 degrees
- moved Y201 60.8 mm to (163.1, 71.0), turned to 0 degrees
- moved C207 60.3 mm to (166.2, 71.5), turned to -90 degrees
- moved SW201 58.1 mm to (176.4, 71.7), turned to 180 degrees
- moved C203 57.1 mm to (160.5, 66.4), turned to -90 degrees
- moved C202 55.7 mm to (157.2, 63.8), turned to 180 degrees
- moved C201 55.2 mm to (165.3, 67.5), turned to -90 degrees
- moved R201 52.7 mm to (157.3, 61.4), turned to 0 degrees
- moved R202 52.3 mm to (153.5, 57.8), turned to 180 degrees
- moved D201 49.0 mm to (157.3, 57.8), turned to 0 degrees
- moved U201 47.4 mm to (163.5, 60.3), turned to 90 degrees
- moved C205 41.8 mm to (160.3, 54.0), turned to 90 degrees
- moved C206 40.0 mm to (169.7, 56.9), turned to 0 degrees
- moved C204 37.0 mm to (169.7, 54.7), turned to 0 degrees
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Connections:
- J301 pad 1: +3V3 -> GNDREF
- J301 pad 10: GNDREF -> +3V3
- J301 pad 3: LIGHT RX -> unconnected-(J301-Pin_3-Pad3)
- J301 pad 4: LIGHT TX -> MCU SWCLK
- J301 pad 5: MCU RST -> MCU SWDIO
- J301 pad 6: MCU SWDIO -> MCU RST
- J301 pad 7: MCU SWCLK -> LIGHT RX
- J301 pad 8: unconnected-(J301-Pin_8-Pad8) -> LIGHT TX
- U301 pad 14: /IMU/IMU NSS -> /IMU/TNSY NSS
- U303 pad 1: /ENC/M1 DIR -> /ENC/M2 DIR
- U303 pad 3: /ENC/M2 DIR -> /ENC/M1 DIR
- U303 pad 4: /driver/M2 IN B -> /driver/M1 IN B
- U303 pad 6: /driver/M1 IN B -> /driver/M2 IN B
- U304 pad 1: /ENC/M3 DIR -> /ENC/M4 DIR
- U304 pad 3: /ENC/M4 DIR -> /ENC/M3 DIR
- U304 pad 4: /driver/M4 IN B -> /driver/M3 IN B
- U304 pad 6: /driver/M3 IN B -> /driver/M4 IN B
- U305 pad 3: /IMU/IMU NSS -> /tnsy/IMU NSS
- U305 pad 7: /tnsy/L1 RX -> LIGHT RX
- U305 pad 8: /tnsy/L1 TX -> LIGHT TX
Routing:
- net +3V3: track 97.5 -> 11.5 mm
- net /ENC/M4 PWM: track 2.30 -> 77.9 mm, vias 0 -> 3
- net /ENC/M4 DIR: track 0.00 -> 73.9 mm, vias 0 -> 3
- net /ENC/M1 DIR: track 0.00 -> 71.1 mm, vias 0 -> 3
- net /ENC/M3 DIR: track 0.00 -> 65.0 mm, vias 0 -> 2
- net +5V FILT: track 243.2 -> 306.6 mm
- net /ENC/M1 PWM: track 2.20 -> 61.8 mm, vias 0 -> 3
- net /IMU/IMU SCK: track 2.32 -> 48.9 mm
- net /ENC/M2 DIR: track 0.00 -> 44.4 mm, vias 0 -> 3
- net /ENC/M3 PWM: track 2.20 -> 44.8 mm, vias 0 -> 3
- net /driver/M4 IN B: track 0.00 -> 26.0 mm, vias 0 -> 1
- net /driver/M2 IN B: track 0.00 -> 25.6 mm, vias 0 -> 1
- net /ENC/M2 PWM: track 2.20 -> 26.7 mm, vias 0 -> 3
- net /driver/M SW: track 111.4 -> 127.3 mm
- net +3V3 FILT: track 99.7 -> 84.0 mm, vias 4 -> 2
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- removed copper zone on B.Cu, net +12V

Commit message: L3
Parts:
- U201: footprint Package_DFN_QFN:QFN-48-1EP_7x7mm_P0.5mm_EP5.6x5.6mm_ThermalVias -> Package_DFN_QFN:QFN-48-1EP_7x7mm_P0.5mm_EP5.6x5.6mm
- moved C310 16.9 mm to (119.0, 69.8), turned to -90 degrees
- moved J309 12.6 mm to (242.6, 122.2)
- moved SW301 11.6 mm to (128.3, 71.7), turned to 180 degrees
- moved J102 6.55 mm to (232.8, 104.8)
- moved SW302 2.71 mm to (125.4, 139.9), turned to -90 degrees
- moved SW201 1.85 mm to (178.2, 71.7)
Connections:
- J301 pad 10: +3V3 -> +3V3 FILT
- U301 pad 14: /IMU/TNSY NSS -> /IMU/IMU STM NSS
- U305 pad 10: unconnected-(U305-Pad10) -> /ENC/ENC NSS
- U305 pad 2: /ENC/ENC NSS -> unconnected-(U305-Pad2)
- U305 pad 3: /tnsy/IMU NSS -> unconnected-(U305-Pad3)
- U305 pad 9: unconnected-(U305-Pad9) -> /IMU/IMU STM NSS
Routing:
- net /ENC/TNSY SCK: track 3.29 -> 148.8 mm, vias 1 -> 2
- net /ENC/ENC NSS: track 0.00 -> 139.1 mm, vias 0 -> 3
- net /ENC/TNSY MISO: track 5.10 -> 133.6 mm, vias 0 -> 2
- net /ENC/TNSY MOSI: track 6.74 -> 134.0 mm, vias 0 -> 2
- net /IMU/IMU STM NSS: track 0.00 -> 80.1 mm, vias 0 -> 1
- net LIGHT TX: track 0.00 -> 66.0 mm, vias 0 -> 1
- net LIGHT RX: track 0.00 -> 64.5 mm, vias 0 -> 1
- net +12V: track 0.00 -> 58.3 mm, vias 0 -> 4
- net /IMU/IMU RST: track 34.5 -> 84.7 mm
- net /IMU/IMU INT: track 2.80 -> 51.5 mm, vias 0 -> 3
- net /driver/M SW: track 127.3 -> 171.1 mm
- net /IMU/IMU MISO: track 2.29 -> 45.9 mm
- net /IMU/IMU MOSI: track 2.49 -> 43.6 mm, vias 0 -> 2
- net /IMU/IMU NSS: track 2.51 -> 37.6 mm, vias 0 -> 2
- net +3V3 FILT: track 84.0 -> 115.4 mm, vias 2 -> 5
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- added copper zone on B.Cu, net +12V

Commit message: L3
Parts:
- moved C207 15.2 mm to (181.2, 69.6)
- moved SW201 7.91 mm to (171.8, 67.2), turned to 0 degrees
Routing:
- net /ENC/ENC RST: track 18.6 -> 25.6 mm

Commit message: L3
Routing:
- net +3V3 FILT: track 115.4 -> 162.1 mm, vias 5 -> 6
- net /ENC/TNSY MISO: track 133.6 -> 135.5 mm
- net /IMU/IMU STM NSS: track 80.1 -> 81.3 mm
- net /ENC/ENC NSS: track 139.1 -> 140.2 mm
- net /IMU/IMU RST: track 84.7 -> 85.8 mm
- net /ENC/TNSY MOSI: track 134.0 -> 135.0 mm
- net /ENC/TNSY SCK: track 148.8 -> 149.5 mm
- net LIGHT TX: track 66.0 -> 65.3 mm
- net /IMU/IMU INT: track 51.5 -> 52.0 mm, vias 3 -> 2
