File: processingUnit/imu.kicad_sch (KiCad schematic)
At the start: 25 parts, among them SW301 IMU RST, U301 STM32F401C_B-C_Ux, U302 BNO085, Y301 16Mhz

Commit message: L3
Connections:
- net IMU NSS: no longer U301.14 (PA4)
- new net TNSY NSS: U301.14 (PA4)
Changed lines of the file:
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@@
 		)
 	)
-	(hierarchical_label "IMU NSS"
+	(hierarchical_label "TNSY NSS"
 		(shape input)
 		(at 38.1 123.19 180)

Commit message: L3
Connections:
- net TNSY NSS renamed IMU STM NSS
Changed lines of the file:
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@@
 		)
 	)
-	(hierarchical_label "TNSY NSS"
+	(hierarchical_label "IMU STM NSS"
 		(shape input)
 		(at 38.1 123.19 180)

Commit message: L3
Parts:
- added J303: Conn_01x04, symbol Connector_Generic:Conn_01x04
Changed lines of the file:
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@@
+	)
+	(symbol
+		(lib_id "Connector_Generic:Conn_01x04")
+		(at 68.58 173.99 180)
+		(unit 1)
+		(exclude_from_sim no)
+		(in_bom yes)
+		(on_board yes)
+		(dnp no)
+		(fields_autoplaced yes)
+		(property "Reference" "J303"
+			(at 68.58 162.56 0)
+			(effects
+				(font
+					(size 1.27 1.27)
+				)
+			)
+		)
+		(property "Value" "Conn_01x04"
+			(at 68.58 165.1 0)
+			(effects
+				(font
+					(size 1.27 1.27)
+				)
+			)
+		)
+		(property "Footprint" ""
+			(at 68.58 173.99 0)
+			(effects
+				(font
+					(size 1.27 1.27)
+				)
+				(hide yes)
+			)
+		)
+		(property "Datasheet" "~"
+			(at 68.58 173.99 0)
+			(effects
+				(font
+					(size 1.27 1.27)
+				)
+				(hide yes)
+			)
+		)
+		(property "Description" "Generic connector, single row, 01x04, script generated (kicad-library-utils/schlib/autogen/connector/)"
+			(at 68.58 173.99 0)
+			(effects
+				(font
+					(size 1.27 1.27)
+				)
+				(hide yes)
+			)
+		)
+		(pin "1"
+		)
+		(pin "2"
+		)
+		(pin "3"
+		)
+		(pin "4"
+		)
+		(instances
+			(project "l3"
+				(path "/1b1408da-cc6a-469f-a506-e797247b3ac8/65597bc7-5aaa-4f27-9286-e75eee7edae8"
+					(reference "J303")
+					(unit 1)
+				)
+			)
+		)
 	)
 	(symbol

Commit message: L3
Parts:
- J303: footprint (none) -> Connector_PinHeader_2.54mm:PinHeader_1x04_P2.54mm_Vertical
Connections:
- net +3V3 FILT: now also J303.1 (Pin_1)
- net GNDREF: now also J303.4 (Pin_4)
- net IMU SWCLK: now also J303.3 (Pin_3)
- net IMU SWDIO: now also J303.2 (Pin_2)
Changed lines of the file:
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@@
 	(wire
 		(pts
+			(xy 74.93 170.18) (xy 92.71 170.18)
+		)
+		(stroke
+			(width 0)
+			(type default)
+		)
+	)
+	(wire
+		(pts
 			(xy 85.09 53.34) (xy 85.09 55.88)
 		)
@@
 	(wire
 		(pts
+			(xy 74.93 167.64) (xy 92.71 167.64)
+		)
+		(stroke
+			(width 0)
+			(type default)
+		)
+	)
+	(wire
+		(pts
 			(xy 62.23 55.88) (xy 73.66 55.88)
 		)
@@
 		)
 	)
+	(label "IMU SWDIO"
+		(at 76.2 167.64 0)
+		(fields_autoplaced yes)
+		(effects
+			(font
+				(size 1.27 1.27)
+			)
+			(justify left bottom)
+		)
+	)
+	(label "IMU SWCLK"
+		(at 76.2 170.18 0)
+		(fields_autoplaced yes)
+		(effects
+			(font
+				(size 1.27 1.27)
+			)
+			(justify left bottom)
+		)
+	)
 	(label "IMU RST"
 		(at 171.45 138.43 180)
@@
 	)
 	(symbol
+		(lib_id "Connector_Generic:Conn_01x04")
+		(at 97.79 167.64 0)
+		(unit 1)
+		(exclude_from_sim no)
+		(in_bom yes)
+		(on_board yes)
+		(dnp no)
+		(fields_autoplaced yes)
+		(property "Reference" "J303"
+			(at 100.33 167.6399 0)
+			(effects
+				(font
+					(size 1.27 1.27)
+				)
+				(justify left)
+			)
+		)
+		(property "Value" "Conn_01x04"
+			(at 100.33 170.1799 0)
+			(effects
+				(font
+					(size 1.27 1.27)
+				)
+				(justify left)
+			)
+		)
+		(property "Footprint" "Connector_PinHeader_2.54mm:PinHeader_1x04_P2.54mm_Vertical"
+			(at 97.79 167.64 0)
+			(effects
+				(font
+					(size 1.27 1.27)
+				)
+				(hide yes)
+			)
+		)
+		(property "Datasheet" "~"
+			(at 97.79 167.64 0)
+			(effects
+				(font
+					(size 1.27 1.27)
+				)
+				(hide yes)
+			)
+		)
+		(property "Description" "Generic connector, single row, 01x04, script generated (kicad-library-utils/schlib/autogen/connector/)"
+			(at 97.79 167.64 0)
+			(effects
+				(font
+					(size 1.27 1.27)
+				)
+				(hide yes)
+			)
+		)
+		(pin "4"
+		)
+		(pin "3"
+		)
+		(pin "1"
+		)
+		(pin "2"
+		)
+		(instances
+			(project "l3"
+				(path "/1b1408da-cc6a-469f-a506-e797247b3ac8/65597bc7-5aaa-4f27-9286-e75eee7edae8"
+					(reference "J303")
+					(unit 1)
+				)
+			)
+		)
+	)
+	(symbol
 		(lib_id "power:GNDREF")
 		(at 113.03 93.98 0)
@@
 	)
 	(symbol
-		(lib_id "Connector_Generic:Conn_01x04")
-		(at 68.58 173.99 180)
+		(lib_id "power:GNDREF")
+		(at 92.71 172.72 0)
 		(unit 1)
 		(exclude_from_sim no)
@@
 		(dnp no)
 		(fields_autoplaced yes)
-		(property "Reference" "J303"
-			(at 68.58 162.56 0)
+		(property "Reference" "#PWR0362"
+			(at 92.71 179.07 0)
 			(effects
 				(font
 					(size 1.27 1.27)
 				)
+				(hide yes)
 			)
 		)
-		(property "Value" "Conn_01x04"
-			(at 68.58 165.1 0)
+		(property "Value" "GNDREF"
+			(at 92.71 177.8 0)
 			(effects
 				(font
 					(size 1.27 1.27)
 				)
+				(hide yes)
 			)
 		)
 		(property "Footprint" ""
-			(at 68.58 173.99 0)
+			(at 92.71 172.72 0)
 			(effects
 				(font
@@
 			)
 		)
-		(property "Datasheet" "~"
-			(at 68.58 173.99 0)
+		(property "Datasheet" ""
+			(at 92.71 172.72 0)
 			(effects
 				(font
@@
 			)
 		)
-		(property "Description" "Generic connector, single row, 01x04, script generated (kicad-library-utils/schlib/autogen/connector/)"
-			(at 68.58 173.99 0)
+		(property "Description" "Power symbol creates a global label with name \"GNDREF\" , reference supply ground"
+			(at 92.71 172.72 0)
 			(effects
 				(font
@@
 		(pin "1"
 		)
-		(pin "2"
-		)
-		(pin "3"
-		)
-		(pin "4"
-		)
 		(instances
 			(project "l3"
 				(path "/1b1408da-cc6a-469f-a506-e797247b3ac8/65597bc7-5aaa-4f27-9286-e75eee7edae8"
-					(reference "J303")
+					(reference "#PWR0362")
 					(unit 1)
 				)
@@
 					(unit 1)
 				)
+			)
+		)
+	)
+	(symbol
+		(lib_id "power:+3V3")
+		(at 92.71 165.1 0)
+		(unit 1)
+		(exclude_from_sim no)
+		(in_bom yes)
+		(on_board yes)
+		(dnp no)
+		(fields_autoplaced yes)
+		(property "Reference" "#PWR0361"
+			(at 92.71 168.91 0)
+			(effects
+				(font
+					(size 1.27 1.27)
+				)
+				(hide yes)
+			)
+		)
+		(property "Value" "+3V3 FILT"
+			(at 92.71 160.02 0)
+			(effects
+				(font
+					(size 1.27 1.27)
+				)
+			)
+		)
+		(property "Footprint" ""
+			(at 92.71 165.1 0)
+			(effects
+				(font
+					(size 1.27 1.27)
+				)
+				(hide yes)
+			)
+		)
+		(property "Datasheet" ""
+			(at 92.71 165.1 0)
+			(effects
+				(font
+					(size 1.27 1.27)
+				)
+				(hide yes)
+			)
+		)
+		(property "Description" "Power symbol creates a global label with name \"+3V3\""
+			(at 92.71 165.1 0)
+			(effects
+				(font
+					(size 1.27 1.27)
+				)
+				(hide yes)
+			)
+		)
+		(pin "1"
+		)
+		(instances
+			(project "l3"
+				(path "/1b1408da-cc6a-469f-a506-e797247b3ac8/65597bc7-5aaa-4f27-9286-e75eee7edae8"
+					(reference "#PWR0361")
+					(unit 1)
+				)

Commit message: i messed up
Connections:
- net +3V3 FILT: no longer C307.1, U301.22 (VCAP1)
- new net: C307.1, U301.22 (VCAP1)
Changed lines of the file:
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@@
-	)
-	(junction
-		(at 137.16 43.18)
-		(diameter 0)
-		(color 0 0 0 0)
 	)
 	(junction
@@
 		(pts
 			(xy 62.23 43.18) (xy 73.66 43.18)
-		)
-		(stroke
-			(width 0)
-			(type default)
-		)
-	)
-	(wire
-		(pts
-			(xy 137.16 40.64) (xy 137.16 43.18)
 		)
 		(stroke
@@
 	(label "IMU SWDIO"
 		(at 76.2 167.64 0)
-		(fields_autoplaced yes)
 		(effects
 			(font
@@
 	(label "IMU SWCLK"
 		(at 76.2 170.18 0)
-		(fields_autoplaced yes)
 		(effects
 			(font
@@
 	(label "IMU RST"
 		(at 171.45 138.43 180)
-		(fields_autoplaced yes)
 		(effects
 			(font
@@
 	(label "IMU MISO"
 		(at 220.98 57.15 0)
-		(fields_autoplaced yes)
 		(effects
 			(font
@@
 	(label "IMU OSC OUT"
 		(at 49.53 78.74 0)
-		(fields_autoplaced yes)
 		(effects
 			(font
@@
 	(label "IMU INT"
 		(at 220.98 72.39 0)
-		(fields_autoplaced yes)
 		(effects
 			(font
@@
 	(label "IMU BOOT0"
 		(at 99.06 81.28 0)
-		(fields_autoplaced yes)
 		(effects
 			(font
@@
 	(label "IMU SCK"
 		(at 171.45 146.05 180)
-		(fields_autoplaced yes)
 		(effects
 			(font
@@
 	(label "IMU OSC IN"
 		(at 49.53 76.2 0)
-		(fields_autoplaced yes)
 		(effects
 			(font
@@
 	(label "IMU SCK"
 		(at 220.98 62.23 0)
-		(fields_autoplaced yes)
 		(effects
 			(font
@@
 	(label "IMU NSS"
 		(at 171.45 143.51 180)
-		(fields_autoplaced yes)
 		(effects
 			(font
@@
 	(label "IMU NSS"
 		(at 220.98 67.31 0)
-		(fields_autoplaced yes)
 		(effects
 			(font
@@
 	(label "IMU SWDIO"
 		(at 39.37 146.05 0)
-		(fields_autoplaced yes)
 		(effects
 			(font
@@
 	(label "IMU MISO"
 		(at 171.45 148.59 180)
-		(fields_autoplaced yes)
 		(effects
 			(font
@@
 	(label "IMU MOSI"
 		(at 220.98 52.07 0)
-		(fields_autoplaced yes)
 		(effects
 			(font
@@
 	(label "IMU RST"
 		(at 99.06 76.2 0)
-		(fields_autoplaced yes)
 		(effects
 			(font
@@
 	(label "IMU RST"
 		(at 269.24 67.31 180)
-		(fields_autoplaced yes)
 		(effects
 			(font
@@
 	(label "IMU SWCLK"
 		(at 39.37 148.59 0)
-		(fields_autoplaced yes)
 		(effects
 			(font
@@
 	(label "IMU MOSI"
 		(at 171.45 151.13 180)
-		(fields_autoplaced yes)
 		(effects
 			(font
@@
 	(label "IMU INT"
 		(at 171.45 140.97 180)
-		(fields_autoplaced yes)
 		(effects
 			(font
@@
 	(label "IMU LED"
 		(at 39.37 151.13 0)
-		(fields_autoplaced yes)
 		(effects
 			(font
@@
 		(shape input)
 		(at 38.1 130.81 180)
-		(fields_autoplaced yes)
 		(effects
 			(font
@@
 		(shape input)
 		(at 38.1 125.73 180)
-		(fields_autoplaced yes)
 		(effects
 			(font
@@
 		(shape output)
 		(at 38.1 128.27 180)
-		(fields_autoplaced yes)
 		(effects
 			(font
@@
 		(shape input)
 		(at 38.1 123.19 180)
-		(fields_autoplaced yes)
 		(effects
 			(font
@@
 				)
 			)
-		)
-	)
-	(symbol
-		(lib_id "power:+3V3")
-		(at 137.16 40.64 0)
-		(unit 1)
-		(exclude_from_sim no)
-		(in_bom yes)
-		(on_board yes)
-		(dnp no)
-		(fields_autoplaced yes)
-		(property "Reference" "#PWR0303"
-			(at 137.16 44.45 0)
-			(effects
-				(font
-					(size 1.27 1.27)
-				)
-				(hide yes)
-			)
-		)
-		(property "Value" "+3V3 FILT"
-			(at 137.16 35.56 0)
-			(effects
-				(font
-					(size 1.27 1.27)
-				)
-			)
-		)
-		(property "Footprint" ""
-			(at 137.16 40.64 0)
-			(effects
-				(font
-					(size 1.27 1.27)
-				)
-				(hide yes)
-			)
-		)
-		(property "Datasheet" ""
-			(at 137.16 40.64 0)
-			(effects
-				(font
-					(size 1.27 1.27)
-				)
-				(hide yes)
-			)
-		)
-		(property "Description" "Power symbol creates a global label with name \"+3V3\""
-			(at 137.16 40.64 0)
-			(effects
-				(font
-					(size 1.27 1.27)
-				)
-				(hide yes)
-			)
-		)
-		(pin "1"
-		)
-		(instances
-			(project "l3"
-				(path "/1b1408da-cc6a-469f-a506-e797247b3ac8/65597bc7-5aaa-4f27-9286-e75eee7edae8"
-					(reference "#PWR0303")
-					(unit 1)
-				)
-			)

Commit message: nerv
Parts:
- C301, C307, C308: value 2u2 -> 2U2
- C302, C303, C304, C305, C306, C309: value 0u1 -> 0U1
- C310: value C -> 0U1
- R303: value R -> 10K
Other:
- moved on the sheet: C307
Changed lines of the file:
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@@
 (kicad_sch
-	(version 20231120)
+	(version 20250114)
 	(generator "eeschema")
-	(generator_version "8.0")
+	(generator_version "9.0")
 	(paper "A4")
+	(rectangle
+		(start 190.5 27.94)
+		(end 283.21 80.01)
+		(stroke
+			(width 0)
+			(type default)
+		)
+		(fill
+			(type none)
+		)
+	)
+	(rectangle
+		(start 13.97 25.4)
+		(end 175.26 177.8)
+		(stroke
+			(width 0)
+			(type default)
+		)
+		(fill
+			(type none)
+		)
+	)
 	(junction
 		(at 135.89 143.51)
@@
 	(wire
 		(pts
-			(xy 137.16 43.18) (xy 137.16 45.72)
+			(xy 137.16 43.18) (xy 137.16 46.99)
 		)
 		(stroke
@@
 	(wire
 		(pts
-			(xy 137.16 53.34) (xy 137.16 57.15)
+			(xy 137.16 54.61) (xy 137.16 58.42)
 		)
 		(stroke
@@
 		)
 	)
-	(rectangle
-		(start 190.5 27.94)
-		(end 283.21 80.01)
-		(stroke
-			(width 0)
-			(type default)
-		)
-		(fill
-			(type none)
-		)
-	)
-	(rectangle
-		(start 13.97 25.4)
-		(end 175.26 177.8)
-		(stroke
-			(width 0)
-			(type default)
-		)
-		(fill
-			(type none)
-		)
-	)
 	(label "IMU SWDIO"
 		(at 76.2 167.64 0)
@@
 	(symbol
 		(lib_id "Device:C")
-		(at 137.16 49.53 0)
+		(at 137.16 50.8 0)
 		(unit 1)
 		(exclude_from_sim no)
@@
 		(dnp no)
 		(property "Reference" "C307"
-			(at 140.97 48.2599 0)
+			(at 140.97 49.5299 0)
 			(effects
 				(font
@@
 			)
 		)
-		(property "Value" "2u2"
-			(at 140.97 50.7999 0)
+		(property "Value" "2U2"
+			(at 140.97 52.0699 0)
 			(effects
 				(font
@@
 		)
 		(property "Footprint" "Library:cap0603"
-			(at 138.1252 53.34 0)
+			(at 138.1252 54.61 0)
 			(effects
 				(font
@@
 		)
 		(property "Datasheet" "~"
-			(at 137.16 49.53 0)
+			(at 137.16 50.8 0)
 			(effects
 				(font
@@
 		)
 		(property "Description" "Unpolarized capacitor"
-			(at 137.16 49.53 0)
+			(at 137.16 50.8 0)
 			(effects
 				(font
@@
 	(symbol
 		(lib_id "power:GNDREF")
-		(at 137.16 57.15 0)
+		(at 137.16 58.42 0)
 		(unit 1)
 		(exclude_from_sim no)
@@
 		(fields_autoplaced yes)
 		(property "Reference" "#PWR0305"
-			(at 137.16 63.5 0)
+			(at 137.16 64.77 0)
 			(effects
 				(font
@@
 		)
 		(property "Value" "GNDREF"
-			(at 137.16 62.23 0)
+			(at 137.16 63.5 0)
 			(effects
 				(font
@@
 		)
 		(property "Footprint" ""
-			(at 137.16 57.15 0)
+			(at 137.16 58.42 0)
 			(effects
 				(font
@@
 		)
 		(property "Datasheet" ""
-			(at 137.16 57.15 0)
+			(at 137.16 58.42 0)
 			(effects
 				(font
@@
 		)
 		(property "Description" "Power symbol creates a global label with name \"GNDREF\" , reference supply ground"
-			(at 137.16 57.15 0)
+			(at 137.16 58.42 0)
 			(effects
 				(font
@@
 			)
 		)
-		(property "Value" "C"
+		(property "Value" "0U1"
 			(at 143.51 83.8199 0)
 			(effects
@@
 			)
 		)
-		(property "Value" "0u1"
+		(property "Value" "0U1"
 			(at 88.9 50.7999 0)
 			(effects
@@
 			)
 		)
-		(property "Value" "0u1"
+		(property "Value" "0U1"
 			(at 100.33 50.7999 0)
 			(effects
@@
 			)
 		)
-		(property "Value" "0u1"
+		(property "Value" "0U1"
 			(at 66.04 50.7999 0)
 			(effects
@@
 			)
 		)
-		(property "Value" "0u1"
+		(property "Value" "0U1"
 			(at 213.36 54.6099 0)
 			(effects
@@
 			)
 		)
-		(property "Value" "0u1"
+		(property "Value" "0U1"
 			(at 77.47 50.7999 0)
 			(effects
@@
 			)
 		)
-		(property "Value" "2u2"
+		(property "Value" "2U2"
 			(at 201.93 54.6099 0)
 			(effects
@@
 			)
 		)
-		(property "Value" "0u1"
+		(property "Value" "0U1"
 			(at 54.61 50.7999 0)
 			(effects
@@
 			)
 		)
-		(property "Value" "2u2"
+		(property "Value" "2U2"
 			(at 43.18 50.7999 0)
 			(effects
@@
 			)
 		)
-		(property "Value" "R"
+		(property "Value" "10K"
 			(at 115.57 88.8999 0)
 			(effects
