File: processingUnit/l3.kicad_sch (KiCad schematic)
At the start: 17 parts, among them J302 M1, J303 Conn_01x06, J304 Conn_01x06, J305 Conn_01x06, J306 M1, J307 M1, J308 M1, U303 SN74LVC2G04, U304 SN74LVC2G04

Commit message: L3
Connections:
- net ENC/M1 DIR: now also U303.3; no longer U303.1
- net ENC/M2 DIR: now also U303.1; no longer U303.3
- net driver/M1 IN B: now also U303.4; no longer U303.6
- net driver/M2 IN B: now also U303.6; no longer U303.4

Commit message: L3
Connections:
- net ENC/M3 DIR: now also U304.3; no longer U304.1
- net ENC/M4 DIR: now also U304.1; no longer U304.3
- net driver/M3 IN B: now also U304.4; no longer U304.6
- net driver/M4 IN B: now also U304.6; no longer U304.4
Other:
- sheet IMU ports: added IMU STM NSS; removed IMU NSS
- sheet tnsy ports: added IMU STM NSS; removed IMU NSS

Commit message: L3
Parts:
- removed J303, J304, J305: Conn_01x06, symbol Connector_Generic:Conn_01x06
Changed lines of the file:
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@@
-	)
-	(symbol
-		(lib_id "Connector_Generic:Conn_01x06")
-		(at 99.06 161.29 0)
-		(mirror y)
-		(unit 1)
-		(exclude_from_sim no)
-		(in_bom yes)
-		(on_board yes)
-		(dnp no)
-		(fields_autoplaced yes)
-		(property "Reference" "J305"
-			(at 99.06 149.86 0)
-			(effects
-				(font
-					(size 1.27 1.27)
-				)
-			)
-		)
-		(property "Value" "Conn_01x06"
-			(at 99.06 152.4 0)
-			(effects
-				(font
-					(size 1.27 1.27)
-				)
-			)
-		)
-		(property "Footprint" ""
-			(at 99.06 161.29 0)
-			(effects
-				(font
-					(size 1.27 1.27)
-				)
-				(hide yes)
-			)
-		)
-		(property "Datasheet" "~"
-			(at 99.06 161.29 0)
-			(effects
-				(font
-					(size 1.27 1.27)
-				)
-				(hide yes)
-			)
-		)
-		(property "Description" "Generic connector, single row, 01x06, script generated (kicad-library-utils/schlib/autogen/connector/)"
-			(at 99.06 161.29 0)
-			(effects
-				(font
-					(size 1.27 1.27)
-				)
-				(hide yes)
-			)
-		)
-		(pin "2"
-		)
-		(pin "4"
-		)
-		(pin "1"
-		)
-		(pin "3"
-		)
-		(pin "6"
-		)
-		(pin "5"
-		)
-		(instances
-			(project "l3"
-				(path "/1b1408da-cc6a-469f-a506-e797247b3ac8"
-					(reference "J305")
-					(unit 1)
-				)
-			)
-		)
 	)
 	(symbol
@@
 					(unit 1)
 				)
-			)
-		)
-	)
-	(symbol
-		(lib_id "Connector_Generic:Conn_01x06")
-		(at 81.28 161.29 0)
-		(mirror y)
-		(unit 1)
-		(exclude_from_sim no)
-		(in_bom yes)
-		(on_board yes)
-		(dnp no)
-		(fields_autoplaced yes)
-		(property "Reference" "J304"
-			(at 81.28 149.86 0)
-			(effects
-				(font
-					(size 1.27 1.27)
-				)
-			)
-		)
-		(property "Value" "Conn_01x06"
-			(at 81.28 152.4 0)
-			(effects
-				(font
-					(size 1.27 1.27)
-				)
-			)
-		)
-		(property "Footprint" ""
-			(at 81.28 161.29 0)
-			(effects
-				(font
-					(size 1.27 1.27)
-				)
-				(hide yes)
-			)
-		)
-		(property "Datasheet" "~"
-			(at 81.28 161.29 0)
-			(effects
-				(font
-					(size 1.27 1.27)
-				)
-				(hide yes)
-			)
-		)
-		(property "Description" "Generic connector, single row, 01x06, script generated (kicad-library-utils/schlib/autogen/connector/)"
-			(at 81.28 161.29 0)
-			(effects
-				(font
-					(size 1.27 1.27)
-				)
-				(hide yes)
-			)
-		)
-		(pin "2"
-		)
-		(pin "4"
-		)
-		(pin "1"
-		)
-		(pin "3"
-		)
-		(pin "6"
-		)
-		(pin "5"
-		)
-		(instances
-			(project "l3"
-				(path "/1b1408da-cc6a-469f-a506-e797247b3ac8"
-					(reference "J304")
-					(unit 1)
-				)
-			)
-		)
-	)
-	(symbol
-		(lib_id "Connector_Generic:Conn_01x06")
-		(at 62.23 161.29 0)
-		(mirror y)
-		(unit 1)
-		(exclude_from_sim no)
-		(in_bom yes)
-		(on_board yes)
-		(dnp no)
-		(fields_autoplaced yes)
-		(property "Reference" "J303"
-			(at 62.23 149.86 0)
-			(effects
-				(font
-					(size 1.27 1.27)
-				)
-			)
-		)
-		(property "Value" "Conn_01x06"
-			(at 62.23 152.4 0)
-			(effects
-				(font
-					(size 1.27 1.27)
-				)
-			)
-		)
-		(property "Footprint" ""
-			(at 62.23 161.29 0)
-			(effects
-				(font
-					(size 1.27 1.27)
-				)
-				(hide yes)
-			)
-		)
-		(property "Datasheet" "~"
-			(at 62.23 161.29 0)
-			(effects
-				(font
-					(size 1.27 1.27)
-				)
-				(hide yes)
-			)
-		)
-		(property "Description" "Generic connector, single row, 01x06, script generated (kicad-library-utils/schlib/autogen/connector/)"
-			(at 62.23 161.29 0)
-			(effects
-				(font
-					(size 1.27 1.27)
-				)
-				(hide yes)
-			)
-		)
-		(pin "2"
-		)
-		(pin "4"
-		)
-		(pin "1"
-		)
-		(pin "3"
-		)
-		(pin "6"
-		)
-		(pin "5"
-		)
-		(instances
-			(project "l3"
-				(path "/1b1408da-cc6a-469f-a506-e797247b3ac8"
-					(reference "J303")
-					(unit 1)
-				)

Commit message: L3
Other:
- sheet connectors renamed Connectors and MTH
- sheet driver renamed Motor Driver
- sheet tnsy renamed Teensy and Bluetooth
Changed lines of the file:
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@@
 			(color 0 0 0 0.0000)
 		)
-		(property "Sheetname" "connectors"
+		(property "Sheetname" "Connectors and MTH"
 			(at 50.8 76.7584 0)
 			(effects
@@
 			(color 0 0 0 0.0000)
 		)
-		(property "Sheetname" "driver"
+		(property "Sheetname" "Motor Driver"
 			(at 214.63 34.8484 0)
 			(effects
@@
 			(color 0 0 0 0.0000)
 		)
-		(property "Sheetname" "tnsy"
+		(property "Sheetname" "Teensy and Bluetooth"
 			(at 63.5 34.8484 0)
 			(effects

Commit message: pull up
Parts:
- added R355, R356, R357, R358, R359: 10K, Library:res0603, symbol Device:R
Connections:
- net ENC/ENC NSS: now also R355.2
- net ENC/TNSY MISO: now also R358.2
- net ENC/TNSY MOSI: now also R359.2
- net ENC/TNSY SCK: now also R357.2
- net IMU/IMU STM NSS: now also R356.2
- new net +3V3 FILT: R355.1, R356.1, R357.1, R358.1, R359.1

Commit message: Damn u SPI
Parts:
- removed R355, R356, R357, R358, R359: 10K, Library:res0603, symbol Device:R
Other:
- sheet ENC ports: added ENC RX, ENC TX; removed ENC NSS, TNSY MISO, TNSY MOSI, TNSY SCK
- sheet IMU ports: added IMU RX, IMU TX; removed IMU STM NSS, TNSY MISO, TNSY MOSI, TNSY SCK
- sheet Teensy and Bluetooth ports: added TNSY ENC RX, TNSY ENC TX, TNSY IMU RX, TNSY IMU TX, TNSY L3 RX, TNSY L3 TX; removed BT RX, BT TX, ENC NSS, IMU STM NSS, TNSY MISO, TNSY MOSI, TNSY SCK
