File: processingUnit/l3.kicad_sch (KiCad schematic)
At the start: 14 parts, among them J302 M1, J306 M1, J307 M1, J308 M1, U303 SN74LVC2G04, U304 SN74LVC2G04

Commit message: Processing Unit
Other:
- sheet Teensy and Bluetooth ports: added ENC RX, ENC TX, IMU RX, IMU TX, L3 RX, L3 TX; removed TNSY ENC RX, TNSY ENC TX, TNSY IMU RX, TNSY IMU TX, TNSY L3 RX, TNSY L3 TX
Changed lines of the file:
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@@
 			)
 		)
-		(pin "TNSY ENC TX" output
+		(pin "ENC TX" output
 			(at 50.8 57.15 0)
 			(effects
@@
 			)
 		)
-		(pin "TNSY IMU TX" output
+		(pin "IMU TX" output
 			(at 50.8 52.07 0)
 			(effects
@@
 			)
 		)
-		(pin "TNSY IMU RX" input
+		(pin "IMU RX" input
 			(at 50.8 54.5467 0)
 			(effects
@@
 			)
 		)
-		(pin "TNSY ENC RX" input
+		(pin "ENC RX" input
 			(at 50.8 59.69 0)
 			(effects
@@
 			)
 		)
-		(pin "TNSY L3 RX" input
+		(pin "L3 RX" input
 			(at 50.8 49.2141 0)
 			(effects
@@
 			)
 		)
-		(pin "TNSY L3 TX" output
+		(pin "L3 TX" output
 			(at 50.8 46.3642 0)
 			(effects

Commit message: sch process
Other:
- removed sheet IMU
Changed lines of the file:
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@@
 	(wire
 		(pts
-			(xy 50.8 54.5467) (xy 127 54.5467)
-		)
-		(stroke
-			(width 0)
-			(type default)
-		)
-	)
-	(wire
-		(pts
 			(xy 191.77 49.53) (xy 189.23 49.53)
 		)
@@
 	(wire
 		(pts
-			(xy 127 54.5467) (xy 127 54.61)
-		)
-		(stroke
-			(width 0)
-			(type default)
-		)
-	)
-	(wire
-		(pts
 			(xy 274.32 71.12) (xy 237.49 71.12)
 		)
@@
 	(wire
 		(pts
-			(xy 50.8 52.07) (xy 127 52.07)
-		)
-		(stroke
-			(width 0)
-			(type default)
-		)
-	)
-	(wire
-		(pts
 			(xy 266.7 113.03) (xy 266.7 109.22)
 		)
@@
 				)
 			)
-		)
-	)
-	(sheet
-		(at 127 45.72)
-		(size 15.24 15.24)
-		(exclude_from_sim no)
-		(in_bom yes)
-		(on_board yes)
-		(dnp no)
-		(fields_autoplaced yes)
-		(stroke
-			(width 0.1524)
-			(type solid)
-		)
-		(fill
-			(color 0 0 0 0.0000)
-		)
-		(property "Sheetname" "IMU"
-			(at 127 45.0084 0)
-			(effects
-				(font
-					(size 1.27 1.27)
-				)
-				(justify left bottom)
-			)
-		)
-		(property "Sheetfile" "imu.kicad_sch"
-			(at 127 61.5446 0)
-			(effects
-				(font
-					(size 1.27 1.27)
-				)
-				(justify left top)
-				(hide yes)
-			)
-		)
-		(pin "IMU TX" output
-			(at 127 54.61 180)
-			(effects
-				(font
-					(size 1.27 1.27)
-				)
-				(justify left)
-			)
-		)
-		(pin "IMU RX" input
-			(at 127 52.07 180)
-			(effects
-				(font
-					(size 1.27 1.27)
-				)
-				(justify left)
-			)
-		)
-		(instances
-			(project "l3"
-				(path "/1b1408da-cc6a-469f-a506-e797247b3ac8"
-					(page "4")
-				)
-			)

Commit message: l3 might redo
Connections:
- net +5V FILT: no longer U303.5 (VCC), U304.5 (VCC)
- new net +3V3 FILT: U303.5 (VCC), U304.5 (VCC)
Other:
- sheet Connectors and MTH ports: added ESC 1, ESC 2, FLAG, GATE RX, GATE TX, KICK SIG, L3 RX, L3 TX, LIGHT RX, LIGHT TX; removed none
- sheet Teensy and Bluetooth ports: added ESC 1, ESC 2, FLAG, GATE RX, GATE TX, KICK SIG, LIGHT RX, LIGHT TX; removed IMU RX, IMU TX, L1 RX, L1 TX
- note added: "Serial is already swapped in the connectors"

Commit message: l3 might redo
Parts:
- removed J302, J306, J307, J308: M1, Connector_JST:JST_PH_B6B-PH-K_1x06_P2.00mm_Vertical, symbol Connector_Generic:Conn_01x06
- removed R343, R344, R345, R346, R347, R348, R349, R350: 1k, Library:res0603, symbol Device:R
- renumbered U303 to U701, U304 to U702
Connections:
- net ENC/M3 DIR: no longer U702.3
- new net Motor Driver/M3 IN A: U702.3
Other:
- sheet Teensy and Bluetooth renamed Teensy
- added sheet Motor Connector (motor-connector.kicad_sch)

Commit message: l3 might redo
Parts:
- renumbered U701 to U601, U702 to U602
Changed lines of the file:
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@@
 		(dnp no)
 		(fields_autoplaced yes)
-		(property "Reference" "U701"
+		(property "Reference" "U601"
 			(at 199.39 67.31 0)
 			(effects
@@
 			(project "l3"
 				(path "/1b1408da-cc6a-469f-a506-e797247b3ac8"
-					(reference "U701")
+					(reference "U601")
 					(unit 1)
 				)
@@
 		(dnp no)
 		(fields_autoplaced yes)
-		(property "Reference" "U702"
+		(property "Reference" "U602"
 			(at 129.54 132.08 0)
 			(effects
@@
 			(project "l3"
 				(path "/1b1408da-cc6a-469f-a506-e797247b3ac8"
-					(reference "U702")
+					(reference "U602")
 					(unit 3)
 				)
@@
 		(dnp no)
 		(fields_autoplaced yes)
-		(property "Reference" "U702"
+		(property "Reference" "U602"
 			(at 199.39 121.92 0)
 			(effects
@@
 			(project "l3"
 				(path "/1b1408da-cc6a-469f-a506-e797247b3ac8"
-					(reference "U702")
+					(reference "U602")
 					(unit 1)
 				)
@@
 		(dnp no)
 		(fields_autoplaced yes)
-		(property "Reference" "U702"
+		(property "Reference" "U602"
 			(at 199.39 93.98 0)
 			(effects
@@
 			(project "l3"
 				(path "/1b1408da-cc6a-469f-a506-e797247b3ac8"
-					(reference "U702")
+					(reference "U602")
 					(unit 2)
 				)
@@
 		(dnp no)
 		(fields_autoplaced yes)
-		(property "Reference" "U701"
+		(property "Reference" "U601"
 			(at 129.54 116.84 0)
 			(effects
@@
 			(project "l3"
 				(path "/1b1408da-cc6a-469f-a506-e797247b3ac8"
-					(reference "U701")
+					(reference "U601")
 					(unit 3)
 				)
@@
 		(dnp no)
 		(fields_autoplaced yes)
-		(property "Reference" "U701"
+		(property "Reference" "U601"
 			(at 199.39 40.64 0)
 			(effects
@@
 			(project "l3"
 				(path "/1b1408da-cc6a-469f-a506-e797247b3ac8"
-					(reference "U701")
+					(reference "U601")
 					(unit 2)
 				)

Commit message: drivers
Connections:
- net Motor Driver/M3 IN A is gone; now on net ENC/M3 DIR: U602.3
Changed lines of the file:
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@@
+	)
+	(junction
+		(at 189.23 91.44)
+		(diameter 0)
+		(color 0 0 0 0)
 	)
 	(junction
@@
 		)
 		(stroke
+			(width 0)
+			(type default)
+		)
+	)
+	(wire
+		(pts
+			(xy 142.24 91.44) (xy 189.23 91.44)
+		)
+		(stroke

Commit message: switch position
Other:
- sheet Connectors and MTH ports: added FLAG 2; removed GATE RX, GATE TX
- sheet Teensy ports: added FLAG 2; removed GATE RX, GATE TX
Changed lines of the file:
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@@
+	(wire
+		(pts
+			(xy 189.23 130.81) (xy 189.23 119.38)
+		)
+		(stroke
+			(width 0)
+			(type default)
+		)
+	)
+	(wire
+		(pts
+			(xy 189.23 49.53) (xy 189.23 38.1)
+		)
+		(stroke
+			(width 0)
+			(type default)
+		)
+	)
+	(wire
+		(pts
+			(xy 189.23 38.1) (xy 214.63 38.1)
+		)
+		(stroke
+			(width 0)
+			(type default)
+		)
+	)
+	(wire
+		(pts
+			(xy 142.24 81.28) (xy 184.15 81.28)
+		)
+		(stroke
+			(width 0)
+			(type default)
+		)
+	)
+	(wire
+		(pts
+			(xy 50.8 60.96) (xy 104.14 60.96)
+		)
+		(stroke
+			(width 0)
+			(type default)
+		)
+	)
 	(wire
 		(pts
@@
 	(wire
 		(pts
-			(xy 189.23 130.81) (xy 189.23 119.38)
-		)
-		(stroke
-			(width 0)
-			(type default)
-		)
-	)
-	(wire
-		(pts
-			(xy 189.23 49.53) (xy 189.23 38.1)
-		)
-		(stroke
-			(width 0)
-			(type default)
-		)
-	)
-	(wire
-		(pts
-			(xy 189.23 38.1) (xy 214.63 38.1)
-		)
-		(stroke
-			(width 0)
-			(type default)
-		)
-	)
-	(wire
-		(pts
-			(xy 142.24 81.28) (xy 184.15 81.28)
-		)
-		(stroke
-			(width 0)
-			(type default)
-		)
-	)
-	(wire
-		(pts
-			(xy 50.8 60.96) (xy 104.14 60.96)
-		)
-		(stroke
-			(width 0)
-			(type default)
-		)
-	)
-	(wire
-		(pts
-			(xy 50.8 41.91) (xy 104.14 41.91)
-		)
-		(stroke
-			(width 0)
-			(type default)
-		)
-	)
-	(wire
-		(pts
 			(xy 207.01 130.81) (xy 214.63 130.81)
 		)
@@
 	(wire
 		(pts
+			(xy 237.49 101.6) (xy 243.84 101.6)
+		)
+		(stroke
+			(width 0)
+			(type default)
+		)
+	)
+	(wire
+		(pts
+			(xy 167.64 38.1) (xy 189.23 38.1)
+		)
+		(stroke
+			(width 0)
+			(type default)
+		)
+	)
+	(wire
+		(pts
+			(xy 237.49 73.66) (xy 243.84 73.66)
+		)
+		(stroke
+			(width 0)
+			(type default)
+		)
+	)
+	(wire
+		(pts
 			(xy 50.8 57.15) (xy 104.14 57.15)
-		)
-		(stroke
-			(width 0)
-			(type default)
-		)
-	)
-	(wire
-		(pts
-			(xy 237.49 101.6) (xy 243.84 101.6)
-		)
-		(stroke
-			(width 0)
-			(type default)
-		)
-	)
-	(wire
-		(pts
-			(xy 167.64 38.1) (xy 189.23 38.1)
-		)
-		(stroke
-			(width 0)
-			(type default)
-		)
-	)
-	(wire
-		(pts
-			(xy 237.49 73.66) (xy 243.84 73.66)
 		)
 		(stroke
@@
 		)
 		(pin "FLAG" output
-			(at 104.14 41.91 180)
+			(at 104.14 54.61 180)
 			(effects
 				(font
@@
 			)
 		)
-		(pin "GATE RX" bidirectional
-			(at 104.14 57.15 180)
-			(effects
-				(font
-					(size 1.27 1.27)
-				)
-				(justify left)
-			)
-		)
 		(pin "LIGHT RX" bidirectional
 			(at 104.14 50.8 180)
@@
 			)
 		)
-		(pin "GATE TX" bidirectional
-			(at 104.14 54.61 180)
-			(effects
-				(font
-					(size 1.27 1.27)
-				)
-				(justify left)
-			)
-		)
 		(pin "LIGHT TX" bidirectional
 			(at 104.14 48.26 180)
+			(effects
+				(font
+					(size 1.27 1.27)
+				)
+				(justify left)
+			)
+		)
+		(pin "FLAG 2" output
+			(at 104.14 57.15 180)
 			(effects
 				(font
@@
 			)
 		)
-		(pin "GATE RX" bidirectional
-			(at 50.8 57.15 0)
-			(effects
-				(font
-					(size 1.27 1.27)
-				)
-				(justify right)
-			)
-		)
-		(pin "GATE TX" bidirectional
+		(pin "FLAG" input
 			(at 50.8 54.61 0)
-			(effects
-				(font
-					(size 1.27 1.27)
-				)
-				(justify right)
-			)
-		)
-		(pin "FLAG" input
-			(at 50.8 41.91 0)
 			(effects
 				(font
@@
 			(effects
 				(font
+					(size 1.27 1.27)
+				)
+				(justify right)
+			)
+		)
+		(pin "FLAG 2" input
+			(at 50.8 57.15 0)
+			(effects
+				(font

Commit message: step
Changed lines of the file:
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@@
 			)
 		)
-		(pin "L3 TX" output
+		(pin "L3 TX" input
 			(at 104.14 63.5 180)
 			(effects
@@
 			)
 		)
-		(pin "L3 RX" output
+		(pin "L3 RX" input
 			(at 50.8 60.96 0)
 			(effects
