File: processingUnit/driver.kicad_sch (KiCad schematic)
At the start: 49 parts

Commit message: L3 Schematic
Parts:
- gave numbers to parts that had none: 49

Commit message: Schematic L3
Connections:
- net GND is gone; now on net +3V3 FILT: SW302.2 (B)
- net +3V3 FILT: no longer R311.2, R312.2, R313.2, R314.2, R327.2, R328.2, R329.2, R330.2
- net GNDREF: now also R311.2, R312.2, R313.2, R314.2, R327.2, R328.2, R329.2, R330.2

Commit message: footprint
Parts:
- IC301, IC302, IC303, IC304: footprint 2024l2:VNH5019A-E -> Library:ST_MultiPowerSO-30
- R311, R312, R313, R314, R315, R316, R317, R318, R319, R320, R321, R322, R323, R324, R325, R326, R327, R328, R329, R330, R331, R332, R333, R334, R335, R336, R337, R338, R339, R340, R341, R342: footprint 2024l2:res0603 -> Library:res0603
Changed lines of the file:
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@@
 			)
 		)
-		(property "Footprint" "2024l2:res0603"
+		(property "Footprint" "Library:res0603"
 			(at 171.958 113.03 90)
 			(effects
@@
 			)
 		)
-		(property "Footprint" "2024l2:res0603"
+		(property "Footprint" "Library:res0603"
 			(at 69.85 124.968 90)
 			(effects
@@
 			)
 		)
-		(property "Footprint" "2024l2:res0603"
+		(property "Footprint" "Library:res0603"
 			(at 176.53 67.818 90)
 			(effects
@@
 			)
 		)
-		(property "Footprint" "2024l2:res0603"
+		(property "Footprint" "Library:res0603"
 			(at 176.53 135.382 90)
 			(effects
@@
 			)
 		)
-		(property "Footprint" "2024l2:res0603"
+		(property "Footprint" "Library:res0603"
 			(at 176.53 121.158 90)
 			(effects
@@
 			)
 		)
-		(property "Footprint" "2024l2:res0603"
+		(property "Footprint" "Library:res0603"
 			(at 69.85 130.302 90)
 			(effects
@@
 			)
 		)
-		(property "Footprint" "2024l2:res0603"
+		(property "Footprint" "Library:res0603"
 			(at 69.85 62.738 90)
 			(effects
@@
 			)
 		)
-		(property "Footprint" "2024l2:res0603"
+		(property "Footprint" "Library:res0603"
 			(at 165.862 143.51 90)
 			(effects
@@
 			)
 		)
-		(property "Footprint" "2024l2:res0603"
+		(property "Footprint" "Library:res0603"
 			(at 176.53 58.928 90)
 			(effects
@@
 			)
 		)
-		(property "Footprint" "2024l2:res0603"
+		(property "Footprint" "Library:res0603"
 			(at 176.53 130.048 90)
 			(effects
@@
 			)
 		)
-		(property "Footprint" "2024l2:VNH5019A-E"
+		(property "Footprint" "Library:ST_MultiPowerSO-30"
 			(at 78.74 149.86 0)
 			(effects
@@
 			)
 		)
-		(property "Footprint" "2024l2:VNH5019A-E"
+		(property "Footprint" "Library:ST_MultiPowerSO-30"
 			(at 185.42 149.86 0)
 			(effects
@@
 			)
 		)
-		(property "Footprint" "2024l2:res0603"
+		(property "Footprint" "Library:res0603"
 			(at 176.53 73.152 90)
 			(effects
@@
 			)
 		)
-		(property "Footprint" "2024l2:VNH5019A-E"
+		(property "Footprint" "Library:ST_MultiPowerSO-30"
 			(at 78.74 87.63 0)
 			(effects
@@
 			)
 		)
-		(property "Footprint" "2024l2:res0603"
+		(property "Footprint" "Library:res0603"
 			(at 59.182 143.51 90)
 			(effects
@@
 			)
 		)
-		(property "Footprint" "2024l2:res0603"
+		(property "Footprint" "Library:res0603"
 			(at 65.278 113.03 90)
 			(effects
@@
 			)
 		)
-		(property "Footprint" "2024l2:VNH5019A-E"
+		(property "Footprint" "Library:ST_MultiPowerSO-30"
 			(at 185.42 87.63 0)
 			(effects
@@
 			)
 		)
-		(property "Footprint" "2024l2:res0603"
+		(property "Footprint" "Library:res0603"
 			(at 69.85 58.928 90)
 			(effects
@@
 			)
 		)
-		(property "Footprint" "2024l2:res0603"
+		(property "Footprint" "Library:res0603"
 			(at 165.862 81.28 90)
 			(effects
@@
 			)
 		)
-		(property "Footprint" "2024l2:res0603"
+		(property "Footprint" "Library:res0603"
 			(at 56.642 113.03 90)
 			(effects
@@
 			)
 		)
-		(property "Footprint" "2024l2:res0603"
+		(property "Footprint" "Library:res0603"
 			(at 69.85 68.072 90)
 			(effects
@@
 			)
 		)
-		(property "Footprint" "2024l2:res0603"
+		(property "Footprint" "Library:res0603"
 			(at 56.642 50.8 90)
 			(effects
@@
 			)
 		)
-		(property "Footprint" "2024l2:res0603"
+		(property "Footprint" "Library:res0603"
 			(at 59.182 81.28 90)
 			(effects
@@
 			)
 		)
-		(property "Footprint" "2024l2:res0603"
+		(property "Footprint" "Library:res0603"
 			(at 69.85 73.152 90)
 			(effects
@@
 			)
 		)
-		(property "Footprint" "2024l2:res0603"
+		(property "Footprint" "Library:res0603"
 			(at 171.958 50.8 90)
 			(effects
@@
 			)
 		)
-		(property "Footprint" "2024l2:res0603"
+		(property "Footprint" "Library:res0603"
 			(at 65.278 50.8 90)
 			(effects
@@
 			)
 		)
-		(property "Footprint" "2024l2:res0603"
+		(property "Footprint" "Library:res0603"
 			(at 69.85 135.382 90)
 			(effects
@@
 			)
 		)
-		(property "Footprint" "2024l2:res0603"
+		(property "Footprint" "Library:res0603"
 			(at 176.53 130.302 90)
 			(effects
@@
 			)
 		)
-		(property "Footprint" "2024l2:res0603"
+		(property "Footprint" "Library:res0603"
 			(at 163.322 50.8 90)
 			(effects
@@
 			)
 		)
-		(property "Footprint" "2024l2:res0603"
+		(property "Footprint" "Library:res0603"
 			(at 69.85 130.048 90)
 			(effects
@@
 			)
 		)
-		(property "Footprint" "2024l2:res0603"
+		(property "Footprint" "Library:res0603"
 			(at 176.53 124.968 90)
 			(effects
@@
 			)
 		)
-		(property "Footprint" "2024l2:res0603"
+		(property "Footprint" "Library:res0603"
 			(at 176.53 62.738 90)
 			(effects
@@
 			)
 		)
-		(property "Footprint" "2024l2:res0603"
+		(property "Footprint" "Library:res0603"
 			(at 176.53 68.072 90)
 			(effects
@@
 			)
 		)
-		(property "Footprint" "2024l2:res0603"
+		(property "Footprint" "Library:res0603"
 			(at 69.85 67.818 90)
 			(effects
@@
 			)
 		)
-		(property "Footprint" "2024l2:res0603"
+		(property "Footprint" "Library:res0603"
 			(at 69.85 121.158 90)
 			(effects
@@
 			)
 		)
-		(property "Footprint" "2024l2:res0603"
+		(property "Footprint" "Library:res0603"
 			(at 163.322 113.03 90)
 			(effects

Commit message: L3
Parts:
- C311, C313, C315, C317: footprint 2024l2:CP_Radial_D8.0mm_P3.50mm -> Library:CP_Radial_D8.0mm_P3.50mm
- C312, C314, C316, C318: footprint 2024l2:cap0603 -> Library:cap0603
- Q301, Q302, Q303, Q304: footprint 2024l2:8-DFN (5x6) -> Library:8-DFN (5x6)
Changed lines of the file:
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@@
 			)
 		)
-		(property "Footprint" "2024l2:cap0603"
+		(property "Footprint" "Library:cap0603"
 			(at 236.5248 82.55 0)
 			(effects
@@
 			)
 		)
-		(property "Footprint" "2024l2:CP_Radial_D8.0mm_P3.50mm"
+		(property "Footprint" "Library:CP_Radial_D8.0mm_P3.50mm"
 			(at 119.0752 82.55 0)
 			(effects
@@
 			)
 		)
-		(property "Footprint" "2024l2:8-DFN (5x6)"
+		(property "Footprint" "Library:8-DFN (5x6)"
 			(at 231.14 58.42 90)
 			(effects
@@
 			)
 		)
-		(property "Footprint" "2024l2:CP_Radial_D8.0mm_P3.50mm"
+		(property "Footprint" "Library:CP_Radial_D8.0mm_P3.50mm"
 			(at 225.7552 144.78 0)
 			(effects
@@
 			)
 		)
-		(property "Footprint" "2024l2:8-DFN (5x6)"
+		(property "Footprint" "Library:8-DFN (5x6)"
 			(at 124.46 120.65 90)
 			(effects
@@
 			)
 		)
-		(property "Footprint" "2024l2:cap0603"
+		(property "Footprint" "Library:cap0603"
 			(at 129.8448 144.78 0)
 			(effects
@@
 			)
 		)
-		(property "Footprint" "2024l2:8-DFN (5x6)"
+		(property "Footprint" "Library:8-DFN (5x6)"
 			(at 124.46 58.42 90)
 			(effects
@@
 			)
 		)
-		(property "Footprint" "2024l2:CP_Radial_D8.0mm_P3.50mm"
+		(property "Footprint" "Library:CP_Radial_D8.0mm_P3.50mm"
 			(at 119.0752 144.78 0)
 			(effects
@@
 			)
 		)
-		(property "Footprint" "2024l2:cap0603"
+		(property "Footprint" "Library:cap0603"
 			(at 236.5248 144.78 0)
 			(effects
@@
 			)
 		)
-		(property "Footprint" "2024l2:cap0603"
+		(property "Footprint" "Library:cap0603"
 			(at 129.8448 82.55 0)
 			(effects
@@
 			)
 		)
-		(property "Footprint" "2024l2:8-DFN (5x6)"
+		(property "Footprint" "Library:8-DFN (5x6)"
 			(at 231.14 120.65 90)
 			(effects
@@
 			)
 		)
-		(property "Footprint" "2024l2:CP_Radial_D8.0mm_P3.50mm"
+		(property "Footprint" "Library:CP_Radial_D8.0mm_P3.50mm"
 			(at 225.7552 82.55 0)
 			(effects

Commit message: l3 might redo
Parts:
- renumbered C311 to C501, C315 to C502, C312 to C503, C316 to C504, C313 to C505, C317 to C506, C314 to C507, C318 to C508, IC301 to IC501, IC303 to IC502, IC302 to IC503, IC304 to IC504, Q301 to Q501, Q303 to Q502, Q302 to Q503, Q304 to Q504, R311 to R501, R327 to R502, R325 to R503, R341 to R504, R312 to R505, R328 to R506, R315 to R507, R317 to R508, R319 to R509, R321 to R510, R323 to R511, R331 to R512, R333 to R513, R335 to R514, R337 to R515, R339 to R516, R313 to R517, R329 to R518, R326 to R519, R342 to R520, R314 to R521, R330 to R522, R316 to R523, R318 to R524, R320 to R525, R322 to R526, R324 to R527, R332 to R528, R334 to R529, R336 to R530, R338 to R531, R340 to R532, SW302 to SW501

Commit message: l3 might redo
Parts:
- renumbered C501 to C401, C502 to C402, C503 to C403, C504 to C404, C505 to C405, C506 to C406, C507 to C407, C508 to C408, IC501 to IC401, IC502 to IC402, IC503 to IC403, IC504 to IC404, Q501 to Q401, Q502 to Q402, Q503 to Q403, Q504 to Q404, R501 to R401, R502 to R402, R503 to R403, R504 to R404, R505 to R405, R506 to R406, R507 to R407, R508 to R408, R509 to R409, R510 to R410, R511 to R411, R512 to R412, R513 to R413, R514 to R414, R515 to R415, R516 to R416, R517 to R417, R518 to R418, R519 to R419, R520 to R420, R521 to R421, R522 to R422, R523 to R423, R524 to R424, R525 to R425, R526 to R426, R527 to R427, R528 to R428, R529 to R429, R530 to R430, R531 to R431, R532 to R432, SW501 to SW401
