File: processingUnit/enc.kicad_sch (KiCad schematic)
At the start: 14 parts, among them J305 Conn_01x04, SW201 ENC RST, U201 STM32F103Cx, Y201 8Mhz

Commit message: l3 might redo
Parts:
- removed U201: STM32F103Cx, Package_DFN_QFN:QFN-48-1EP_7x7mm_P0.5mm_EP5.6x5.6mm, symbol vincent:STM32F103Cx
- removed Y201: 8Mhz, Library:CSTCE8M00G52-R0, symbol Device:Crystal_GND3
- added C407: 0u1, Library:cap0603, symbol Device:C
- added U403: STM32F401C_B-C_Ux, Package_DFN_QFN:QFN-48-1EP_7x7mm_P0.5mm_EP5.6x5.6mm, symbol vincent:STM32F401C_B-C_Ux
- added Y401: 16Mhz, Library:CX3225SB16000D0FPLCC, symbol Device:Crystal_GND24
- renumbered C201 to C401, C202 to C402, C203 to C403, C204 to C404, C205 to C405, C206 to C406, C207 to C408, D201 to D401, J305 to J405, R202 to R409, R201 to R410, SW201 to SW401
Connections:
- net +3V3 FILT: now also U403.1 (VBAT), U403.24 (VDD), U403.36 (VDD), U403.48 (VDD), U403.9 (VREF+)
- net ENC BOOT0: now also U403.44 (BOOT0)
- net ENC LED: now also U403.38 (PA15)
- net ENC OSC IN: now also U403.5 (PH0), Y401.1
- net ENC OSC OUT: now also U403.6 (PH1), Y401.3
- net ENC RST: now also U403.7 (NRST)
- net ENC RX: now also U403.21 (PB10)
- net ENC SWCLK: now also U403.37 (PA14)
- net ENC SWDIO: now also U403.34 (PA13)
- net ENC TX: now also U403.46 (PB9)
- net GNDREF: now also C407.2, U403.23 (VSS), U403.35 (VSS), U403.47 (VSS), U403.49 (VSS), U403.8 (VERF-), Y401.2, Y401.4
- net M1 DIR: now also U403.11 (PA1)
- net M1 ENC A: now also U403.17 (PA7)
- net M1 ENC B: now also U403.16 (PA6)
- net M1 PWM: now also U403.10 (PA0)
- net M2 DIR: now also U403.13 (PA3)
- net M2 ENC A: now also U403.15 (PA5)
- net M2 ENC B: now also U403.14 (PA4)
- net M2 PWM: now also U403.12 (PA2)
- net M3 DIR: now also U403.40 (PB4)
- net M3 ENC A: now also U403.29 (PA8)
- net M3 ENC B: now also U403.30 (PA9)
- net M3 PWM: now also U403.39 (PB3)
- net M4 DIR: now also U403.42 (PB6)
- net M4 ENC A: now also U403.32 (PA11)
- net M4 ENC B: now also U403.33 (PA12)
- net M4 PWM: now also U403.41 (PB5)
- new net: C407.1, U403.22 (VCAP1)
- no-connect marks 14 -> 13
Other:
- moved on the sheet: C401, C402, C403, C404, C405, C406, C408, D401, J405, R409, R410, SW401

Commit message: l3 might redo
Parts:
- renumbered C401 to C301, C402 to C302, C403 to C303, C404 to C304, C405 to C305, C406 to C306, C407 to C307, C408 to C308, D401 to D301, J405 to J301, R409 to R301, R410 to R302, SW401 to SW301, U403 to U301, Y401 to Y301
Changed lines of the file:
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@@
 		(dnp no)
 		(fields_autoplaced yes)
-		(property "Reference" "#PWR0435"
+		(property "Reference" "#PWR0304"
 			(at 111.76 104.14 0)
 			(effects
@@
 			(project "l3"
 				(path "/1b1408da-cc6a-469f-a506-e797247b3ac8/a77b9f5f-62f3-4e77-8724-0da5576d6cec"
-					(reference "#PWR0435")
+					(reference "#PWR0304")
 					(unit 1)
 				)
@@
 		(dnp no)
 		(fields_autoplaced yes)
-		(property "Reference" "J405"
+		(property "Reference" "J301"
 			(at 133.35 176.5299 0)
 			(effects
@@
 			(project "l3"
 				(path "/1b1408da-cc6a-469f-a506-e797247b3ac8/a77b9f5f-62f3-4e77-8724-0da5576d6cec"
-					(reference "J405")
+					(reference "J301")
 					(unit 1)
 				)
@@
 		(dnp no)
 		(fields_autoplaced yes)
-		(property "Reference" "#PWR0440"
+		(property "Reference" "#PWR0309"
 			(at 210.82 96.52 0)
 			(effects
@@
 			(project "l3"
 				(path "/1b1408da-cc6a-469f-a506-e797247b3ac8/a77b9f5f-62f3-4e77-8724-0da5576d6cec"
-					(reference "#PWR0440")
+					(reference "#PWR0309")
 					(unit 1)
 				)
@@
 		(dnp no)
 		(fields_autoplaced yes)
-		(property "Reference" "U403"
+		(property "Reference" "U301"
 			(at 190.5 31.75 0)
 			(effects
@@
 			(project ""
 				(path "/1b1408da-cc6a-469f-a506-e797247b3ac8/a77b9f5f-62f3-4e77-8724-0da5576d6cec"
-					(reference "U403")
+					(reference "U301")
 					(unit 1)
 				)
@@
 		(dnp no)
 		(fields_autoplaced yes)
-		(property "Reference" "#PWR0434"
+		(property "Reference" "#PWR0303"
 			(at 110.49 60.96 0)
 			(effects
@@
 			(project "l3"
 				(path "/1b1408da-cc6a-469f-a506-e797247b3ac8/a77b9f5f-62f3-4e77-8724-0da5576d6cec"
-					(reference "#PWR0434")
+					(reference "#PWR0303")
 					(unit 1)
 				)
@@
 		(on_board yes)
 		(dnp no)
-		(property "Reference" "D401"
+		(property "Reference" "D301"
 			(at 111.76 149.606 0)
 			(effects
@@
 			(project "l3"
 				(path "/1b1408da-cc6a-469f-a506-e797247b3ac8/a77b9f5f-62f3-4e77-8724-0da5576d6cec"
-					(reference "D401")
+					(reference "D301")
 					(unit 1)
 				)
@@
 		(dnp no)
 		(fields_autoplaced yes)
-		(property "Reference" "U403"
+		(property "Reference" "U301"
 			(at 153.67 101.6 0)
 			(effects
@@
 			(project ""
 				(path "/1b1408da-cc6a-469f-a506-e797247b3ac8/a77b9f5f-62f3-4e77-8724-0da5576d6cec"
-					(reference "U403")
+					(reference "U301")
 					(unit 3)
 				)
@@
 		(on_board yes)
 		(dnp no)
-		(property "Reference" "C401"
+		(property "Reference" "C301"
 			(at 114.3 44.4499 0)
 			(effects
@@
 			(project "l3"
 				(path "/1b1408da-cc6a-469f-a506-e797247b3ac8/a77b9f5f-62f3-4e77-8724-0da5576d6cec"
-					(reference "C401")
+					(reference "C301")
 					(unit 1)
 				)
@@
 		(dnp no)
 		(fields_autoplaced yes)
-		(property "Reference" "R410"
+		(property "Reference" "R302"
 			(at 186.69 82.5499 0)
 			(effects
@@
 			(project "l3"
 				(path "/1b1408da-cc6a-469f-a506-e797247b3ac8/a77b9f5f-62f3-4e77-8724-0da5576d6cec"
-					(reference "R410")
+					(reference "R302")
 					(unit 1)
 				)
@@
 		(dnp no)
 		(fields_autoplaced yes)
-		(property "Reference" "#PWR0432"
+		(property "Reference" "#PWR0301"
 			(at 95.25 156.21 0)
 			(effects
@@
 			(project "l3"
 				(path "/1b1408da-cc6a-469f-a506-e797247b3ac8/a77b9f5f-62f3-4e77-8724-0da5576d6cec"
-					(reference "#PWR0432")
+					(reference "#PWR0301")
 					(unit 1)
 				)
@@
 		(dnp no)
 		(fields_autoplaced yes)
-		(property "Reference" "C403"
+		(property "Reference" "C303"
 			(at 137.16 44.4499 0)
 			(effects
@@
 			(project "l3"
 				(path "/1b1408da-cc6a-469f-a506-e797247b3ac8/a77b9f5f-62f3-4e77-8724-0da5576d6cec"
-					(reference "C403")
+					(reference "C303")
 					(unit 1)
 				)
@@
 		(dnp no)
 		(fields_autoplaced yes)
-		(property "Reference" "#PWR0436"
+		(property "Reference" "#PWR0305"
 			(at 123.19 175.26 0)
 			(effects
@@
 			(project "l3"
 				(path "/1b1408da-cc6a-469f-a506-e797247b3ac8/a77b9f5f-62f3-4e77-8724-0da5576d6cec"
-					(reference "#PWR0436")
+					(reference "#PWR0305")
 					(unit 1)
 				)
@@
 		(dnp no)
 		(fields_autoplaced yes)
-		(property "Reference" "#PWR0438"
+		(property "Reference" "#PWR0307"
 			(at 184.15 96.52 0)
 			(effects
@@
 			(project "l3"
 				(path "/1b1408da-cc6a-469f-a506-e797247b3ac8/a77b9f5f-62f3-4e77-8724-0da5576d6cec"
-					(reference "#PWR0438")
+					(reference "#PWR0307")
 					(unit 1)
 				)
@@
 		(dnp no)
 		(fields_autoplaced yes)
-		(property "Reference" "#PWR0437"
+		(property "Reference" "#PWR0306"
 			(at 123.19 190.5 0)
 			(effects
@@
 			(project "l3"
 				(path "/1b1408da-cc6a-469f-a506-e797247b3ac8/a77b9f5f-62f3-4e77-8724-0da5576d6cec"
-					(reference "#PWR0437")
+					(reference "#PWR0306")
 					(unit 1)
 				)
@@
 		(dnp no)
 		(fields_autoplaced yes)
-		(property "Reference" "C402"
+		(property "Reference" "C302"
 			(at 125.73 44.4499 0)
 			(effects
@@
 			(project "l3"
 				(path "/1b1408da-cc6a-469f-a506-e797247b3ac8/a77b9f5f-62f3-4e77-8724-0da5576d6cec"
-					(reference "C402")
+					(reference "C302")
 					(unit 1)
 				)
@@
 		(dnp no)
 		(fields_autoplaced yes)
-		(property "Reference" "#PWR0433"
+		(property "Reference" "#PWR0302"
 			(at 110.49 40.64 0)
 			(effects
@@
 			(project "l3"
 				(path "/1b1408da-cc6a-469f-a506-e797247b3ac8/a77b9f5f-62f3-4e77-8724-0da5576d6cec"
-					(reference "#PWR0433")
+					(reference "#PWR0302")
 					(unit 1)
 				)
@@
 		(dnp no)
 		(fields_autoplaced yes)
-		(property "Reference" "C405"
+		(property "Reference" "C305"
 			(at 160.02 44.4499 0)
 			(effects
@@
 			(project "l3"
 				(path "/1b1408da-cc6a-469f-a506-e797247b3ac8/a77b9f5f-62f3-4e77-8724-0da5576d6cec"
-					(reference "C405")
+					(reference "C305")
 					(unit 1)
 				)
@@
 		(on_board yes)
 		(dnp no)
-		(property "Reference" "R409"
+		(property "Reference" "R301"
 			(at 101.6 144.78 90)
 			(effects
@@
 			(project "l3"
 				(path "/1b1408da-cc6a-469f-a506-e797247b3ac8/a77b9f5f-62f3-4e77-8724-0da5576d6cec"
-					(reference "R409")
+					(reference "R301")
 					(unit 1)
 				)
@@
 		(dnp no)
 		(fields_autoplaced yes)
-		(property "Reference" "C407"
+		(property "Reference" "C307"
 			(at 212.09 45.7199 0)
 			(effects
@@
 			(project "l3"
 				(path "/1b1408da-cc6a-469f-a506-e797247b3ac8/a77b9f5f-62f3-4e77-8724-0da5576d6cec"
-					(reference "C407")
+					(reference "C307")
 					(unit 1)
 				)
@@
 		(dnp no)
 		(fields_autoplaced yes)
-		(property "Reference" "#PWR0439"
+		(property "Reference" "#PWR0308"
 			(at 205.74 63.5 0)
 			(effects
@@
 			(project "l3"
 				(path "/1b1408da-cc6a-469f-a506-e797247b3ac8/a77b9f5f-62f3-4e77-8724-0da5576d6cec"
-					(reference "#PWR0439")
+					(reference "#PWR0308")
 					(unit 1)
 				)
@@
 		(dnp no)
 		(fields_autoplaced yes)
-		(property "Reference" "SW401"
+		(property "Reference" "SW301"
 			(at 198.12 77.4699 90)
 			(effects
@@
 			(project "l3"
 				(path "/1b1408da-cc6a-469f-a506-e797247b3ac8/a77b9f5f-62f3-4e77-8724-0da5576d6cec"
-					(reference "SW401")
+					(reference "SW301")
 					(unit 1)
 				)
@@
 		(dnp no)
 		(fields_autoplaced yes)
-		(property "Reference" "C406"
+		(property "Reference" "C306"
 			(at 171.45 44.4499 0)
 			(effects
@@
 			(project "l3"
 				(path "/1b1408da-cc6a-469f-a506-e797247b3ac8/a77b9f5f-62f3-4e77-8724-0da5576d6cec"
-					(reference "C406")
+					(reference "C306")
 					(unit 1)
 				)
@@
 		(on_board yes)
 		(dnp no)
-		(property "Reference" "Y401"
+		(property "Reference" "Y301"
 			(at 118.11 90.17 0)
 			(effects
@@
 			(project "l3"
 				(path "/1b1408da-cc6a-469f-a506-e797247b3ac8/a77b9f5f-62f3-4e77-8724-0da5576d6cec"
-					(reference "Y401")
+					(reference "Y301")
 					(unit 1)
 				)
@@
 		(dnp no)
 		(fields_autoplaced yes)
-		(property "Reference" "U403"
+		(property "Reference" "U301"
 			(at 152.4 64.77 0)
 			(effects
@@
 			(project ""
 				(path "/1b1408da-cc6a-469f-a506-e797247b3ac8/a77b9f5f-62f3-4e77-8724-0da5576d6cec"
-					(reference "U403")
+					(reference "U301")
 					(unit 2)
 				)
@@
 		(dnp no)
 		(fields_autoplaced yes)
-		(property "Reference" "C404"
+		(property "Reference" "C304"
 			(at 148.59 44.4499 0)
 			(effects
@@
 			(project "l3"
 				(path "/1b1408da-cc6a-469f-a506-e797247b3ac8/a77b9f5f-62f3-4e77-8724-0da5576d6cec"
-					(reference "C404")
+					(reference "C304")
 					(unit 1)
 				)
@@
 		(dnp no)
 		(fields_autoplaced yes)
-		(property "Reference" "C408"
+		(property "Reference" "C308"
 			(at 214.63 77.4699 0)
 			(effects
@@
 			(project "l3"
 				(path "/1b1408da-cc6a-469f-a506-e797247b3ac8/a77b9f5f-62f3-4e77-8724-0da5576d6cec"
-					(reference "C408")
-					(unit 1)
-				)
+					(reference "C308")
+					(unit 1)
+				)

Commit message: drivers
Connections:
- net ENC RX: now also U301.13 (PA3); no longer U301.21 (PB10)
- net ENC TX: now also U301.12 (PA2); no longer U301.46 (PB9)
- net M1 DIR: now also U301.17 (PA7); no longer U301.11 (PA1)
- net M1 ENC A: now also U301.32 (PA11); no longer U301.17 (PA7)
- net M1 ENC B: now also U301.31 (PA10); no longer U301.16 (PA6)
- net M1 PWM: now also U301.16 (PA6); no longer U301.10 (PA0)
- net M2 DIR: now also U301.41 (PB5); no longer U301.13 (PA3)
- net M2 ENC A: now also U301.30 (PA9); no longer U301.15 (PA5)
- net M2 ENC B: now also U301.29 (PA8); no longer U301.14 (PA4)
- net M2 PWM: now also U301.42 (PB6); no longer U301.12 (PA2)
- net M3 DIR: now also U301.11 (PA1); no longer U301.40 (PB4)
- net M3 ENC A: now also U301.19 (PB1); no longer U301.29 (PA8)
- net M3 ENC B: now also U301.20 (PB2); no longer U301.30 (PA9)
- net M3 PWM: now also U301.10 (PA0); no longer U301.39 (PB3)
- net M4 DIR: now also U301.14 (PA4); no longer U301.42 (PB6)
- net M4 ENC A: now also U301.40 (PB4); no longer U301.32 (PA11)
- net M4 ENC B: now also U301.39 (PB3); no longer U301.33 (PA12)
- net M4 PWM: now also U301.15 (PA5); no longer U301.41 (PB5)
- no-connect marks 13 -> 10

Commit message: l3 routing
Connections:
- net M1 ENC A: now also U301.27 (PB14); no longer U301.32 (PA11)
- net M1 ENC B: now also U301.28 (PB15); no longer U301.31 (PA10)
- net M2 ENC A: now also U301.25 (PB12); no longer U301.30 (PA9)
- net M2 ENC B: now also U301.26 (PB13); no longer U301.29 (PA8)
- net M3 ENC A: now also U301.32 (PA11); no longer U301.19 (PB1)
- net M3 ENC B: now also U301.31 (PA10); no longer U301.20 (PB2)
- net M4 ENC A: now also U301.29 (PA8); no longer U301.40 (PB4)
- net M4 ENC B: now also U301.30 (PA9); no longer U301.39 (PB3)
- no-connect marks 10 -> 13

Commit message: logo
Connections:
- net M3 ENC A: now also U301.31 (PA10); no longer U301.32 (PA11)
- net M3 ENC B: now also U301.32 (PA11); no longer U301.31 (PA10)
Changed lines of the file:
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@@
 	(global_label "M3 ENC A"
 		(shape input)
+		(at 115.57 134.62 180)
+		(fields_autoplaced yes)
+		(effects
+			(font
+				(size 1.27 1.27)
+			)
+			(justify right)
+		)
+		(property "Intersheetrefs" "${INTERSHEET_REFS}"
+			(at 103.1506 134.62 0)
+			(effects
+				(font
+					(size 1.27 1.27)
+				)
+				(justify right)
+				(hide yes)
+			)
+		)
+	)
+	(global_label "M1 ENC A"
+		(shape input)
+		(at 191.77 144.78 0)
+		(fields_autoplaced yes)
+		(effects
+			(font
+				(size 1.27 1.27)
+			)
+			(justify left)
+		)
+		(property "Intersheetrefs" "${INTERSHEET_REFS}"
+			(at 204.1894 144.78 0)
+			(effects
+				(font
+					(size 1.27 1.27)
+				)
+				(justify left)
+				(hide yes)
+			)
+		)
+	)
+	(global_label "M4 ENC A"
+		(shape input)
+		(at 115.57 129.54 180)
+		(fields_autoplaced yes)
+		(effects
+			(font
+				(size 1.27 1.27)
+			)
+			(justify right)
+		)
+		(property "Intersheetrefs" "${INTERSHEET_REFS}"
+			(at 103.1506 129.54 0)
+			(effects
+				(font
+					(size 1.27 1.27)
+				)
+				(justify right)
+				(hide yes)
+			)
+		)
+	)
+	(global_label "M1 ENC B"
+		(shape input)
+		(at 191.77 147.32 0)
+		(fields_autoplaced yes)
+		(effects
+			(font
+				(size 1.27 1.27)
+			)
+			(justify left)
+		)
+		(property "Intersheetrefs" "${INTERSHEET_REFS}"
+			(at 204.3708 147.32 0)
+			(effects
+				(font
+					(size 1.27 1.27)
+				)
+				(justify left)
+				(hide yes)
+			)
+		)
+	)
+	(global_label "M1 ENC A"
+		(shape input)
+		(at 276.86 132.08 0)
+		(fields_autoplaced yes)
+		(effects
+			(font
+				(size 1.27 1.27)
+			)
+			(justify left)
+		)
+		(property "Intersheetrefs" "${INTERSHEET_REFS}"
+			(at 289.2794 132.08 0)
+			(effects
+				(font
+					(size 1.27 1.27)
+				)
+				(justify left)
+				(hide yes)
+			)
+		)
+	)
+	(global_label "M2 ENC B"
+		(shape input)
+		(at 191.77 142.24 0)
+		(fields_autoplaced yes)
+		(effects
+			(font
+				(size 1.27 1.27)
+			)
+			(justify left)
+		)
+		(property "Intersheetrefs" "${INTERSHEET_REFS}"
+			(at 204.3708 142.24 0)
+			(effects
+				(font
+					(size 1.27 1.27)
+				)
+				(justify left)
+				(hide yes)
+			)
+		)
+	)
+	(global_label "M1 ENC B"
+		(shape input)
+		(at 276.86 129.54 0)
+		(fields_autoplaced yes)
+		(effects
+			(font
+				(size 1.27 1.27)
+			)
+			(justify left)
+		)
+		(property "Intersheetrefs" "${INTERSHEET_REFS}"
+			(at 289.4608 129.54 0)
+			(effects
+				(font
+					(size 1.27 1.27)
+				)
+				(justify left)
+				(hide yes)
+			)
+		)
+	)
+	(global_label "M4 ENC B"
+		(shape input)
+		(at 115.57 132.08 180)
+		(fields_autoplaced yes)
+		(effects
+			(font
+				(size 1.27 1.27)
+			)
+			(justify right)
+		)
+		(property "Intersheetrefs" "${INTERSHEET_REFS}"
+			(at 102.9692 132.08 0)
+			(effects
+				(font
+					(size 1.27 1.27)
+				)
+				(justify right)
+				(hide yes)
+			)
+		)
+	)
+	(global_label "M2 ENC A"
+		(shape input)
+		(at 191.77 139.7 0)
+		(fields_autoplaced yes)
+		(effects
+			(font
+				(size 1.27 1.27)
+			)
+			(justify left)
+		)
+		(property "Intersheetrefs" "${INTERSHEET_REFS}"
+			(at 204.1894 139.7 0)
+			(effects
+				(font
+					(size 1.27 1.27)
+				)
+				(justify left)
+				(hide yes)
+			)
+		)
+	)
+	(global_label "M3 ENC B"
+		(shape input)
 		(at 115.57 137.16 180)
 		(fields_autoplaced yes)
@@
 		)
 		(property "Intersheetrefs" "${INTERSHEET_REFS}"
-			(at 103.1506 137.16 0)
-			(effects
-				(font
-					(size 1.27 1.27)
-				)
-				(justify right)
-				(hide yes)
-			)
-		)
-	)
-	(global_label "M1 ENC A"
-		(shape input)
-		(at 191.77 144.78 0)
-		(fields_autoplaced yes)
-		(effects
-			(font
-				(size 1.27 1.27)
-			)
-			(justify left)
-		)
-		(property "Intersheetrefs" "${INTERSHEET_REFS}"
-			(at 204.1894 144.78 0)
-			(effects
-				(font
-					(size 1.27 1.27)
-				)
-				(justify left)
-				(hide yes)
-			)
-		)
-	)
-	(global_label "M4 ENC A"
-		(shape input)
-		(at 115.57 129.54 180)
-		(fields_autoplaced yes)
-		(effects
-			(font
-				(size 1.27 1.27)
-			)
-			(justify right)
-		)
-		(property "Intersheetrefs" "${INTERSHEET_REFS}"
-			(at 103.1506 129.54 0)
-			(effects
-				(font
-					(size 1.27 1.27)
-				)
-				(justify right)
-				(hide yes)
-			)
-		)
-	)
-	(global_label "M1 ENC B"
-		(shape input)
-		(at 191.77 147.32 0)
-		(fields_autoplaced yes)
-		(effects
-			(font
-				(size 1.27 1.27)
-			)
-			(justify left)
-		)
-		(property "Intersheetrefs" "${INTERSHEET_REFS}"
-			(at 204.3708 147.32 0)
-			(effects
-				(font
-					(size 1.27 1.27)
-				)
-				(justify left)
-				(hide yes)
-			)
-		)
-	)
-	(global_label "M1 ENC A"
-		(shape input)
-		(at 276.86 132.08 0)
-		(fields_autoplaced yes)
-		(effects
-			(font
-				(size 1.27 1.27)
-			)
-			(justify left)
-		)
-		(property "Intersheetrefs" "${INTERSHEET_REFS}"
-			(at 289.2794 132.08 0)
-			(effects
-				(font
-					(size 1.27 1.27)
-				)
-				(justify left)
-				(hide yes)
-			)
-		)
-	)
-	(global_label "M2 ENC B"
-		(shape input)
-		(at 191.77 142.24 0)
-		(fields_autoplaced yes)
-		(effects
-			(font
-				(size 1.27 1.27)
-			)
-			(justify left)
-		)
-		(property "Intersheetrefs" "${INTERSHEET_REFS}"
-			(at 204.3708 142.24 0)
-			(effects
-				(font
-					(size 1.27 1.27)
-				)
-				(justify left)
-				(hide yes)
-			)
-		)
-	)
-	(global_label "M1 ENC B"
-		(shape input)
-		(at 276.86 129.54 0)
-		(fields_autoplaced yes)
-		(effects
-			(font
-				(size 1.27 1.27)
-			)
-			(justify left)
-		)
-		(property "Intersheetrefs" "${INTERSHEET_REFS}"
-			(at 289.4608 129.54 0)
-			(effects
-				(font
-					(size 1.27 1.27)
-				)
-				(justify left)
-				(hide yes)
-			)
-		)
-	)
-	(global_label "M4 ENC B"
-		(shape input)
-		(at 115.57 132.08 180)
-		(fields_autoplaced yes)
-		(effects
-			(font
-				(size 1.27 1.27)
-			)
-			(justify right)
-		)
-		(property "Intersheetrefs" "${INTERSHEET_REFS}"
-			(at 102.9692 132.08 0)
-			(effects
-				(font
-					(size 1.27 1.27)
-				)
-				(justify right)
-				(hide yes)
-			)
-		)
-	)
-	(global_label "M2 ENC A"
-		(shape input)
-		(at 191.77 139.7 0)
-		(fields_autoplaced yes)
-		(effects
-			(font
-				(size 1.27 1.27)
-			)
-			(justify left)
-		)
-		(property "Intersheetrefs" "${INTERSHEET_REFS}"
-			(at 204.1894 139.7 0)
-			(effects
-				(font
-					(size 1.27 1.27)
-				)
-				(justify left)
-				(hide yes)
-			)
-		)
-	)
-	(global_label "M3 ENC B"
-		(shape input)
-		(at 115.57 134.62 180)
-		(fields_autoplaced yes)
-		(effects
-			(font
-				(size 1.27 1.27)
-			)
-			(justify right)
-		)
-		(property "Intersheetrefs" "${INTERSHEET_REFS}"
-			(at 102.9692 134.62 0)
-			(effects
-				(font
+			(at 102.9692 137.16 0)
+			(effects
+				(font

Commit message: step
Changed lines of the file:
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@@
-	(wire
-		(pts
-			(xy 276.86 132.08) (xy 259.08 132.08)
-		)
-		(stroke
-			(width 0)
-			(type default)
-		)
-	)
 	(wire
 		(pts
@@
 		(pts
 			(xy 106.68 95.25) (xy 111.76 95.25)
-		)
-		(stroke
-			(width 0)
-			(type default)
-		)
-	)
-	(wire
-		(pts
-			(xy 276.86 129.54) (xy 259.08 129.54)
 		)
 		(stroke
@@
 		)
 	)
-	(global_label "M1 ENC A"
-		(shape input)
-		(at 276.86 132.08 0)
-		(fields_autoplaced yes)
-		(effects
-			(font
-				(size 1.27 1.27)
-			)
-			(justify left)
-		)
-		(property "Intersheetrefs" "${INTERSHEET_REFS}"
-			(at 289.2794 132.08 0)
-			(effects
-				(font
-					(size 1.27 1.27)
-				)
-				(justify left)
-				(hide yes)
-			)
-		)
-	)
 	(global_label "M2 ENC B"
 		(shape input)
@@
 			(effects
 				(font
-					(size 1.27 1.27)
-				)
-				(justify left)
-				(hide yes)
-			)
-		)
-	)
-	(global_label "M1 ENC B"
-		(shape input)
-		(at 276.86 129.54 0)
-		(fields_autoplaced yes)
-		(effects
-			(font
-				(size 1.27 1.27)
-			)
-			(justify left)
-		)
-		(property "Intersheetrefs" "${INTERSHEET_REFS}"
-			(at 289.4608 129.54 0)
-			(effects
-				(font

Commit message: nightmare fuel
Connections:
- net M1 ENC A: now also U301.26 (PB13); no longer U301.27 (PB14)
- net M1 ENC B: now also U301.25 (PB12); no longer U301.28 (PB15)
- net M2 ENC A: now also U301.29 (PA8); no longer U301.25 (PB12)
- net M2 ENC B: now also U301.30 (PA9); no longer U301.26 (PB13)
- net M3 DIR: now also U301.46 (PB9); no longer U301.11 (PA1)
- net M3 PWM: now also U301.45 (PB8); no longer U301.10 (PA0)
- net M4 ENC A: now also U301.19 (PB1); no longer U301.29 (PA8)
- net M4 ENC B: now also U301.18 (PB0); no longer U301.30 (PA9)

Commit message: schematic
Connections:
- net M2 ENC A: now also U301.30 (PA9); no longer U301.29 (PA8)
- net M2 ENC B: now also U301.29 (PA8); no longer U301.30 (PA9)
Changed lines of the file:
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@@
 	(global_label "M2 ENC A"
 		(shape input)
-		(at 115.57 129.54 180)
+		(at 115.57 132.08 180)
 		(fields_autoplaced yes)
 		(effects
@@
 		)
 		(property "Intersheetrefs" "${INTERSHEET_REFS}"
-			(at 103.1506 129.54 0)
+			(at 102.9692 132.08 0)
 			(effects
 				(font
@@
 	(global_label "M2 ENC B"
 		(shape input)
-		(at 115.57 132.08 180)
+		(at 115.57 129.54 180)
 		(fields_autoplaced yes)
 		(effects
@@
 		)
 		(property "Intersheetrefs" "${INTERSHEET_REFS}"
-			(at 102.9692 132.08 0)
+			(at 103.1506 129.54 0)
 			(effects
 				(font
