File: breakout/LED/LED.kicad_pcb (KiCad board)
At the start: 2 copper layers, 9.1 x 18.8 mm, 2 parts, among them J1 Conn_01x02

Commit message: breakout
Parts:
- added D2: LED, Library:led2835, F.Cu at (161.0, 74.1)
- moved D1 1.39 mm to (161.0, 70.2)
Routing:
- net +3V3: track 10.5 -> 11.8 mm
