File: breakout/Receiver/Receiver.kicad_pcb (KiCad board)
At the start: 2 copper layers, 9.1 x 18.8 mm, 4 parts, among them J1 Conn_01x03, U1 TSSP58038

Commit message: breakout
Parts:
- removed C1: 0.1uF, Library:cap0603
- removed R1: 100r, Library:res0603
- moved U1 2.00 mm to (149.5, 99.6)
Connections:
- U1 pad 3: Net-(U1-Vs) -> +3V3
Routing:
- net Net-(U1-Vs): track 6.29 -> 0.00 mm
- net +3V3: track 3.32 -> 8.10 mm
- net Net-(J1-Pin_2): track 7.12 -> 4.61 mm
