File: breakout/Emmiter/Emmiter.kicad_pcb (KiCad board)
At the start: 2 copper layers, 9.1 x 18.8 mm, 5 parts, among them J1 Conn_01x03, Q1 IRLML6344TRPBF

Commit message: emmiter changes
Parts:
- D1: footprint LED_THT:LED_D5.0mm -> Library:DIO_VSMB2020X01
- moved D1 1.28 mm to (64.5, 41.5)
Routing:
- net +3V3: track 11.9 -> 12.2 mm, vias 0 -> 1
Changed lines of the file:
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@@
 		)
 	)
-	(footprint "LED_THT:LED_D5.0mm"
-		(layer "F.Cu")
-		(at 63.262501 41.475001)
-		(descr "LED, diameter 5.0mm, 2 pins, http://cdn-reichelt.de/documents/datenblatt/A500/LL-504BC2E-009.pdf")
-		(tags "LED diameter 5.0mm 2 pins")
+	(footprint "Library:DIO_VSMB2020X01"
+		(layer "F.Cu")
+		(at 64.537501 41.500001)
 		(property "Reference" "D1"
-			(at 1.27 -3.96 0)
+			(at 0.381 -2.286 0)
 			(layer "F.SilkS")
 			(hide yes)
@@
 		)
 		(property "Value" "LED"
-			(at 1.27 3.96 0)
+			(at 6.731 2.286 0)
 			(layer "F.Fab")
 			(effects
@@
 			)
 		)
-		(property "Footprint" "LED_THT:LED_D5.0mm"
+		(property "Footprint" "Library:DIO_VSMB2020X01"
 			(at 0 0 0)
 			(unlocked yes)
@@
 			)
 		)
-		(attr through_hole)
-		(fp_line
-			(start -1.29 -1.545)
-			(end -1.29 1.545)
-			(stroke
-				(width 0.12)
-				(type solid)
-			)
-			(layer "F.SilkS")
-		)
-		(fp_arc
-			(start -1.29 -1.54483)
-			(mid 2.072002 -2.880433)
-			(end 4.26 0.000462)
-			(stroke
-				(width 0.12)
-				(type solid)
-			)
-			(layer "F.SilkS")
-		)
-		(fp_arc
-			(start 4.26 -0.000462)
-			(mid 2.072002 2.880433)
-			(end -1.29 1.54483)
-			(stroke
-				(width 0.12)
+		(property ki_fp_filters "LED* LED_SMD:* LED_THT:*")
+		(sheetname "Root")
+		(sheetfile "Emmiter.kicad_sch")
+		(attr smd)
+		(fp_line
+			(start -1.25 -1.25)
+			(end -1.25 -0.695)
+			(stroke
+				(width 0.127)
+				(type solid)
+			)
+			(layer "F.SilkS")
+		)
+		(fp_line
+			(start -1.25 -1.25)
+			(end 1.25 -1.25)
+			(stroke
+				(width 0.127)
+				(type solid)
+			)
+			(layer "F.SilkS")
+		)
+		(fp_line
+			(start -1.25 1.25)
+			(end -1.25 0.695)
+			(stroke
+				(width 0.127)
+				(type solid)
+			)
+			(layer "F.SilkS")
+		)
+		(fp_line
+			(start 1.25 -1.25)
+			(end 1.25 -0.695)
+			(stroke
+				(width 0.127)
+				(type solid)
+			)
+			(layer "F.SilkS")
+		)
+		(fp_line
+			(start 1.25 1.25)
+			(end -1.25 1.25)
+			(stroke
+				(width 0.127)
+				(type solid)
+			)
+			(layer "F.SilkS")
+		)
+		(fp_line
+			(start 1.25 1.25)
+			(end 1.25 0.695)
+			(stroke
+				(width 0.127)
 				(type solid)
 			)
@@
 		)
 		(fp_circle
-			(center 1.27 0)
-			(end 3.77 0)
-			(stroke
-				(width 0.12)
+			(center -3.025 0)
+			(end -2.925 0)
+			(stroke
+				(width 0.2)
 				(type solid)
 			)
@@
 		)
 		(fp_line
-			(start -1.95 -3.25)
-			(end -1.95 3.25)
+			(start -2.825 -1.5)
+			(end -2.825 1.5)
 			(stroke
 				(width 0.05)
@@
 		)
 		(fp_line
-			(start -1.95 3.25)
-			(end 4.5 3.25)
+			(start -2.825 -1.5)
+			(end 2.825 -1.5)
 			(stroke
 				(width 0.05)
@@
 		)
 		(fp_line
-			(start 4.5 -3.25)
-			(end -1.95 -3.25)
+			(start 2.825 1.5)
+			(end -2.825 1.5)
 			(stroke
 				(width 0.05)
@@
 		)
 		(fp_line
-			(start 4.5 3.25)
-			(end 4.5 -3.25)
+			(start 2.825 1.5)
+			(end 2.825 -1.5)
 			(stroke
 				(width 0.05)
@@
 		)
 		(fp_line
-			(start -1.23 -1.469694)
-			(end -1.23 1.469694)
-			(stroke
-				(width 0.1)
+			(start -1.25 -1.25)
+			(end -1.25 1.25)
+			(stroke
+				(width 0.127)
 				(type solid)
 			)
 			(layer "F.Fab")
 		)
-		(fp_arc
-			(start -1.23 -1.469694)
-			(mid 4.17 0.000016)
-			(end -1.230016 1.469666)
-			(stroke
-				(width 0.1)
+		(fp_line
+			(start -1.25 -1.25)
+			(end 1.25 -1.25)
+			(stroke
+				(width 0.127)
 				(type solid)
 			)
 			(layer "F.Fab")
 		)
+		(fp_line
+			(start -1.25 1.25)
+			(end 1.25 1.25)
+			(stroke
+				(width 0.127)
+				(type solid)
+			)
+			(layer "F.Fab")
+		)
+		(fp_line
+			(start 1.25 -1.25)
+			(end 1.25 1.25)
+			(stroke
+				(width 0.127)
+				(type solid)
+			)
+			(layer "F.Fab")
+		)
 		(fp_circle
-			(center 1.27 0)
-			(end 3.77 0)
-			(stroke
-				(width 0.1)
+			(center -3.025 0)
+			(end -2.925 0)
+			(stroke
+				(width 0.2)
 				(type solid)
 			)
@@
 			(layer "F.Fab")
 		)
-		(fp_text user "${REFERENCE}"
-			(at 1.25 0 0)
-			(layer "F.Fab")
-			(effects
-				(font
-					(size 0.8 0.8)
-					(thickness 0.2)
-				)
-			)
-		)
-		(pad "1" thru_hole rect
-			(at 0 0)
-			(size 1.8 1.8)
-			(drill 0.9)
-			(layers "*.Cu" "*.Mask")
-			(remove_unused_layers no)
+		(pad "1" smd rect
+			(at -1.9 0)
+			(size 1.35 0.75)
+			(layers "F.Cu" "F.Paste" "F.Mask")
 			(net 5 "Net-(D1-K)")
 			(pinfunction "K")
 			(pintype "passive")
-		)
-		(pad "2" thru_hole circle
-			(at 2.54 0)
-			(size 1.8 1.8)
-			(drill 0.9)
-			(layers "*.Cu" "*.Mask")
-			(remove_unused_layers no)
+			(solder_mask_margin 0.102)
+		)
+		(pad "2" smd rect
+			(at 1.9 0)
+			(size 1.35 0.75)
+			(layers "F.Cu" "F.Paste" "F.Mask")
 			(net 1 "+3V3")
 			(pinfunction "A")
 			(pintype "passive")
-		)
-		(model "${KICAD8_3DMODEL_DIR}/LED_THT.3dshapes/LED_D5.0mm.wrl"
-			(offset
-				(xyz 0 0 -3)
-			)
-			(scale
-				(xyz 1 1 1)
-			)
-			(rotate
-				(xyz 0 0 0)
-			)
+			(solder_mask_margin 0.102)
 		)
 	)
@@
 	)
 	(segment
-		(start 65.79 41.45)
-		(end 65.79 48.045)
+		(start 66.537501 41.500001)
+		(end 66.537501 43.500001)
 		(width 0.2)
-		(layer "B.Cu")
+		(layer "F.Cu")
 		(net 1)
 	)
+	(via
+		(at 66.537501 43.500001)
+		(size 0.6)
+		(drill 0.3)
+		(layers "F.Cu" "B.Cu")
+		(net 1)
+	)
 	(segment
-		(start 65.79 48.045)
+		(start 66.537501 47.297499)
 		(end 62.01 51.825)
 		(width 0.2)
@@
 	)
 	(segment
+		(start 66.537501 43.500001)
+		(end 66.537501 47.297499)
+		(width 0.2)
+		(layer "B.Cu")
+		(net 1)
+	)
+	(segment
 		(start 65.490001 48.2925)
 		(end 65.490001 50.884999)
@@
 	)
 	(segment
+		(start 62.737501 42.500001)
+		(end 62.737501 41.500001)
+		(width 0.2)
+		(layer "F.Cu")
+		(net 5)
+	)
+	(segment
 		(start 61.715 45.9)
-		(end 61.715 42.985)
+		(end 61.715 43.522502)
 		(width 0.2)
 		(layer "F.Cu")
@@
 	)
 	(segment
-		(start 61.715 42.985)
-		(end 63.25 41.45)
+		(start 61.715 43.522502)
+		(end 62.737501 42.500001)
 		(width 0.2)
 		(layer "F.Cu")
@@
 	)
 	(zone
+		(net 4)
+		(net_name "Net-(Q1-D)")
+		(layer "F.Cu")
+		(name "$teardrop_padvia$")
+		(hatch full 0.1)
+		(priority 30002)
+		(attr
+			(teardrop
+				(type padvia)
+			)
+		)
+		(connect_pads yes
+			(clearance 0)
+		)
+		(min_thickness 0.0254)
+		(filled_areas_thickness no)
+		(fill yes
+			(thermal_gap 0.5)
+			(thermal_bridge_width 0.5)
+			(island_removal_mode 1)
+			(island_area_min 10)
+		)
+		(polygon
+			(pts
+				(xy 64.315 45.8) (xy 64.262071 45.784737) (xy 64.209142 45.764629) (xy 64.156213 45.739674) (xy 64.103284 45.709872)
+				(xy 64.050355 45.675225) (xy 63.997426 45.63573) (xy 63.944497 45.591389) (xy 63.891568 45.542202)
+				(xy 63.838639 45.488169) (xy 63.785711 45.429289) (xy 63.314 45.9) (xy 63.785711 46.370711) (xy 63.838639 46.31183)
+				(xy 63.891568 46.257797) (xy 63.944497 46.20861) (xy 63.997426 46.164269) (xy 64.050355 46.124775)
+				(xy 64.103284 46.090127) (xy 64.156213 46.060325) (xy 64.209142 46.03537) (xy 64.262071 46.015262)
+				(xy 64.315 46)
+			)
+		)
+	)
+	(zone
 		(net 3)
 		(net_name "/PULSE")
@@
 			)
 		)
-	)
-	(zone
-		(net 4)
-		(net_name "Net-(Q1-D)")
-		(layer "F.Cu")
-		(name "$teardrop_padvia$")
-		(hatch full 0.1)
-		(priority 30002)
-		(attr
-			(teardrop
-				(type padvia)
-			)
-		)
-		(connect_pads yes
-			(clearance 0)
-		)
-		(min_thickness 0.0254)
-		(filled_areas_thickness no)
-		(fill yes
-			(thermal_gap 0.5)
-			(thermal_bridge_width 0.5)
-			(island_removal_mode 1)
-			(island_area_min 10)
-		)
-		(polygon
-			(pts
-				(xy 64.315 45.8) (xy 64.262071 45.784737) (xy 64.209142 45.764629) (xy 64.156213 45.739674) (xy 64.103284 45.709872)
-				(xy 64.050355 45.675225) (xy 63.997426 45.63573) (xy 63.944497 45.591389) (xy 63.891568 45.542202)
-				(xy 63.838639 45.488169) (xy 63.785711 45.429289) (xy 63.314 45.9) (xy 63.785711 46.370711) (xy 63.838639 46.31183)
-				(xy 63.891568 46.257797) (xy 63.944497 46.20861) (xy 63.997426 46.164269) (xy 64.050355 46.124775)
-				(xy 64.103284 46.090127) (xy 64.156213 46.060325) (xy 64.209142 46.03537) (xy 64.262071 46.015262)
-				(xy 64.315 46)
-			)
-		)
