File: breakout/Emmiter/Emmiter.kicad_sch (KiCad schematic)
At the start: 5 parts, among them J1 Conn_01x03, Q1 IRLML6344TRPBF

Commit message: emmiter changes
Parts:
- D1: footprint LED_THT:LED_D5.0mm -> Library:DIO_VSMB2020X01
Changed lines of the file:
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@@
 			)
 		)
-		(property "Footprint" "LED_THT:LED_D5.0mm"
+		(property "Footprint" "Library:DIO_VSMB2020X01"
 			(at 92.71 69.85 0)
 			(effects
