File: supplyUnit/boostUnit/boostUnit.kicad_sch (KiCad schematic)
At the start: 22 parts, among them J1 Conn_02x03_Counter_Clockwise, J2 Conn_02x03_Counter_Clockwise

Commit message: boost
Parts:
- removed BSQ1: IRLB3036PbF, 2024l1:TO-220-3_Vertical, symbol vincent:IPD050N10N5ATMA1
- added BSQ1: ISC011N06LM5ATMA1, Library:8-DFN (5x6), symbol vincent:AON6354
Connections:
- net GND: now also BSQ1.1 (S), BSQ1.2 (S), BSQ1.3 (S)
- net at BSD1.2 (A), BSJ1.2 (Pin_2), BSR1.1: now also BSQ1.5 (D), BSQ1.6 (D), BSQ1.7 (D), BSQ1.8 (D), BSQ1.9 (D)
- net at BSR2.2, BSR3.2: now also BSQ1.4 (G)
Changed lines of the file:
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@@
+	)
+	(symbol
+		(lib_id "vincent:AON6354")
+		(at 72.39 66.04 0)
+		(unit 1)
+		(exclude_from_sim no)
+		(in_bom yes)
+		(on_board yes)
+		(dnp no)
+		(fields_autoplaced yes)
+		(property "Reference" "BSQ1"
+			(at 83.82 64.7699 0)
+			(effects
+				(font
+					(size 1.27 1.27)
+				)
+				(justify left)
+			)
+		)
+		(property "Value" "ISC011N06LM5ATMA1"
+			(at 83.82 67.3099 0)
+			(effects
+				(font
+					(size 1.27 1.27)
+				)
+				(justify left)
+			)
+		)
+		(property "Footprint" "Library:8-DFN (5x6)"
+			(at 80.01 66.04 0)
+			(effects
+				(font
+					(size 1.27 1.27)
+				)
+				(hide yes)
+			)
+		)
+		(property "Datasheet" "https://www.mouser.sg/datasheet/2/196/Infineon_ISC011N06LM5_DataSheet_v02_02_EN-3363456.pdf"
+			(at 80.01 66.04 0)
+			(effects
+				(font
+					(size 1.27 1.27)
+				)
+				(hide yes)
+			)
+		)
+		(property "Description" ""
+			(at 72.39 66.04 0)
+			(effects
+				(font
+					(size 1.27 1.27)
+				)
+				(hide yes)
+			)
+		)
+		(pin "7"
+		)
+		(pin "8"
+		)
+		(pin "9"
+		)
+		(pin "1"
+		)
+		(pin "3"
+		)
+		(pin "2"
+		)
+		(pin "5"
+		)
+		(pin "4"
+		)
+		(pin "6"
+		)
+		(instances
+			(project ""
+				(path "/697a38d4-3409-462e-879c-d6eee2cce560"
+					(reference "BSQ1")
+					(unit 1)
+				)
+			)
+		)
 	)
 	(symbol
@@
 					(unit 1)
 				)
-			)
-		)
-	)
-	(symbol
-		(lib_id "vincent:IPD050N10N5ATMA1")
-		(at 72.39 66.04 0)
-		(unit 1)
-		(exclude_from_sim no)
-		(in_bom yes)
-		(on_board yes)
-		(dnp no)
-		(fields_autoplaced yes)
-		(property "Reference" "BSQ1"
-			(at 83.82 64.7699 0)
-			(effects
-				(font
-					(size 1.27 1.27)
-				)
-				(justify left)
-			)
-		)
-		(property "Value" "IRLB3036PbF"
-			(at 83.82 67.3099 0)
-			(effects
-				(font
-					(size 1.27 1.27)
-				)
-				(justify left)
-			)
-		)
-		(property "Footprint" "2024l1:TO-220-3_Vertical"
-			(at 83.82 164.77 0)
-			(effects
-				(font
-					(size 1.27 1.27)
-				)
-				(justify left top)
-				(hide yes)
-			)
-		)
-		(property "Datasheet" "https://www.infineon.com/dgdl/Infineon-IPD050N10N5-DS-v02_01-EN.pdf?fileId=5546d4625b3ca4ec015b615bb7536713"
-			(at 83.82 264.77 0)
-			(effects
-				(font
-					(size 1.27 1.27)
-				)
-				(justify left top)
-				(hide yes)
-			)
-		)
-		(property "Description" ""
-			(at 72.39 66.04 0)
-			(effects
-				(font
-					(size 1.27 1.27)
-				)
-				(hide yes)
-			)
-		)
-		(property "LCSC" "C13678"
-			(at 72.39 66.04 0)
-			(effects
-				(font
-					(size 1.27 1.27)
-				)
-				(hide yes)
-			)
-		)
-		(property "Mouser Part Number" "726-IPD050N10N5ATMA1"
-			(at 83.82 564.77 0)
-			(effects
-				(font
-					(size 1.27 1.27)
-				)
-				(justify left top)
-				(hide yes)
-			)
-		)
-		(property "Manufacturer_Name" "Infineon"
-			(at 83.82 764.77 0)
-			(effects
-				(font
-					(size 1.27 1.27)
-				)
-				(justify left top)
-				(hide yes)
-			)
-		)
-		(property "Manufacturer_Part_Number" "IPD050N10N5ATMA1"
-			(at 83.82 864.77 0)
-			(effects
-				(font
-					(size 1.27 1.27)
-				)
-				(justify left top)
-				(hide yes)
-			)
-		)
-		(property "Height" "2.41"
-			(at 83.82 464.77 0)
-			(effects
-				(font
-					(size 1.27 1.27)
-				)
-				(justify left top)
-				(hide yes)
-			)
-		)
-		(property "Mouser Price/Stock" "https://www.mouser.co.uk/ProductDetail/Infineon-Technologies/IPD050N10N5ATMA1?qs=u4fy%2FsgLU9Pgz4QwaVUqjg%3D%3D"
-			(at 83.82 664.77 0)
-			(effects
-				(font
-					(size 1.27 1.27)
-				)
-				(justify left top)
-				(hide yes)
-			)
-		)
-		(pin "1"
-		)
-		(pin "2"
-		)
-		(pin "3"
-		)
-		(instances
-			(project "boostUnit"
-				(path "/697a38d4-3409-462e-879c-d6eee2cce560"
-					(reference "BSQ1")
-					(unit 1)
-				)

Commit message: Boost Driver
Parts:
- BSU1: footprint Library:SON50P200X200X100-9N -> Package_SO:SOIC-8_3.9x4.9mm_P1.27mm
Changed lines of the file:
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@@
 			)
 		)
-		(property "Footprint" "Library:SON50P200X200X100-9N"
+		(property "Footprint" "Package_SO:SOIC-8_3.9x4.9mm_P1.27mm"
 			(at 41.91 66.04 0)
 			(effects
