File: camUnit/tof.kicad_sch (KiCad schematic)
At the start: 18 parts, among them J2 Conn_01x04, J3 Conn_01x06, J4 Conn_01x06, J5 Conn_01x06, J6 Conn_01x06, SW2 ENC RST, U2 STM32F103Cx, Y1 8Mhz

Commit message: Cam Layer
Parts:
- added R3, R4: 1k, Library:res0603, symbol Device:R
- added SW3: SW_SPDT, Library:SS12D00G3, symbol Switch:SW_SPDT
- J3, J4, J5, J6: footprint (none) -> Connector_JST:JST_PH_B6B-PH-K_1x06_P2.00mm_Vertical
Connections:
- net +3V3 FILT: now also R3.1, R4.1
- net TOF SCL: now also U2.42 (PB6), R3.2
- net TOF SDA: now also U2.43 (PB7), R4.2
- net TOF1: now also U2.18 (PB0)
- net TOF2: now also U2.19 (PB1)
- net TOF3: now also U2.20 (PB2)
- net TOF4: now also U2.39 (PB3)
- net TOF TX: now reaches U2.30 (PA9)
- net TOF RX: now reaches U2.31 (PA10)
- net +5V renamed TOF PWR
- net TOF PWR: now also SW3.2 (B)
- new net +5V FILT: SW3.1 (A)
- no-connect marks 3 -> 25

Commit message: CamUnit
Parts:
- added Q2: IRLML6344TRPBF, Library:SOT95P237X112-3N, symbol Library:IRLML6344TRPBF
- added R7, R8: 1k, Library:res0603, symbol Device:R
Connections:
- net +3V3 FILT: now also SW3.2 (B)
- net +5V FILT: now also R8.1; no longer SW3.1 (A)
- net GNDREF: now also Q2.2 (S), R7.2
- net TOF PWR: now also Q2.3 (D), R8.2; no longer SW3.2 (B)
- new net: Q2.1 (G), R7.1, SW3.1 (A)

Commit message: Fab
Parts:
- Y1: footprint Crystal:Resonator_SMD_Murata_CSTxExxV-3Pin_3.0x1.1mm -> Library:CSTCE8M00G52-R0
Changed lines of the file:
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@@
 (kicad_sch
-	(version 20231120)
+	(version 20250114)
 	(generator "eeschema")
-	(generator_version "8.0")
+	(generator_version "9.0")
 	(paper "A4")
 	(junction
@@
 			)
 		)
-		(property "Footprint" "Crystal:Resonator_SMD_Murata_CSTxExxV-3Pin_3.0x1.1mm"
+		(property "Footprint" "Library:CSTCE8M00G52-R0"
 			(at 39.37 86.36 0)
 			(effects
