File: camUnit/camUnit.kicad_sch (KiCad schematic)
At the start: 16 parts, among them J1 Conn_01x08, Q1 IRLML6344TRPBF, SW1 SW_SPDT

Commit message: CamUnit
Connections:
- net +3V3: now also J1.7 (Pin_7)
- net +3V3 FILT: no longer J1.7 (Pin_7)
- net +5V: now also J1.8 (Pin_8)
- net +5V FILT: no longer J1.8 (Pin_8)
Changed lines of the file:
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@@
 	(label "CAM PWR"
 		(at 163.83 64.77 0)
-		(fields_autoplaced yes)
 		(effects
 			(font
@@
 	(label "CAM PWR"
 		(at 214.63 48.26 0)
-		(fields_autoplaced yes)
 		(effects
 			(font
@@
 	(label "CAM RST"
 		(at 165.1 26.67 0)
-		(fields_autoplaced yes)
 		(effects
 			(font
@@
 	)
 	(symbol
-		(lib_id "power:+3V3")
-		(at 35.56 40.64 0)
-		(unit 1)
-		(exclude_from_sim no)
-		(in_bom yes)
-		(on_board yes)
-		(dnp no)
-		(fields_autoplaced yes)
-		(property "Reference" "#PWR08"
-			(at 35.56 44.45 0)
-			(effects
-				(font
-					(size 1.27 1.27)
-				)
-				(hide yes)
-			)
-		)
-		(property "Value" "+3V3 FILT"
-			(at 35.56 35.56 0)
-			(effects
-				(font
-					(size 1.27 1.27)
-				)
-			)
-		)
-		(property "Footprint" ""
-			(at 35.56 40.64 0)
-			(effects
-				(font
-					(size 1.27 1.27)
-				)
-				(hide yes)
-			)
-		)
-		(property "Datasheet" ""
-			(at 35.56 40.64 0)
-			(effects
-				(font
-					(size 1.27 1.27)
-				)
-				(hide yes)
-			)
-		)
-		(property "Description" "Power symbol creates a global label with name \"+3V3\""
-			(at 35.56 40.64 0)
-			(effects
-				(font
-					(size 1.27 1.27)
-				)
-				(hide yes)
-			)
-		)
-		(pin "1"
-		)
-		(instances
-			(project "camUnit"
-				(path "/6130ea90-01d1-434c-a614-117c329ecbc2"
-					(reference "#PWR08")
-					(unit 1)
-				)
-			)
-		)
-	)
-	(symbol
 		(lib_id "power:+5V")
 		(at 231.14 92.71 0)
@@
 	)
 	(symbol
-		(lib_id "power:+5V")
-		(at 30.48 38.1 0)
-		(unit 1)
-		(exclude_from_sim no)
-		(in_bom yes)
-		(on_board yes)
-		(dnp no)
-		(fields_autoplaced yes)
-		(property "Reference" "#PWR07"
-			(at 30.48 41.91 0)
-			(effects
-				(font
-					(size 1.27 1.27)
-				)
-				(hide yes)
-			)
-		)
-		(property "Value" "+5V FILT"
-			(at 30.48 33.02 0)
-			(effects
-				(font
-					(size 1.27 1.27)
-				)
-			)
-		)
-		(property "Footprint" ""
-			(at 30.48 38.1 0)
-			(effects
-				(font
-					(size 1.27 1.27)
-				)
-				(hide yes)
-			)
-		)
-		(property "Datasheet" ""
-			(at 30.48 38.1 0)
-			(effects
-				(font
-					(size 1.27 1.27)
-				)
-				(hide yes)
-			)
-		)
-		(property "Description" "Power symbol creates a global label with name \"+5V\""
-			(at 30.48 38.1 0)
-			(effects
-				(font
-					(size 1.27 1.27)
-				)
-				(hide yes)
-			)
-		)
-		(pin "1"
-		)
-		(instances
-			(project "camUnit"
-				(path "/6130ea90-01d1-434c-a614-117c329ecbc2"
-					(reference "#PWR07")
-					(unit 1)
-				)
-			)
-		)
-	)
-	(symbol
 		(lib_id "power:GNDREF")
 		(at 30.48 60.96 0)
@@
 	)
 	(symbol
+		(lib_id "power:+5V")
+		(at 30.48 38.1 0)
+		(unit 1)
+		(exclude_from_sim no)
+		(in_bom yes)
+		(on_board yes)
+		(dnp no)
+		(fields_autoplaced yes)
+		(property "Reference" "#PWR07"
+			(at 30.48 41.91 0)
+			(effects
+				(font
+					(size 1.27 1.27)
+				)
+				(hide yes)
+			)
+		)
+		(property "Value" "+5V"
+			(at 30.48 33.02 0)
+			(effects
+				(font
+					(size 1.27 1.27)
+				)
+			)
+		)
+		(property "Footprint" ""
+			(at 30.48 38.1 0)
+			(effects
+				(font
+					(size 1.27 1.27)
+				)
+				(hide yes)
+			)
+		)
+		(property "Datasheet" ""
+			(at 30.48 38.1 0)
+			(effects
+				(font
+					(size 1.27 1.27)
+				)
+				(hide yes)
+			)
+		)
+		(property "Description" "Power symbol creates a global label with name \"+5V\""
+			(at 30.48 38.1 0)
+			(effects
+				(font
+					(size 1.27 1.27)
+				)
+				(hide yes)
+			)
+		)
+		(pin "1"
+		)
+		(instances
+			(project "camUnit"
+				(path "/6130ea90-01d1-434c-a614-117c329ecbc2"
+					(reference "#PWR07")
+					(unit 1)
+				)
+			)
+		)
+	)
+	(symbol
 		(lib_id "Device:FerriteBead")
 		(at 201.93 96.52 90)
@@
 					(unit 1)
 				)
+			)
+		)
+	)
+	(symbol
+		(lib_id "power:+3V3")
+		(at 35.56 40.64 0)
+		(unit 1)
+		(exclude_from_sim no)
+		(in_bom yes)
+		(on_board yes)
+		(dnp no)
+		(fields_autoplaced yes)
+		(property "Reference" "#PWR08"
+			(at 35.56 44.45 0)
+			(effects
+				(font
+					(size 1.27 1.27)
+				)
+				(hide yes)
+			)
+		)
+		(property "Value" "+3V3"
+			(at 35.56 35.56 0)
+			(effects
+				(font
+					(size 1.27 1.27)
+				)
+			)
+		)
+		(property "Footprint" ""
+			(at 35.56 40.64 0)
+			(effects
+				(font
+					(size 1.27 1.27)
+				)
+				(hide yes)
+			)
+		)
+		(property "Datasheet" ""
+			(at 35.56 40.64 0)
+			(effects
+				(font
+					(size 1.27 1.27)
+				)
+				(hide yes)
+			)
+		)
+		(property "Description" "Power symbol creates a global label with name \"+3V3\""
+			(at 35.56 40.64 0)
+			(effects
+				(font
+					(size 1.27 1.27)
+				)
+				(hide yes)
+			)
+		)
+		(pin "1"
+		)
+		(instances
+			(project "camUnit"
+				(path "/6130ea90-01d1-434c-a614-117c329ecbc2"
+					(reference "#PWR08")
+					(unit 1)
+				)

Commit message: Damn u SPI
Parts:
- added Q305, Q306: IRLML6344TRPBF, Library:SOT95P237X112-3N, symbol Library:IRLML6344TRPBF
- added R351, R352, R353, R354: 1k, Library:res0603, symbol Device:R
- added SW303, SW305: SW_SPDT, Library:SS12D00G3, symbol Switch:SW_SPDT
- added U305: Teensy 4.0, Library:Teensy 4.0, symbol vincent:Teensy 4.0
- added U306: xiao-esp32c3, Library:xiao-esp32c3, symbol vincent:xiao-esp32c3
Connections:
- net +3V3 FILT: now also SW303.2 (B), SW305.2 (B)
- net +5V FILT: now also R353.1, R354.1
- net GNDREF: now also Q305.2 (S), Q306.2 (S), R351.2, R352.2, U305.G1, U305.G3 (GND), U306.12 (GND)
- new net: Q305.1 (G), R351.1, SW303.1 (A)
- new net: Q306.1 (G), R352.1, SW305.1 (A)
- new net BT PWR: Q306.3 (D), R353.2, U306.13 (5V)
- new net BT RX: U306.7 (RX)
- new net BT TX: U306.6 (TX)
- new net ENC NSS: U305.6
- new net ESC1: U305.9
- new net ESC2: U305.4
- new net FLAG: U305.3
- new net GATE RX: U305.21
- new net GATE TX: U305.20
- new net IMU STM NSS: U305.5
- new net KICK SIG: U305.2
- new net LIGHT RX: U305.7
- new net LIGHT TX: U305.8
- new net TEENSY PWR: Q305.3 (D), R354.2, U305.VIN
- new net TNSY ENC RX: U305.15
- new net TNSY ENC TX: U305.14
- new net TNSY IMU RX: U305.16
- new net TNSY IMU TX: U305.17
- new net TNSY L3 RX: U305.0
- new net TNSY L3 TX: U305.1
- no-connect marks 23 -> 44
