File: camUnit/camUnit-new.kicad_pcb (KiCad board)
At the start: 2 copper layers, 130 x 130 mm, 32 parts, among them J1 XH2.54, J2 Conn_01x06, J3 Conn_01x06, J4 Conn_01x06, J5 Conn_01x06, SW1 SW_SPDT, SW2 SW_SPDT, SW3 SW_SPDT, SW4 SW_SPDT, U2 BNO085, U3 xiao-esp32c3, U4 Teensy 4.0, U5 xiao-esp32c3

Commit message: Routed
Parts:
- added C5: 2u2, Library:cap0603, F.Cu at (106.4, 111.9)
- added C6: 2u2, Library:cap0603, F.Cu at (113.2, 111.9)
- added D2: 3V PWR, Library:led0603, F.Cu at (112.4, 115.3)
- added FB1: 100R, Library:fb0805, F.Cu at (109.8, 87.3)
- added FB2: 100R, Library:fb0805, F.Cu at (109.8, 112.7)
- added R6: 470, Library:res0603, F.Cu at (107.3, 115.3)
- J1: value XH2.54 -> Conn_01x06; footprint Connector_JST:JST_XH_S4B-XH-A_1x04_P2.50mm_Horizontal -> Connector_JST:JST_XH_S6B-XH-A_1x06_P2.50mm_Horizontal
- moved R3 156.8 mm to (107.2, 84.7), turned to 180 degrees
- moved C1 155.3 mm to (106.4, 88.1), turned to -90 degrees
- moved D1 151.1 mm to (112.3, 84.7)
- moved C2 149.1 mm to (113.2, 88.1), turned to -90 degrees
- moved SW4 123.5 mm to (129.2, 116.9)
- moved SW2 66.3 mm to (199.2, 76.3), turned to 90 degrees
- moved SW3 65.7 mm to (190.2, 139.2), turned to 180 degrees
- moved SW1 59.1 mm to (199.2, 85.8), turned to -90 degrees
- moved J1 2.50 mm to (112.5, 93.8)
- turned R2 to -90 degrees
Connections:
- J1 pad 2: /L3 TX -> +3V3
- J1 pad 3: /L3 RX -> /L3 TX
- J1 pad 4: GNDREF -> /L3 RX
- J2 pad 6: /TOF PWR -> +5V FILT
- J3 pad 6: /TOF PWR -> +5V FILT
- J4 pad 6: /TOF PWR -> +5V FILT
- J5 pad 6: /TOF PWR -> +5V FILT
- R4 pad 2: unconnected-(R4-Pad2) -> +3V3 FILT
- U1 pad 15: GND -> GNDREF
- U1 pad 31: GND -> GNDREF
- U3 pad 12: GND -> GNDREF
- U4 pad 16: /ESP TX -> /ESP1 TX
- U4 pad 17: /ESP RX -> /ESP1 RX
- U4 pad G3: GND -> GNDREF
Routing:
- net +5V FILT: track 0.00 -> 330.4 mm, vias 0 -> 2
- net /TOF SCL: track 0.00 -> 220.5 mm
- net /TOF SDA: track 0.00 -> 215.1 mm
- net /T1: track 0.00 -> 137.9 mm, vias 0 -> 3
- net /L3 RX: track 0.00 -> 111.9 mm
- net +3V3 FILT: track 0.00 -> 106.3 mm, vias 0 -> 4
- net /L3 TX: track 0.00 -> 103.0 mm
- net /T2: track 0.00 -> 95.8 mm
- net /ESP2 TX: track 0.00 -> 88.5 mm, vias 0 -> 2
- net /CAM TX: track 0.00 -> 79.3 mm
- net /CAM RX: track 0.00 -> 74.6 mm
- net /IMU CS: track 0.00 -> 73.9 mm
- net /ESP2 RX: track 0.00 -> 71.6 mm, vias 0 -> 1
- net /ESP1 RX: track 0.00 -> 63.0 mm, vias 0 -> 1
- net /IMU MOSI: track 0.00 -> 57.5 mm
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- added copper zone on F.Cu, net +3V3
- added copper zone on F.Cu, net +3V3 FILT
- added copper zone on F.Cu, net +5V
- added copper zone on F.Cu, net +5V FILT
- added copper zone on B.Cu, net GNDREF
- added copper zone on F.Cu, net GNDREF
Other:
- outline, holes or cut-outs redrawn

Commit message: serial
Parts:
- C1, C2, C5, C6, D1, D2, FB1, FB2, R3, R6: moved to B.Cu
- moved C1 0.84 mm to (105.6, 88.1)
- moved C2 0.84 mm to (112.3, 88.1)
- moved FB1 0.84 mm to (109.0, 87.3)
- moved R6 0.82 mm to (106.4, 115.3)
- moved D2 0.82 mm to (111.6, 115.3)
- moved C5 0.82 mm to (105.6, 112.0)
- moved C6 0.81 mm to (112.3, 111.9)
- moved R3 0.78 mm to (106.4, 84.7)
- moved D1 0.78 mm to (111.6, 84.7)
- moved FB2 0.76 mm to (109.0, 112.7)
Connections:
- U3 pad 1: /T3 -> /T1
- U3 pad 8: /T2 -> /T3
- U3 pad 9: /T1 -> /T2
Routing:
- net /L3 RX: track 111.9 -> 19.3 mm
- net /L3 TX: track 103.0 -> 13.1 mm
- net /ESP2 TX: track 88.5 -> 0.00 mm, vias 2 -> 0
- net /ESP2 RX: track 71.6 -> 0.00 mm, vias 1 -> 0
- net /TOF SDA: track 215.1 -> 274.2 mm
- net /T1: track 137.9 -> 86.9 mm, vias 3 -> 0
- net +5V FILT: track 330.4 -> 299.5 mm, vias 2 -> 0
- net /CAM TX: track 79.3 -> 59.0 mm
- net /IMU MOSI: track 57.5 -> 76.3 mm
- net /TOF SCL: track 220.5 -> 235.1 mm, vias 0 -> 2
- net /CAM RX: track 74.6 -> 62.0 mm
- net /T3: track 29.9 -> 18.0 mm
- net /T2: track 95.8 -> 84.0 mm, vias 0 -> 1
- net /IMU SCK: track 30.8 -> 42.5 mm
- net /IMU INT: track 40.2 -> 50.9 mm, vias 1 -> 0
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- added copper zone on B.Cu, net +3V3
- added copper zone on B.Cu, net +3V3 FILT
- added copper zone on B.Cu, net +5V
- added copper zone on B.Cu, net +5V FILT
- removed copper zone on F.Cu, net +3V3
- removed copper zone on F.Cu, net +5V
- removed copper zone on F.Cu, net +5V FILT

Commit message: cam prod ready
Connections:
- U4 pad 0: /L3 RX -> /ESP2 TX
- U4 pad 1: /L3 TX -> /ESP2 RX
- U4 pad 7: /ESP2 TX -> /L3 RX
- U4 pad 8: /ESP2 RX -> /L3 TX
Routing:
- net /ESP2 TX: track 0.00 -> 108.8 mm, vias 0 -> 2
- net /ESP2 RX: track 0.00 -> 94.3 mm, vias 0 -> 2
- net /L3 TX: track 13.1 -> 78.4 mm, vias 0 -> 2
- net /L3 RX: track 19.3 -> 83.9 mm, vias 0 -> 2
- net /T PWR: track 0.00 -> 5.32 mm
- net /TOF SDA: track 274.2 -> 272.4 mm

Commit message: cam prod ready
Parts:
- U3, U5: value xiao-esp32c3 -> >VALUE
- moved R4 0.12 mm to (179.9, 123.4)
- moved R5 0.12 mm to (182.5, 123.4)

Commit message: routing
Parts:
- removed H3, H4, H5, H6: MountingHole_Pad, MountingHole:MountingHole_3.2mm_M3_Pad_Via
- moved C1 1.00 mm to (106.6, 88.1)
- moved C2 1.00 mm to (113.3, 88.1)
- moved C5 1.00 mm to (106.6, 112.0)
- moved C6 1.00 mm to (113.3, 111.9)
- moved D1 1.00 mm to (112.6, 84.7)
- moved D2 1.00 mm to (112.6, 115.3)
- moved FB1 1.00 mm to (110.0, 87.3)
- moved FB2 1.00 mm to (110.0, 112.7)
- moved R3 1.00 mm to (107.4, 84.7)
- moved R6 1.00 mm to (107.4, 115.3)
Other:
- board size 130 x 130 mm -> 118 x 120.1 mm

Commit message: fab + 3d model
Parts:
- U3, U5: value >VALUE -> xiao-esp32c3
- renumbered H8 to H3, H7 to H4
Other:
- outline, holes or cut-outs redrawn
