File: camUnit/camUnit-new.kicad_pcb (KiCad board)
At the start: 2 copper layers, 118 x 120.1 mm, 34 parts, among them J1 Conn_01x06, J2 Conn_01x06, J3 Conn_01x06, J4 Conn_01x06, J5 Conn_01x06, SW1 SW_SPDT, SW2 SW_SPDT, SW3 SW_SPDT, SW4 SW_SPDT, U2 BNO085, U3 xiao-esp32c3, U4 Teensy 4.0, U5 xiao-esp32c3

Commit message: 3d models
Routing:
- net /ESP2 RX: track 94.3 -> 93.3 mm

Commit message: switch position
Parts:
- moved R3 109.5 mm to (212.6, 115.3), turned to 0 degrees
- moved R6 109.5 mm to (212.6, 84.7), turned to 0 degrees
- moved C5 109.5 mm to (213.4, 88.0), turned to -90 degrees
- moved C1 109.4 mm to (213.4, 111.9), turned to 90 degrees
- moved FB1 103.2 mm to (210.0, 112.7), turned to 180 degrees
- moved FB2 103.2 mm to (210.0, 87.3), turned to 180 degrees
- moved D1 99.7 mm to (207.4, 115.3), turned to 180 degrees
- moved D2 99.7 mm to (207.4, 84.7), turned to 180 degrees
- moved C2 96.3 mm to (206.6, 111.9), turned to 90 degrees
- moved C6 96.3 mm to (206.6, 88.1), turned to -90 degrees
- moved J1 95.9 mm to (207.5, 106.2), turned to 90 degrees
Routing:
- net /L3 RX: track 83.9 -> 63.8 mm, vias 2 -> 1
- net +3V3 FILT: track 100.4 -> 120.4 mm, vias 2 -> 4
- net /L3 TX: track 78.4 -> 67.7 mm, vias 2 -> 1
- net +5V FILT: track 299.5 -> 304.4 mm
- net /TOF SCL: track 235.0 -> 233.4 mm
- net /TOF SDA: track 272.7 -> 271.3 mm

Commit message: fab
Parts:
- moved H2 124.4 mm to (126.8, 47.4), turned to 180 degrees
- moved H3 124.4 mm to (126.8, 152.6), turned to 180 degrees
- moved H1 124.4 mm to (193.2, 47.4), turned to 180 degrees
- moved H4 124.4 mm to (193.2, 152.6), turned to 180 degrees
- moved R3 109.5 mm to (107.4, 84.7), turned to 180 degrees
- moved R6 109.5 mm to (107.4, 115.3), turned to 180 degrees
- moved C5 109.5 mm to (106.6, 112.0), turned to 90 degrees
- moved C1 109.4 mm to (106.6, 88.1), turned to -90 degrees
- moved FB1 103.2 mm to (110.0, 87.3), turned to 0 degrees
- moved FB2 103.2 mm to (110.0, 112.7), turned to 0 degrees
- moved D1 99.7 mm to (112.6, 84.7), turned to 0 degrees
- moved D2 99.7 mm to (112.6, 115.3), turned to 0 degrees
- moved SW3 98.9 mm to (129.8, 60.8), turned to 0 degrees
- moved C2 96.3 mm to (113.3, 88.1), turned to -90 degrees
- moved C6 96.3 mm to (113.3, 111.9), turned to 90 degrees
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Other:
- outline, holes or cut-outs redrawn

Commit message: step
Routing:
- net +5V FILT: track 304.4 -> 297.4 mm
Other:
- board text added: "JLCJLCJLCJLC"
