File: camUnit/camUnit-new.kicad_sch (KiCad schematic)
At the start: 33 parts, among them J1 XH2.54, J2 Conn_01x06, J3 Conn_01x06, J4 Conn_01x06, J5 Conn_01x06, SW1 SW_SPDT, SW2 SW_SPDT, SW3 SW_SPDT, SW4 SW_SPDT, U2 BNO085, U3 xiao-esp32c3, U4 Teensy 4.0, U5 xiao-esp32c3

Commit message: Routed
Parts:
- removed J1: XH2.54, Connector_JST:JST_XH_S4B-XH-A_1x04_P2.50mm_Horizontal, symbol Connector_Generic:Conn_01x04
- added C5, C6: 2u2, Library:cap0603, symbol Device:C
- added D2: 3V PWR, Library:led0603, symbol Device:LED
- added FB2: 100R, Library:fb0805, symbol Device:FerriteBead
- added J1: Conn_01x06, Connector_JST:JST_XH_S6B-XH-A_1x06_P2.50mm_Horizontal, symbol Connector_Generic:Conn_01x06
- added R6: 470, Library:res0603, symbol Device:R
Connections:
- net ESP RX is gone; now on net ESP1 RX: U4.17
- net ESP TX is gone; now on net ESP1 TX: U4.16
- net TOF PWR is gone; now on net +5V FILT: J2.6 (Pin_6), J3.6 (Pin_6), J4.6 (Pin_6), J5.6 (Pin_6)
- net +3V3 FILT: now also R4.2, C6.1, D2.2 (A), FB2.2
- net +5V: now also J1.1 (Pin_1)
- net GND: no longer U1.15 (GND), U1.31 (GND), U3.12 (GND), U4.G3 (GND)
- net GNDREF: now also U1.15 (GND), U1.31 (GND), U3.12 (GND), U4.G3 (GND), C5.2, C6.2, J1.5 (Pin_5), J1.6 (Pin_6), R6.2
- net L3 RX: now also J1.4 (Pin_4)
- net L3 TX: now also J1.3 (Pin_3)
- new net: D2.1 (K), R6.1
- new net +3V3: C5.1, FB2.1, J1.2 (Pin_2)
- no-connect marks 60 -> 62
Other:
- moved on the sheet: J3, J5, SW1, SW2, SW3, SW4, U4

Commit message: serial
Connections:
- net T1: now also U3.1 (A1); no longer U3.9 (MISO)
- net T2: now also U3.9 (MISO); no longer U3.8 (SCK)
- net T3: now also U3.8 (SCK); no longer U3.1 (A1)
Changed lines of the file:
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@@
-		)
-	)
-	(label "T2"
-		(at 193.04 121.92 180)
-		(effects
-			(font
-				(size 1.27 1.27)
-			)
-			(justify right bottom)
 		)
 	)
@@
 	(label "TOF SCL"
 		(at 157.48 121.92 0)
-		(effects
-			(font
-				(size 1.27 1.27)
-			)
-			(justify left bottom)
-		)
-	)
-	(label "T3"
-		(at 157.48 111.76 0)
 		(effects
 			(font
@@
 		)
 	)
+	(label "T1"
+		(at 157.48 111.76 0)
+		(effects
+			(font
+				(size 1.27 1.27)
+			)
+			(justify left bottom)
+		)
+	)
 	(label "TOF SCL"
 		(at 214.63 107.95 0)
@@
 		)
 	)
-	(label "T1"
-		(at 193.04 119.38 180)
-		(effects
-			(font
-				(size 1.27 1.27)
-			)
-			(justify right bottom)
-		)
-	)
 	(label "TOF PWR"
 		(at 214.63 132.08 0)
@@
 		)
 	)
+	(label "T3"
+		(at 193.04 121.92 180)
+		(effects
+			(font
+				(size 1.27 1.27)
+			)
+			(justify right bottom)
+		)
+	)
 	(label "T4"
 		(at 157.48 109.22 0)
@@
 		)
 	)
+	(label "T2"
+		(at 193.04 119.38 180)
+		(effects
+			(font
+				(size 1.27 1.27)
+			)
+			(justify right bottom)
+		)
+	)

Commit message: cam prod ready
Connections:
- net ESP2 RX: now also U4.1; no longer U4.8
- net ESP2 TX: now also U4.0; no longer U4.7
- net L3 RX: now also U4.7; no longer U4.0
- net L3 TX: now also U4.8; no longer U4.1
Changed lines of the file:
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@@
-		)
-	)
-	(label "L3 TX"
-		(at 266.7 41.91 0)
-		(effects
-			(font
-				(size 1.27 1.27)
-			)
-			(justify left bottom)
-		)
-	)
-	(label "ESP2 RX"
-		(at 265.43 59.69 0)
-		(effects
-			(font
-				(size 1.27 1.27)
-			)
-			(justify left bottom)
 		)
 	)
@@
 	)
 	(label "L3 RX"
-		(at 266.7 39.37 0)
-		(effects
-			(font
-				(size 1.27 1.27)
-			)
-			(justify left bottom)
-		)
-	)
-	(label "L3 RX"
 		(at 53.34 54.61 180)
 		(effects
@@
 		)
 	)
+	(label "L3 RX"
+		(at 265.43 57.15 0)
+		(effects
+			(font
+				(size 1.27 1.27)
+			)
+			(justify left bottom)
+		)
+	)
 	(label "IMU CS"
 		(at 60.96 133.35 0)
@@
 		)
 	)
+	(label "ESP2 TX"
+		(at 266.7 39.37 0)
+		(effects
+			(font
+				(size 1.27 1.27)
+			)
+			(justify left bottom)
+		)
+	)
 	(label "IMU RST"
 		(at 321.31 64.77 180)
@@
 		)
 	)
-	(label "ESP2 TX"
-		(at 265.43 57.15 0)
-		(effects
-			(font
-				(size 1.27 1.27)
-			)
-			(justify left bottom)
-		)
-	)
 	(label "CAM RX"
 		(at 30.48 205.74 0)
@@
 		)
 	)
+	(label "L3 TX"
+		(at 265.43 59.69 0)
+		(effects
+			(font
+				(size 1.27 1.27)
+			)
+			(justify left bottom)
+		)
+	)
 	(label "TOF SDA"
 		(at 246.38 105.41 0)
@@
 			)
 			(justify right bottom)
+		)
+	)
+	(label "ESP2 RX"
+		(at 266.7 41.91 0)
+		(effects
+			(font
+				(size 1.27 1.27)
+			)
+			(justify left bottom)
 		)
 	)
@@
 		)
 		(pin "1"
+			(alternate "TX1")
 		)
 		(pin "19"
@@
 		)
 		(pin "0"
+			(alternate "RX1")
 		)
 		(pin "5"

Commit message: fab + 3d model
Parts:
- removed H5, H6, H7, H8: MountingHole_Pad, MountingHole:MountingHole_3.2mm_M3_Pad_Via, symbol Mechanical:MountingHole_Pad
Connections:
- no-connect marks 62 -> 58

Commit message: step
Changed lines of the file:
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@@
 		)
 		(pin "16"
+			(alternate "RX4")
 		)
 		(pin "3.3V_2"
@@
 		)
 		(pin "17"
+			(alternate "TX4")
 		)
 		(pin "23"
@@
 		)
 		(pin "21"
+			(alternate "RX5")
 		)
 		(pin "20"
+			(alternate "TX5")
 		)
 		(pin "13"
