File: breakout/Capacitor Bank/Capacitor Bank.kicad_pcb (KiCad board)
At the start: 2 copper layers, 72.7 x 33.9 mm, 9 parts, among them J1 Conn_01x02

Commit message: JLCJLJCJLCJLC
Other:
- board text added: "JLCJLCJLCJLC"
Changed lines of the file:
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@@
 		(layer "Edge.Cuts")
+	)
+	(gr_text "JLCJLCJLCJLC"
+		(at 124.200001 111.930173 0)
+		(layer "F.SilkS")
+		(effects
+			(font
+				(size 1.3 1.3)
+				(thickness 0.3)
+				(bold yes)
+			)
+			(justify left bottom)
+		)
 	)
 	(zone

Commit message: update
Connections:
- J1 pad 1: +24V -> GNDREF
- J1 pad 2: GNDREF -> +24V
Changed lines of the file:
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@@
 				(font
 					(size 1.27 1.27)
+					(thickness 0.15)
 				)
 			)
@@
 				(font
 					(size 1.27 1.27)
+					(thickness 0.15)
 				)
 			)
@@
 				(font
 					(size 1.27 1.27)
+					(thickness 0.15)
 				)
 			)
@@
 				(font
 					(size 1.27 1.27)
+					(thickness 0.15)
 				)
 			)
@@
 				(font
 					(size 1.27 1.27)
+					(thickness 0.15)
 				)
 			)
@@
 				(font
 					(size 1.27 1.27)
+					(thickness 0.15)
 				)
 			)
@@
 			(remove_unused_layers no)
 			(roundrect_rratio 0.22)
-			(net 1 "+24V")
+			(net 2 "GNDREF")
 			(pinfunction "Pin_1")
 			(pintype "passive")
@@
 			(layers "*.Cu" "*.Mask")
 			(remove_unused_layers no)
-			(net 2 "GNDREF")
+			(net 1 "+24V")
 			(pinfunction "Pin_2")
 			(pintype "passive")
@@
 				(font
 					(size 1.27 1.27)
+					(thickness 0.15)
 				)
 			)
@@
 				(font
 					(size 1.27 1.27)
+					(thickness 0.15)
 				)
 			)
@@
 				(font
 					(size 1.27 1.27)
+					(thickness 0.15)
 				)
 			)
@@
 				(font
 					(size 1.27 1.27)
+					(thickness 0.15)
 				)
 			)
@@
 				(font
 					(size 1.27 1.27)
+					(thickness 0.15)
 				)
 			)
@@
 				(font
 					(size 1.27 1.27)
+					(thickness 0.15)
 				)
 			)
@@
 		(polygon
 			(pts
-				(xy 150.000001 106.530173) (xy 145.000001 106.530173) (xy 145.000001 101.730173) (xy 139.800001 101.730173)
+				(xy 154.550001 106.530173) (xy 150.370001 106.550173) (xy 150.370001 101.750173) (xy 139.800001 101.730173)
 				(xy 139.800001 111.530173) (xy 131.000001 111.530173) (xy 131.000001 93.930173) (xy 169.800001 93.930173)
-				(xy 169.800001 111.130173) (xy 160.200001 111.130173) (xy 160.200001 101.730173) (xy 150.000001 101.730173)
-			)
-		)
+				(xy 169.800001 111.130173) (xy 160.200001 111.130173) (xy 160.200001 101.730173) (xy 154.550001 101.730173)
+			)
+		)
